Commit message: update urdf to source mesh from kortex_description

File: kortex_description/urdf/JACO3_URDF_V10.urdf (robot description, URDF)
Before this commit: robot JACO3_URDF_V10, 9 links, 8 joints
Links:
- link Bracelet_Link: geometry collision mesh filename=package://kortex_description/meshes/Bracelet_Link.STL; visual mesh filename=package://kortex_description/meshes/Bracelet_Link.STL
- link EndEffector_Link: geometry collision mesh filename=package://kortex_description/meshes/EndEffector_Link.STL; visual mesh filename=package://kortex_description/meshes/EndEffector_Link.STL
- link ForeArm_Link: geometry collision mesh filename=package://kortex_description/meshes/ForeArm_Link.STL; visual mesh filename=package://kortex_description/meshes/ForeArm_Link.STL
- link HalfArm1_Link: geometry collision mesh filename=package://kortex_description/meshes/HalfArm1_Link.STL; visual mesh filename=package://kortex_description/meshes/HalfArm1_Link.STL
- link HalfArm2_Link: geometry collision mesh filename=package://kortex_description/meshes/HalfArm2_Link.STL; visual mesh filename=package://kortex_description/meshes/HalfArm2_Link.STL
- link Shoulder_Link: geometry collision mesh filename=package://kortex_description/meshes/Shoulder_Link.STL; visual mesh filename=package://kortex_description/meshes/Shoulder_Link.STL
- link Wrist1_Link: geometry collision mesh filename=package://kortex_description/meshes/Wrist1_Link.STL; visual mesh filename=package://kortex_description/meshes/Wrist1_Link.STL
- link Wrist2_Link: geometry collision mesh filename=package://kortex_description/meshes/Wrist2_Link.STL; visual mesh filename=package://kortex_description/meshes/Wrist2_Link.STL
- link base_link: geometry collision mesh filename=package://kortex_description/meshes/base_link.STL; visual mesh filename=package://kortex_description/meshes/base_link.STL
