Commit message: Added kortex_control package and updated the kortex_description package for release 2.0

File: kortex_description/arms/gen3/urdf/gen3_macro.xacro (robot description, xacro)
@@ -4,81 +4,45 @@
   <xacro:property name="last_arm_link" value="end_effector_link"/>
   <xacro:macro name="load_arm" params="parent:='' *origin">
-    <link
-      name="base_link">
-      <inertial>
-        <origin
-          xyz="-0.000648 -0.000166 0.084487"
-          rpy="0 0 0" />
-        <mass
-          value="1.697353" />
-        <inertia
-          ixx="0.004622"
-          ixy="9E-06"
-          ixz="6E-05"
-          iyy="0.004495"
-          iyz="9E-06"
-          izz="0.002079" />
-      </inertial>
-      <visual>
-        <origin
-          xyz="0 0 0"
-          rpy="0 0 0" />
-        <geometry>
-          <mesh
-            filename="package://kortex_description/arms/gen3/meshes/base_link.STL" />
-        </geometry>
-        <material
-          name="">
-          <color
-            rgba="0.79216 0.81961 0.93333 1" />
-        </material>
-      </visual>
-      <collision>
-        <origin
-          xyz="0 0 0"
-          rpy="0 0 0" />
-        <geometry>
-          <mesh
-            filename="package://kortex_description/arms/gen3/meshes/base_link.STL" />
-        </geometry>
-      </collision>
-    </link>
-    <link
-      name="shoulder_link">
-      <inertial>
-        <origin
-          xyz="-2.3E-05 -0.010364 -0.07336"
-          rpy="0 0 0" />
-        <mass
-          value="1.377353" />
-        <inertia
-          ixx="0.00457"
-          ixy="1E-06"
-          ixz="2E-06"
-          iyy="0.004831"
-          iyz="0.000448"
-          izz="0.001409" />
-      </inertial>
-      <visual>
-        <origin
-          xyz="0 0 0"
-          rpy="0 0 0" />
-        <geometry>
-          <mesh
-            filename="package://kortex_description/arms/gen3/meshes/shoulder_link.STL" />
-        </geometry>
-        <material
-          name="">
-          <color
-            rgba="0.75294 0.75294 0.75294 1" />
-        </material>
-      </visual>
-      <collision>
-        <origin
-          xyz="0 0 0"
-          rpy="0 0 0" />
-        <geometry>
-          <mesh
-            filename="package://kortex_description/arms/gen3/meshes/shoulder_link.STL" />
+      <link name="base_link">
+        <inertial>
+          <origin xyz="-0.000648 -0.000166 0.084487" rpy="0 0 0" />
+          <mass value="1.697" />
+          <inertia ixx="0.004622" ixy="9E-06" ixz="6E-05" iyy="0.004495" iyz="9E-06" izz="0.002079" />
+        </inertial>
+        <visual>
+          <origin xyz="0 0 0" rpy="0 0 0" />
+          <geometry>
+            <mesh filename="package://kortex_description/arms/gen3/meshes/base_link.STL" />
+          </geometry>
+          <material name="">
+            <color rgba="0.75294 0.75294 0.75294 1" />
+          </material>
+        </visual>
+        <collision>
+          <origin xyz="0 0 0" rpy="0 0 0" />
+          <geometry>
+            <mesh filename="package://kortex_description/arms/gen3/meshes/base_link.STL" />
+          </geometry>
+        </collision>
+    </link>
+    <link name="shoulder_link">
+      <inertial>
+        <origin xyz="-2.3E-05 -0.010364 -0.07336" rpy="0 0 0" />
+        <mass value="1.3773" />
+        <inertia ixx="0.00457" ixy="1E-06" ixz="2E-06" iyy="0.004831" iyz="0.000448" izz="0.001409" />
+      </inertial>
+      <visual>
+        <origin xyz="0 0 0" rpy="0 0 0" />
+        <geometry>
+          <mesh filename="package://kortex_description/arms/gen3/meshes/shoulder_link.STL" />
+        </geometry>
+        <material name="">
+          <color rgba="0.75294 0.75294 0.75294 1" />
+        </material>
+      </visual>
+      <collision>
+        <origin xyz="0 0 0" rpy="0 0 0" />
+        <geometry>
+          <mesh filename="package://kortex_description/arms/gen3/meshes/shoulder_link.STL" />
         </geometry>
       </collision>
@@ -87,7 +51,5 @@
       name="joint_1"
       type="continuous">
-      <origin
-        xyz="6.1995E-05 0 0.15643"
-        rpy="-3.1416 3.2891E-18 1.9637E-50" />
+      <origin xyz="0 0 0.15643" rpy="3.1416 2.7629E-18 -4.9305E-36" />
       <parent
         link="base_link" />
@@ -100,41 +62,23 @@
         velocity="0.8727" />
     </joint>
-    <link
-      name="half_arm_1_link">
-      <inertial>
-        <origin
-          xyz="-4.4E-05 -0.09958 -0.013278"
-          rpy="0 0 0" />
-        <mass
-          value="1.163667" />
-        <inertia
-          ixx="0.011088"
-          ixy="5E-06"
-          ixz="0"
-          iyy="0.001072"
-          iyz="-0.000691"
-          izz="0.011255" />
-      </inertial>
-      <visual>
-        <origin
-          xyz="0 0 0"
-          rpy="0 0 0" />
-        <geometry>
-          <mesh
-            filename="package://kortex_description/arms/gen3/meshes/half_arm_1_link.STL" />
-        </geometry>
-        <material
-          name="">
-          <color
-            rgba="0.75294 0.75294 0.75294 1" />
-        </material>
-      </visual>
-      <collision>
-        <origin
-          xyz="0 0 0"
-          rpy="0 0 0" />
-        <geometry>
-          <mesh
-            filename="package://kortex_description/arms/gen3/meshes/half_arm_1_link.STL" />
+    <link name="half_arm_1_link">
+      <inertial>
+        <origin xyz="-4.4E-05 -0.09958 -0.013278" rpy="0 0 0" />
+        <mass value="1.1636" />
+        <inertia ixx="0.011088" ixy="5E-06" ixz="0" iyy="0.001072" iyz="-0.000691" izz="0.011255" />
+      </inertial>
+      <visual>
+        <origin xyz="0 0 0" rpy="0 0 0" />
+        <geometry>
+          <mesh filename="package://kortex_description/arms/gen3/meshes/half_arm_1_link.STL" />
+        </geometry>
+        <material name="">
+          <color rgba="0.75294 0.75294 0.75294 1" />
+        </material>
+      </visual>
+      <collision>
+        <origin xyz="0 0 0" rpy="0 0 0" />
+        <geometry>
+          <mesh filename="package://kortex_description/arms/gen3/meshes/half_arm_1_link.STL" />
         </geometry>
       </collision>
@@ -143,7 +87,5 @@
       name="joint_2"
       type="revolute">
-      <origin
-        xyz="0 0.005375 -0.12838"
-        rpy="1.5708 2.4106E-17 3.1919E-16" />
+      <origin xyz="0 0.005375 -0.12838" rpy="1.5708 2.1343E-17 -1.1102E-16" />
       <parent
         link="shoulder_link" />
@@ -152,103 +94,61 @@
       <axis
         xyz="0 0 1" />
-      <limit
-        lower="-2.2"
-        upper="2.2"
+      <limit lower="-2.41" upper="2.41" effort="39" velocity="0.8727" />
+    </joint>
+    <link name="half_arm_2_link">
+      <inertial>
+        <origin xyz="-4.4E-05 -0.006641 -0.117892" rpy="0 0 0" />
+        <mass value="1.1636" />
+        <inertia ixx="0.010932" ixy="0" ixz="-7E-06" iyy="0.011127" iyz="0.000606" izz="0.001043" />
+      </inertial>
+      <visual>
+        <origin xyz="0 0 0" rpy="0 0 0" />
+        <geometry>
+          <mesh filename="package://kortex_description/arms/gen3/meshes/half_arm_2_link.STL" />
+        </geometry>
+        <material name="">
+          <color rgba="0.75294 0.75294 0.75294 1" />
+        </material>
+      </visual>
+      <collision>
+        <origin xyz="0 0 0" rpy="0 0 0" />
+        <geometry>
+          <mesh filename="package://kortex_description/arms/gen3/meshes/half_arm_2_link.STL" />
+        </geometry>
+      </collision>
+    </link>
+    <joint
+      name="joint_3"
+      type="continuous">
+      <origin xyz="0 -0.21038 -0.006375" rpy="-1.5708 1.2326E-32 -2.9122E-16" />
+      <parent
+        link="half_arm_1_link" />
+      <child
+        link="half_arm_2_link" />
+      <axis
+        xyz="0 0 1" />
+      <limit
         effort="39"
         velocity="0.8727" />
     </joint>
-    <link
-      name="half_arm_2_link">
-      <inertial>
-        <origin
-          xyz="-4.4E-05 -0.006641 -0.117892"
-          rpy="0 0 0" />
-        <mass
-          value="1.16366" />
-        <inertia
-          ixx="0.010932"
-          ixy="0"
-          ixz="-7E-06"
-          iyy="0.011127"
-          iyz="0.000606"
-          izz="0.001043" />
-      </inertial>
-      <visual>
-        <origin
-          xyz="0 0 0"
-          rpy="0 0 0" />
-        <geometry>
-          <mesh
-            filename="package://kortex_description/arms/gen3/meshes/half_arm_2_link.STL" />
-        </geometry>
-        <material
-          name="">
-          <color
-            rgba="0.75294 0.75294 0.75294 1" />
-        </material>
-      </visual>
-      <collision>
-        <origin
-          xyz="0 0 0"
-          rpy="0 0 0" />
-        <geometry>
-          <mesh
-            filename="package://kortex_description/arms/gen3/meshes/half_arm_2_link.STL" />
-        </geometry>
-      </collision>
-    </link>
-    <joint
-      name="joint_3"
-      type="continuous">
-      <origin
-        xyz="0 -0.21038 -0.006375"
-        rpy="-1.5708 9.8608E-32 -2.7983E-16" />
-      <parent
-        link="half_arm_1_link" />
-      <child
-        link="half_arm_2_link" />
-      <axis
-        xyz="0 0 1" />
-      <limit
-        effort="39"
-        velocity="0.8727" />
-    </joint>
-    <link
-      name="forearm_link">
-      <inertial>
-        <origin
-          xyz="-1.8E-05 -0.075478 -0.015006"
-          rpy="0 0 0" />
-        <mass
-          value="0.930287" />
-        <inertia
-          ixx="0.008147"
-          ixy="-1E-06"
-          ixz="0"
-          iyy="0.000631"
-          iyz="-0.0005"
-          izz="0.008316" />
-      </inertial>
-      <visual>
-        <origin
-          xyz="0 0 0"
-          rpy="0 0 0" />
-        <geometry>
-          <mesh
-            filename="package://kortex_description/arms/gen3/meshes/forearm_link.STL" />
-        </geometry>
-        <material
-          name="">
-          <color
-            rgba="0.75294 0.75294 0.75294 1" />
-        </material>
-      </visual>
-      <collision>
-        <origin
-          xyz="0 0 0"
-          rpy="0 0 0" />
-        <geometry>
-          <mesh
-            filename="package://kortex_description/arms/gen3/meshes/forearm_link.STL" />
+    <link name="forearm_link">
+      <inertial>
+        <origin xyz="-1.8E-05 -0.075478 -0.015006" rpy="0 0 0" />
+        <mass value="0.9302" />
+        <inertia ixx="0.008147" ixy="-1E-06" ixz="0" iyy="0.000631" iyz="-0.0005" izz="0.008316" />
+      </inertial>
+      <visual>
+        <origin xyz="0 0 0" rpy="0 0 0" />
+        <geometry>
+          <mesh filename="package://kortex_description/arms/gen3/meshes/forearm_link.STL" />
+        </geometry>
+        <material name="">
+          <color rgba="0.75294 0.75294 0.75294 1" />
+        </material>
+      </visual>
+      <collision>
+        <origin xyz="0 0 0" rpy="0 0 0" />
+        <geometry>
+          <mesh filename="package://kortex_description/arms/gen3/meshes/forearm_link.STL" />
         </geometry>
       </collision>
@@ -257,7 +157,5 @@
       name="joint_4"
       type="revolute">
-      <origin
-        xyz="0 0.006375 -0.21038"
-        rpy="1.5708 3.0688E-17 -6.9389E-18" />
+      <origin xyz="0 0.006375 -0.21038" rpy="1.5708 -6.6954E-17 -1.6653E-16" />
       <parent
         link="half_arm_2_link" />
@@ -266,47 +164,25 @@
       <axis
         xyz="0 0 1" />
-      <limit
-        lower="-2.5656"
-        upper="2.5656"
-        effort="39"
-        velocity="0.8727" />
-    </joint>
-    <link
-      name="spherical_wrist_1_link">
-      <inertial>
-        <origin
-          xyz="1E-06 -0.009432 -0.063883"
-          rpy="0 0 0" />
-        <mass
-          value="0.678106" />
-        <inertia
-          ixx="0.001596"
-          ixy="0"
-          ixz="0"
-          iyy="0.001607"
-          iyz="0.000256"
-          izz="0.000399" />
-      </inertial>
-      <visual>
-        <origin
-          xyz="0 0 0"
-          rpy="0 0 0" />
-        <geometry>
-          <mesh
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
File: kortex_description/robots/gen3_robotiq_2f_85.xacro (robot description, xacro)
@@ -1,9 +1,9 @@
 <?xml version="1.0"?>
-<robot name="gen3" xmlns:xacro="http://ros.org/wiki/xacro">
+<robot name="gen3_robotiq_2f_85" xmlns:xacro="http://ros.org/wiki/xacro">
     <!-- Arguments -->
     <xacro:arg name="arm" default="gen3" />
-    <xacro:arg name="gripper" default="" />
+    <xacro:arg name="gripper" default="robotiq_2f_85" />
     <xacro:arg name="sim" default="false" />
     <xacro:include filename="$(find kortex_description)/robots/kortex_robot.xacro" />
-    <xacro:load_robot arm="$(arg arm)" gripper="$(arg gripper)" sim="$(arg sim)" />
+    <xacro:load_robot arm="$(arg arm)" gripper="$(arg gripper)" sim="$(arg sim)"/>
 </robot>
