Commit message: Add custom colours for Gen3 lite simulation - more realistic textures to come later

File: kortex_description/arms/gen3_lite/6dof/urdf/gen3_lite_macro.xacro (robot description, xacro)
@@ -26,4 +26,7 @@
       </collision>
     </link>
+    <gazebo reference="${prefix}base_link">
+      <material>Kortex/Gray</material>
+    </gazebo>
     <link name="${prefix}shoulder_link">
       <inertial>
@@ -48,4 +51,7 @@
       </collision>
     </link>
+    <gazebo reference="${prefix}shoulder_link">
+      <material>Kortex/Gray</material>
+    </gazebo>
     <joint name="${prefix}joint_1" type="revolute">
       <origin xyz="0 0 0.12825" rpy="0 0 0" />
@@ -77,4 +83,7 @@
       </collision>
     </link>
+    <gazebo reference="${prefix}arm_link">
+      <material>Kortex/Gray</material>
+    </gazebo>
     <joint name="${prefix}joint_2" type="revolute">
       <origin xyz="0 -0.03 0.115" rpy="1.5708 0 0" />
@@ -106,4 +115,7 @@
       </collision>
     </link>
+    <gazebo reference="${prefix}forearm_link">
+      <material>Kortex/Gray</material>
+    </gazebo>
     <joint name="${prefix}joint_3" type="revolute">
       <origin xyz="0 0.28 0" rpy="-3.1416 0 0" />
@@ -135,4 +147,7 @@
       </collision>
     </link>
+    <gazebo reference="${prefix}lower_wrist_link">
+      <material>Kortex/Gray</material>
+    </gazebo>
     <joint name="${prefix}joint_4" type="revolute">
       <origin xyz="0 -0.14 0.02" rpy="1.5708 0 0" />
@@ -164,4 +179,7 @@
       </collision>
     </link>
+    <gazebo reference="${prefix}upper_wrist_link">
+      <material>Kortex/Gray</material>
+    </gazebo>
     <joint name="${prefix}joint_5" type="revolute">
       <origin xyz="0.0285 0 0.105" rpy="0 1.5708 0" />

File: kortex_description/grippers/gen3_lite_2f/urdf/gen3_lite_2f_macro.xacro (robot description, xacro)
@@ -30,4 +30,7 @@
       </collision>
     </link>
+    <gazebo reference="${prefix}gripper_base_link">
+      <material>Kortex/Gray</material>
+    </gazebo>
     <link name="${prefix}right_finger_prox_link">
     <inertial>
@@ -52,4 +55,7 @@
     </collision>
     </link>
+    <gazebo reference="${prefix}right_finger_prox_link">
+      <material>Gazebo/Black</material>
+    </gazebo>
     <joint name="${prefix}right_finger_bottom_joint" type="revolute">
       <origin xyz="0 -0.030501 0.070003" rpy="0 1.5708 0" />
@@ -81,4 +87,7 @@
       </collision>
     </link>
+    <gazebo reference="${prefix}right_finger_dist_link">
+      <material>Kortex/Blue</material>
+    </gazebo>
     <joint name="${prefix}right_finger_tip_joint" type="revolute">
       <origin xyz="-0.045636 0.020423 0" rpy="0 0 0" />
@@ -111,4 +120,7 @@
       </collision>
     </link>
+    <gazebo reference="${prefix}left_finger_prox_link">
+      <material>Gazebo/Black</material>
+    </gazebo>
     <joint name="${prefix}left_finger_bottom_joint" type="revolute">
       <origin xyz="0 0.0305 0.070003" rpy="0 1.5708 0" />
@@ -141,4 +153,7 @@
       </collision>
     </link>
+    <gazebo reference="${prefix}left_finger_dist_link">
+      <material>Kortex/Blue</material>
+    </gazebo>
     <joint name="${prefix}left_finger_tip_joint" type="revolute">
       <origin xyz="-0.045636 -0.020423 6.9901E-05" rpy="0 0 0" />

Commit message: Corrected colours and put them in RViz too

File: kortex_description/arms/gen3_lite/6dof/urdf/gen3_lite_macro.xacro (robot description, xacro)
@@ -16,5 +16,5 @@
         </geometry>
         <material name="">
-          <color rgba="0.75294 0.75294 0.75294 1" />
+          <color rgba="0.803 0.824 0.820 1" />
         </material>
       </visual>
@@ -41,5 +41,5 @@
         </geometry>
         <material name="">
-          <color rgba="0.75294 0.75294 0.75294 1" />
+          <color rgba="0.803 0.824 0.820 1" />
         </material>
       </visual>
@@ -73,5 +73,5 @@
         </geometry>
         <material name="">
-          <color rgba="0.75294 0.75294 0.75294 1" />
+          <color rgba="0.803 0.824 0.820 1" />
         </material>
       </visual>
@@ -105,5 +105,5 @@
         </geometry>
         <material name="">
-          <color rgba="0.75294 0.75294 0.75294 1" />
+          <color rgba="0.803 0.824 0.820 1" />
         </material>
       </visual>
@@ -137,5 +137,5 @@
         </geometry>
         <material name="">
-          <color rgba="0.75294 0.75294 0.75294 1" />
+          <color rgba="0.803 0.824 0.820 1" />
         </material>
       </visual>
@@ -169,5 +169,5 @@
         </geometry>
         <material name="">
-          <color rgba="0.75294 0.75294 0.75294 1" />
+          <color rgba="0.803 0.824 0.820 1" />
         </material>
       </visual>

File: kortex_description/grippers/gen3_lite_2f/urdf/gen3_lite_2f_macro.xacro (robot description, xacro)
@@ -20,5 +20,5 @@
         </geometry>
         <material name="">
-          <color rgba="0.75294 0.75294 0.75294 1" />
+          <color rgba="0.803 0.824 0.820 1" />
         </material>
       </visual>
@@ -45,5 +45,5 @@
       </geometry>
       <material name="">
-          <color rgba="0.75294 0.75294 0.75294 1" />
+          <color rgba="0.803 0.824 0.820 1" />
       </material>
     </visual>
@@ -56,5 +56,5 @@
     </link>
     <gazebo reference="${prefix}right_finger_prox_link">
-      <material>Gazebo/Black</material>
+      <material>Kortex/Gray</material>
     </gazebo>
     <joint name="${prefix}right_finger_bottom_joint" type="revolute">
@@ -77,5 +77,5 @@
         </geometry>
         <material name="">
-          <color rgba="0.75294 0.75294 0.75294 1" />
+          <color rgba="0 0.055 0.525 1" />
         </material>
       </visual>
@@ -110,5 +110,5 @@
         </geometry>
         <material name="">
-          <color rgba="0.75294 0.75294 0.75294 1" />
+          <color rgba="0.803 0.824 0.820 1" />
         </material>
       </visual>
@@ -121,5 +121,5 @@
     </link>
     <gazebo reference="${prefix}left_finger_prox_link">
-      <material>Gazebo/Black</material>
+      <material>Kortex/Gray</material>
     </gazebo>
     <joint name="${prefix}left_finger_bottom_joint" type="revolute">
@@ -143,5 +143,5 @@
         </geometry>
         <material name="">
-          <color rgba="0.75294 0.75294 0.75294 1" />
+          <color rgba="0 0.055 0.525 1" />
         </material>
       </visual>

Commit message: Add colours to Gen3 lite simulation (#93)
* Add custom colours for Gen3 lite simulation - more realistic textures to come later

* Corrected colours and put them in RViz too

File: kortex_description/arms/gen3_lite/6dof/urdf/gen3_lite_macro.xacro (robot description, xacro)
@@ -16,5 +16,5 @@
         </geometry>
         <material name="">
-          <color rgba="0.75294 0.75294 0.75294 1" />
+          <color rgba="0.803 0.824 0.820 1" />
         </material>
       </visual>
@@ -26,4 +26,7 @@
       </collision>
     </link>
+    <gazebo reference="${prefix}base_link">
+      <material>Kortex/Gray</material>
+    </gazebo>
     <link name="${prefix}shoulder_link">
       <inertial>
@@ -38,5 +41,5 @@
         </geometry>
         <material name="">
-          <color rgba="0.75294 0.75294 0.75294 1" />
+          <color rgba="0.803 0.824 0.820 1" />
         </material>
       </visual>
@@ -48,4 +51,7 @@
       </collision>
     </link>
+    <gazebo reference="${prefix}shoulder_link">
+      <material>Kortex/Gray</material>
+    </gazebo>
     <joint name="${prefix}joint_1" type="revolute">
       <origin xyz="0 0 0.12825" rpy="0 0 0" />
@@ -67,5 +73,5 @@
         </geometry>
         <material name="">
-          <color rgba="0.75294 0.75294 0.75294 1" />
+          <color rgba="0.803 0.824 0.820 1" />
         </material>
       </visual>
@@ -77,4 +83,7 @@
       </collision>
     </link>
+    <gazebo reference="${prefix}arm_link">
+      <material>Kortex/Gray</material>
+    </gazebo>
     <joint name="${prefix}joint_2" type="revolute">
       <origin xyz="0 -0.03 0.115" rpy="1.5708 0 0" />
@@ -96,5 +105,5 @@
         </geometry>
         <material name="">
-          <color rgba="0.75294 0.75294 0.75294 1" />
+          <color rgba="0.803 0.824 0.820 1" />
         </material>
       </visual>
@@ -106,4 +115,7 @@
       </collision>
     </link>
+    <gazebo reference="${prefix}forearm_link">
+      <material>Kortex/Gray</material>
+    </gazebo>
     <joint name="${prefix}joint_3" type="revolute">
       <origin xyz="0 0.28 0" rpy="-3.1416 0 0" />
@@ -125,5 +137,5 @@
         </geometry>
         <material name="">
-          <color rgba="0.75294 0.75294 0.75294 1" />
+          <color rgba="0.803 0.824 0.820 1" />
         </material>
       </visual>
@@ -135,4 +147,7 @@
       </collision>
     </link>
+    <gazebo reference="${prefix}lower_wrist_link">
+      <material>Kortex/Gray</material>
+    </gazebo>
     <joint name="${prefix}joint_4" type="revolute">
       <origin xyz="0 -0.14 0.02" rpy="1.5708 0 0" />
@@ -154,5 +169,5 @@
         </geometry>
         <material name="">
-          <color rgba="0.75294 0.75294 0.75294 1" />
+          <color rgba="0.803 0.824 0.820 1" />
         </material>
       </visual>
@@ -164,4 +179,7 @@
       </collision>
     </link>
+    <gazebo reference="${prefix}upper_wrist_link">
+      <material>Kortex/Gray</material>
+    </gazebo>
     <joint name="${prefix}joint_5" type="revolute">
       <origin xyz="0.0285 0 0.105" rpy="0 1.5708 0" />

File: kortex_description/grippers/gen3_lite_2f/urdf/gen3_lite_2f_macro.xacro (robot description, xacro)
@@ -20,5 +20,5 @@
         </geometry>
         <material name="">
-          <color rgba="0.75294 0.75294 0.75294 1" />
+          <color rgba="0.803 0.824 0.820 1" />
         </material>
       </visual>
@@ -30,4 +30,7 @@
       </collision>
     </link>
+    <gazebo reference="${prefix}gripper_base_link">
+      <material>Kortex/Gray</material>
+    </gazebo>
     <link name="${prefix}right_finger_prox_link">
     <inertial>
@@ -42,5 +45,5 @@
       </geometry>
       <material name="">
-          <color rgba="0.75294 0.75294 0.75294 1" />
+          <color rgba="0.803 0.824 0.820 1" />
       </material>
     </visual>
@@ -52,4 +55,7 @@
     </collision>
     </link>
+    <gazebo reference="${prefix}right_finger_prox_link">
+      <material>Kortex/Gray</material>
+    </gazebo>
     <joint name="${prefix}right_finger_bottom_joint" type="revolute">
       <origin xyz="0 -0.030501 0.070003" rpy="0 1.5708 0" />
@@ -71,5 +77,5 @@
         </geometry>
         <material name="">
-          <color rgba="0.75294 0.75294 0.75294 1" />
+          <color rgba="0 0.055 0.525 1" />
         </material>
       </visual>
@@ -81,4 +87,7 @@
       </collision>
     </link>
+    <gazebo reference="${prefix}right_finger_dist_link">
+      <material>Kortex/Blue</material>
+    </gazebo>
     <joint name="${prefix}right_finger_tip_joint" type="revolute">
       <origin xyz="-0.045636 0.020423 0" rpy="0 0 0" />
@@ -101,5 +110,5 @@
         </geometry>
         <material name="">
-          <color rgba="0.75294 0.75294 0.75294 1" />
+          <color rgba="0.803 0.824 0.820 1" />
         </material>
       </visual>
@@ -111,4 +120,7 @@
       </collision>
     </link>
+    <gazebo reference="${prefix}left_finger_prox_link">
+      <material>Kortex/Gray</material>
+    </gazebo>
     <joint name="${prefix}left_finger_bottom_joint" type="revolute">
       <origin xyz="0 0.0305 0.070003" rpy="0 1.5708 0" />
@@ -131,5 +143,5 @@
         </geometry>
         <material name="">
-          <color rgba="0.75294 0.75294 0.75294 1" />
+          <color rgba="0 0.055 0.525 1" />
         </material>
       </visual>
@@ -141,4 +153,7 @@
       </collision>
     </link>
+    <gazebo reference="${prefix}left_finger_dist_link">
+      <material>Kortex/Blue</material>
+    </gazebo>
     <joint name="${prefix}left_finger_tip_joint" type="revolute">
       <origin xyz="-0.045636 -0.020423 6.9901E-05" rpy="0 0 0" />
