Commit message: Update GEN3-LITE.urdf

File: kortex_description/arms/gen3_lite/6dof/urdf/GEN3-LITE.urdf (robot description, URDF)
Before this commit: robot KR7108-URDF, 8 links, 7 joints
Links:
- link ARM: geometry collision mesh filename=/Users/juniortchapdieu/Desktop/CubeSat Simulation/ros_korte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; visual mesh filename=/Users/juniortchapdieu/Desktop/CubeSat Simulation/ros_korte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
- link BASE: geometry collision mesh filename=/Users/juniortchapdieu/Desktop/CubeSat Simulation/ros_korte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; visual mesh filename=/Users/juniortchapdieu/Desktop/CubeSat Simulation/ros_korte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
- link FOREARM: geometry collision mesh filename=/Users/juniortchapdieu/Desktop/CubeSat Simulation/ros_korte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; visual mesh filename=/Users/juniortchapdieu/Desktop/CubeSat Simulation/ros_korte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
- link LOWER_WRIST: geometry collision mesh filename=/Users/juniortchapdieu/Desktop/CubeSat Simulation/ros_korte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; visual mesh filename=/Users/juniortchapdieu/Desktop/CubeSat Simulation/ros_korte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
- link SHOULDER: geometry collision mesh filename=/Users/juniortchapdieu/Desktop/CubeSat Simulation/ros_korte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; visual mesh filename=/Users/juniortchapdieu/Desktop/CubeSat Simulation/ros_korte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
- link UPPER_WRIST: geometry collision mesh filename=/Users/juniortchapdieu/Desktop/CubeSat Simulation/ros_korte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; visual mesh filename=/Users/juniortchapdieu/Desktop/CubeSat Simulation/ros_korte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
