Commit message: Added tool_frame's for every gripper

File: kortex_description/grippers/gen3_lite_2f/urdf/gen3_lite_2f_macro.xacro (robot description, xacro)
@@ -2,4 +2,13 @@
 <robot name="gen3_lite_2f_gripper" xmlns:xacro="http://ros.org/wiki/xacro">
   <xacro:macro name="load_gripper" params="parent prefix">
+    <!-- Tool frame used by the arm -->
+    <link name="${prefix}tool_frame"/>
+    <joint name="${prefix}tool_frame_joint" type="fixed">
+        <origin xyz="0 0 0.130" rpy="0 0 1.57079632679" />
+        <parent link="${parent}" />
+        <child link="${prefix}tool_frame" />
+        <axis xyz="0 0 0" />
+    </joint>
+    <!-- Gripper description -->
     <joint name="${prefix}gripper_base_joint" type="fixed">
       <origin xyz="0 0 0" rpy="0 0 0" />

File: kortex_description/grippers/robotiq_2f_140/urdf/robotiq_arg2f_140_model_macro.xacro (robot description, xacro)
@@ -203,4 +203,13 @@
   </xacro:macro>
   <xacro:macro name="robotiq_arg2f_140" params="parent prefix">
+    <!-- Tool frame used by the arm -->
+    <link name="${prefix}tool_frame"/>
+    <joint name="${prefix}tool_frame_joint" type="fixed">
+        <origin xyz="0 0 0.20" rpy="0 0 0" />
+        <parent link="${parent}" />
+        <child link="${prefix}tool_frame" />
+        <axis xyz="0 0 0" />
+    </joint>
+    <!-- Gripper description -->
     <xacro:robotiq_arg2f_base_link prefix="${prefix}" parent="${parent}"/>
     <xacro:finger_links prefix="${prefix}" fingerprefix="left" stroke="140"/>

File: kortex_description/grippers/robotiq_2f_85/urdf/robotiq_arg2f_85_model_macro.xacro (robot description, xacro)
@@ -183,4 +183,13 @@
   <!-- Initialization of all joints and links -->
   <xacro:macro name="robotiq_arg2f_85" params="prefix parent">
+    <!-- Tool frame used by the arm -->
+    <link name="${prefix}tool_frame"/>
+    <joint name="${prefix}tool_frame_joint" type="fixed">
+        <origin xyz="0 0 0.120" rpy="0 0 0" />
+        <parent link="${parent}" />
+        <child link="${prefix}tool_frame" />
+        <axis xyz="0 0 0" />
+    </joint>
+    <!-- Gripper description -->
     <xacro:robotiq_arg2f_base_link prefix="${prefix}" parent="${parent}"/>
     <xacro:finger_links prefix="${prefix}" fingerprefix="left" stroke="85"/>

File: kortex_description/robots/kortex_robot.xacro (robot description, xacro)
@@ -34,4 +34,14 @@
             <xacro:load_gripper parent="${prefix}${last_arm_link}"  prefix="${prefix}"/>
         </xacro:unless>
+        <!-- If no gripper, define tool frame here -->
+        <xacro:if value="${not gripper}">
+            <link name="${prefix}tool_frame"/>
+            <joint name="${prefix}tool_frame_joint" type="fixed">
+                <origin xyz="0 0 0" rpy="0 0 0" />
+                <parent link="${prefix}${last_arm_link}" />
+                <child link="${prefix}tool_frame" />
+                <axis xyz="0 0 0" />
+            </joint>
+        </xacro:if>
         <!-- Load the Gazebo transmissions and gazebo_ros_control plugin -->
         <xacro:if value="${sim}">
