Commit message: Change description and control files to support prefix option

File: kortex_description/grippers/gen3_lite_2f/urdf/gen3_lite_2f_transmission_macro.xacro (robot description, xacro)
@@ -2,10 +2,10 @@
 <robot xmlns:xacro="http://ros.org/wiki/xacro">
     <xacro:macro name="load_gazebo_gripper_transmissions" params="prefix">
-        <transmission name="right_finger_bottom_trans">
+        <transmission name="${prefix}right_finger_bottom_trans">
             <type>transmission_interface/SimpleTransmission</type>
-            <joint name="right_finger_bottom_joint">
+            <joint name="${prefix}right_finger_bottom_joint">
                 <hardwareInterface>hardware_interface/PositionJointInterface</hardwareInterface>
             </joint>
-            <actuator name="right_finger_bottom_motor">
+            <actuator name="${prefix}right_finger_bottom_motor">
                 <mechanicalReduction>1</mechanicalReduction>
                 <hardwareInterface>hardware_interface/PositionJointInterface</hardwareInterface>
@@ -14,6 +14,6 @@
         <gazebo>
             <plugin filename="libroboticsgroup_gazebo_mimic_joint_plugin.so" name="mimic_gen3_lite_2f_1">
-                <joint>right_finger_bottom_joint</joint>
-                <mimicJoint>right_finger_tip_joint</mimicJoint>
+                <joint>${prefix}right_finger_bottom_joint</joint>
+                <mimicJoint>${prefix}right_finger_tip_joint</mimicJoint>
                 <multiplier>-0.676</multiplier>
                 <offset>0.149</offset>
@@ -22,6 +22,6 @@
             </plugin>
             <plugin filename="libroboticsgroup_gazebo_mimic_joint_plugin.so" name="mimic_gen3_lite_2f_2">
-                <joint>right_finger_bottom_joint</joint>
-                <mimicJoint>left_finger_bottom_joint</mimicJoint>
+                <joint>${prefix}right_finger_bottom_joint</joint>
+                <mimicJoint>${prefix}left_finger_bottom_joint</mimicJoint>
                 <multiplier>-1.0</multiplier>
                 <offset>0.0</offset>
@@ -30,6 +30,6 @@
             </plugin>
             <plugin filename="libroboticsgroup_gazebo_mimic_joint_plugin.so" name="mimic_gen3_lite_2f_3">
-                <joint>right_finger_bottom_joint</joint>
-                <mimicJoint>left_finger_tip_joint</mimicJoint>
+                <joint>${prefix}right_finger_bottom_joint</joint>
+                <mimicJoint>${prefix}left_finger_tip_joint</mimicJoint>
                 <multiplier>-0.676</multiplier>
                 <offset>0.149</offset>
@@ -40,7 +40,7 @@
                 <arm>
                     <arm_name>my_gen3_lite_gripper</arm_name>
-                    <palm_link>end_effector_link</palm_link> <!-- Gazebo merges links connected by fixed joints, so here we would have put gripper_base_link but it is merged with Bracelet_Link internally -->
-                    <gripper_link> right_finger_dist_link </gripper_link>
-                    <gripper_link> left_finger_dist_link </gripper_link>
+                    <palm_link>${prefix}end_effector_link</palm_link> <!-- Gazebo merges links connected by fixed joints, so here we would have put gripper_base_link but it is merged with Bracelet_Link internally -->
+                    <gripper_link> ${prefix}right_finger_dist_link </gripper_link>
+                    <gripper_link> ${prefix}left_finger_dist_link </gripper_link>
                 </arm>
                 <forces_angle_tolerance>100</forces_angle_tolerance>

File: kortex_description/grippers/robotiq_2f_140/urdf/robotiq_2f_140_transmission_macro.xacro (robot description, xacro)
@@ -2,10 +2,10 @@
 <robot xmlns:xacro="http://ros.org/wiki/xacro">
   <xacro:macro name="load_gazebo_gripper_transmissions" params="prefix">
-        <transmission name="finger_joint_trans">
+        <transmission name="${prefix}finger_joint_trans">
             <type>transmission_interface/SimpleTransmission</type>
-            <joint name="finger_joint">
+            <joint name="${prefix}finger_joint">
                 <hardwareInterface>hardware_interface/PositionJointInterface</hardwareInterface>
             </joint>
-            <actuator name="finger_joint_motor">
+            <actuator name="${prefix}finger_joint_motor">
                 <mechanicalReduction>1</mechanicalReduction>
                 <hardwareInterface>hardware_interface/PositionJointInterface</hardwareInterface>
@@ -14,6 +14,6 @@
         <gazebo>
             <plugin filename="libroboticsgroup_gazebo_mimic_joint_plugin.so" name="mimic_robotiq_140_1">
-                <joint>finger_joint</joint>
-                <mimicJoint>right_outer_knuckle_joint</mimicJoint>
+                <joint>${prefix}finger_joint</joint>
+                <mimicJoint>${prefix}right_outer_knuckle_joint</mimicJoint>
                 <multiplier>-1.0</multiplier>
                 <offset>0.0</offset>
@@ -22,6 +22,6 @@
             </plugin>
             <plugin filename="libroboticsgroup_gazebo_mimic_joint_plugin.so" name="mimic_robotiq_140_2">
-                <joint>finger_joint</joint>
-                <mimicJoint>right_inner_knuckle_joint</mimicJoint>
+                <joint>${prefix}finger_joint</joint>
+                <mimicJoint>${prefix}right_inner_knuckle_joint</mimicJoint>
                 <multiplier>-1.0</multiplier>
                 <offset>0.0</offset>
@@ -30,6 +30,6 @@
             </plugin>
             <plugin filename="libroboticsgroup_gazebo_mimic_joint_plugin.so" name="mimic_robotiq_140_3">
-                <joint>finger_joint</joint>
-                <mimicJoint>left_inner_knuckle_joint</mimicJoint>
+                <joint>${prefix}finger_joint</joint>
+                <mimicJoint>${prefix}left_inner_knuckle_joint</mimicJoint>
                 <multiplier>-1.0</multiplier>
                 <offset>0.0</offset>
@@ -38,6 +38,6 @@
             </plugin>
             <plugin filename="libroboticsgroup_gazebo_mimic_joint_plugin.so" name="mimic_robotiq_140_4">
-                <joint>finger_joint</joint>
-                <mimicJoint>left_inner_finger_joint</mimicJoint>
+                <joint>${prefix}finger_joint</joint>
+                <mimicJoint>${prefix}left_inner_finger_joint</mimicJoint>
                 <multiplier>1.0</multiplier>
                 <offset>0.0</offset>
@@ -46,6 +46,6 @@
             </plugin>
             <plugin filename="libroboticsgroup_gazebo_mimic_joint_plugin.so" name="mimic_robotiq_140_5">
-                <joint>finger_joint</joint>
-                <mimicJoint>right_inner_finger_joint</mimicJoint>
+                <joint>${prefix}finger_joint</joint>
+                <mimicJoint>${prefix}right_inner_finger_joint</mimicJoint>
                 <multiplier>1.0</multiplier>
                 <offset>0.0</offset>
@@ -56,7 +56,7 @@
                 <arm>
                     <arm_name>my_robotiq_gripper</arm_name>
-                    <palm_link>bracelet_link</palm_link> <!-- Gazebo merges links connected by fixed joints, so here we would have put gripper_base_link but it is merged with Bracelet_Link internally -->
-                    <gripper_link> left_inner_finger </gripper_link>
-                    <gripper_link> right_inner_finger </gripper_link>
+                    <palm_link>${prefix}bracelet_link</palm_link> <!-- Gazebo merges links connected by fixed joints, so here we would have put gripper_base_link but it is merged with Bracelet_Link internally -->
+                    <gripper_link> ${prefix}left_inner_finger </gripper_link>
+                    <gripper_link> ${prefix}right_inner_finger </gripper_link>
                 </arm>
                 <forces_angle_tolerance>100</forces_angle_tolerance>

File: kortex_description/grippers/robotiq_2f_85/urdf/robotiq_2f_85_transmission_macro.xacro (robot description, xacro)
@@ -2,10 +2,10 @@
 <robot xmlns:xacro="http://ros.org/wiki/xacro">
   <xacro:macro name="load_gazebo_gripper_transmissions" params="prefix">
-        <transmission name="finger_joint_trans">
+        <transmission name="${prefix}finger_joint_trans">
             <type>transmission_interface/SimpleTransmission</type>
-            <joint name="finger_joint">
+            <joint name="${prefix}finger_joint">
                 <hardwareInterface>hardware_interface/PositionJointInterface</hardwareInterface>
             </joint>
-            <actuator name="finger_joint_motor">
+            <actuator name="${prefix}finger_joint_motor">
                 <mechanicalReduction>1</mechanicalReduction>
                 <hardwareInterface>hardware_interface/PositionJointInterface</hardwareInterface>
@@ -14,6 +14,6 @@
         <gazebo>
             <plugin filename="libroboticsgroup_gazebo_mimic_joint_plugin.so" name="mimic_robotiq_85_1">
-                <joint>finger_joint</joint>
-                <mimicJoint>right_outer_knuckle_joint</mimicJoint>
+                <joint>${prefix}finger_joint</joint>
+                <mimicJoint>${prefix}right_outer_knuckle_joint</mimicJoint>
                 <multiplier>1.0</multiplier>
                 <offset>0.0</offset>
@@ -22,6 +22,6 @@
             </plugin>
             <plugin filename="libroboticsgroup_gazebo_mimic_joint_plugin.so" name="mimic_robotiq_85_2">
-                <joint>finger_joint</joint>
-                <mimicJoint>right_inner_knuckle_joint</mimicJoint>
+                <joint>${prefix}finger_joint</joint>
+                <mimicJoint>${prefix}right_inner_knuckle_joint</mimicJoint>
                 <multiplier>1.0</multiplier>
                 <offset>0.0</offset>
@@ -30,6 +30,6 @@
             </plugin>
             <plugin filename="libroboticsgroup_gazebo_mimic_joint_plugin.so" name="mimic_robotiq_85_3">
-                <joint>finger_joint</joint>
-                <mimicJoint>left_inner_knuckle_joint</mimicJoint>
+                <joint>${prefix}finger_joint</joint>
+                <mimicJoint>${prefix}left_inner_knuckle_joint</mimicJoint>
                 <multiplier>1.0</multiplier>
                 <offset>0.0</offset>
@@ -38,6 +38,6 @@
             </plugin>
             <plugin filename="libroboticsgroup_gazebo_mimic_joint_plugin.so" name="mimic_robotiq_85_4">
-                <joint>finger_joint</joint>
-                <mimicJoint>left_inner_finger_joint</mimicJoint>
+                <joint>${prefix}finger_joint</joint>
+                <mimicJoint>${prefix}left_inner_finger_joint</mimicJoint>
                 <multiplier>-1.0</multiplier>
                 <offset>0.0</offset>
@@ -46,6 +46,6 @@
             </plugin>
             <plugin filename="libroboticsgroup_gazebo_mimic_joint_plugin.so" name="mimic_robotiq_85_5">
-                <joint>finger_joint</joint>
-                <mimicJoint>right_inner_finger_joint</mimicJoint>
+                <joint>${prefix}finger_joint</joint>
+                <mimicJoint>${prefix}right_inner_finger_joint</mimicJoint>
                 <multiplier>-1.0</multiplier>
                 <offset>0.0</offset>
@@ -56,7 +56,7 @@
                 <arm>
                     <arm_name>my_robotiq_gripper</arm_name>
-                    <palm_link>bracelet_link</palm_link> <!-- Gazebo merges links connected by fixed joints, so here we would have put gripper_base_link but it is merged with Bracelet_Link internally -->
-                    <gripper_link> left_inner_finger </gripper_link>
-                    <gripper_link> right_inner_finger </gripper_link>
+                    <palm_link>${prefix}bracelet_link</palm_link> <!-- Gazebo merges links connected by fixed joints, so here we would have put gripper_base_link but it is merged with Bracelet_Link internally -->
+                    <gripper_link> ${prefix}left_inner_finger </gripper_link>
+                    <gripper_link> ${prefix}right_inner_finger </gripper_link>
                 </arm>
                 <forces_angle_tolerance>100</forces_angle_tolerance>
