Commit message: Adjust colors for the Robotiq 140 model

File: kortex_description/grippers/robotiq_2f_140/urdf/robotiq_arg2f_140_model_macro.xacro (robot description, xacro)
@@ -30,4 +30,12 @@
       </collision>
     </link>
+    <gazebo reference="${prefix}${fingerprefix}_outer_knuckle">
+      <visual>
+        <material>
+          <ambient>0.792156862745098 0.819607843137255 0.933333333333333 1</ambient>
+          <diffuse>0.792156862745098 0.819607843137255 0.933333333333333 1</diffuse>
+        </material>
+      </visual>
+    </gazebo>
   </xacro:macro>
   <xacro:macro name="outer_finger" params="prefix fingerprefix stroke">
@@ -60,4 +68,7 @@
       </collision>
     </link>
+    <gazebo reference="${prefix}${fingerprefix}_outer_finger">
+      <material>Gazebo/Black</material>
+    </gazebo>
   </xacro:macro>
   <xacro:macro name="inner_knuckle" params="prefix fingerprefix stroke">
@@ -90,4 +101,7 @@
       </collision>
     </link>
+    <gazebo reference="${prefix}${fingerprefix}_inner_knuckle">
+      <material>Gazebo/Black</material>
+    </gazebo>
   </xacro:macro>
   <xacro:macro name="inner_finger" params="prefix fingerprefix stroke">
@@ -120,4 +134,7 @@
       </collision>
     </link>
+    <gazebo reference="${prefix}${fingerprefix}_inner_finger">
+      <material>Gazebo/Black</material>
+    </gazebo>
   </xacro:macro>
   <!-- Finger pad link, the default are the "big pads" with rubber-->

Commit message: Tool frame (#97)
* Added tool_frame's for every gripper

* Add tool_frame to MoveIt arm planning group and a small description of the frame

File: kortex_description/grippers/robotiq_2f_140/urdf/robotiq_arg2f_140_model_macro.xacro (robot description, xacro)
@@ -220,4 +220,13 @@
   </xacro:macro>
   <xacro:macro name="robotiq_arg2f_140" params="parent prefix">
+    <!-- Tool frame used by the arm -->
+    <link name="${prefix}tool_frame"/>
+    <joint name="${prefix}tool_frame_joint" type="fixed">
+        <origin xyz="0 0 0.20" rpy="0 0 0" />
+        <parent link="${parent}" />
+        <child link="${prefix}tool_frame" />
+        <axis xyz="0 0 0" />
+    </joint>
+    <!-- Gripper description -->
     <xacro:robotiq_arg2f_base_link prefix="${prefix}" parent="${parent}"/>
     <xacro:finger_links prefix="${prefix}" fingerprefix="left" stroke="140"/>
