Commit message: Fix MoveIt config Gen3 lite home position

File: kortex_move_it_config/gen3_lite_gen3_lite_2f_move_it_config/config/gen3_lite_gen3_lite_2f.srdf.xacro (robot description, xacro)
@@ -32,8 +32,8 @@
         <joint name="$(arg prefix)joint_1" value="0" />
         <joint name="$(arg prefix)joint_2" value="-0.28" />
-        <joint name="$(arg prefix)joint_3" value="1.33" />
+        <joint name="$(arg prefix)joint_3" value="1.309" />
         <joint name="$(arg prefix)joint_4" value="0" />
         <joint name="$(arg prefix)joint_5" value="-1.047" />
-        <joint name="$(arg prefix)joint_6" value="2.67" />
+        <joint name="$(arg prefix)joint_6" value="0" />
     </group_state>
     <group_state name="retract" group="arm">
