Commit message: Add description and moveit configs for release 2.2

File: kortex_description/arms/gen3/7dof/urdf/gen3_macro.xacro (robot description, xacro)
@@ -60,5 +60,5 @@
       <limit
         effort="39"
-        velocity="0.8727" />
+        velocity="1.3963" />
     </joint>
     <link name="${prefix}half_arm_1_link">
@@ -94,5 +94,5 @@
       <axis
         xyz="0 0 1" />
-      <limit lower="-2.41" upper="2.41" effort="39" velocity="0.8727" />
+      <limit lower="-2.41" upper="2.41" effort="39" velocity="1.3963" />
     </joint>
     <link name="${prefix}half_arm_2_link">
@@ -130,5 +130,5 @@
       <limit
         effort="39"
-        velocity="0.8727" />
+        velocity="1.3963" />
     </joint>
     <link name="${prefix}forearm_link">
@@ -164,5 +164,5 @@
       <axis
         xyz="0 0 1" />
-      <limit lower="-2.66" upper="2.66" effort="39" velocity="0.8727" />
+      <limit lower="-2.66" upper="2.66" effort="39" velocity="1.3963" />
     </joint>
     <link name="${prefix}spherical_wrist_1_link">
@@ -200,5 +200,5 @@
       <limit
         effort="9"
-        velocity="0.8727" />
+        velocity="1.2218" />
     </joint>
     <link name="${prefix}spherical_wrist_2_link">
@@ -234,28 +234,54 @@
       <axis
         xyz="0 0 1" />
-      <limit lower="-2.23" upper="2.23" effort="9" velocity="0.8727" />
-    </joint>
+      <limit lower="-2.23" upper="2.23" effort="9" velocity="1.2218" />
+    </joint>
+    <xacro:if value="${vision}">
     <link name="${prefix}bracelet_link">
       <inertial>
-        <origin xyz="-0.000281 -0.011402 -0.029798" rpy="0 0 0" />
-        <mass value="0.5006" />
-        <inertia ixx="0.000587" ixy="3E-06" ixz="3E-06" iyy="0.000369" iyz="0.000118" izz="0.000609" />
-      </inertial>
-      <visual>
-        <origin xyz="0 0 0" rpy="0 0 0" />
-        <geometry>
-          <mesh filename="package://kortex_description/arms/gen3/${dof}dof/meshes/bracelet_link.STL" />
-        </geometry>
-        <material name="">
-          <color rgba="0.75294 0.75294 0.75294 1" />
-        </material>
-      </visual>
-      <collision>
-        <origin xyz="0 0 0" rpy="0 0 0" />
-        <geometry>
-          <mesh filename="package://kortex_description/arms/gen3/${dof}dof/meshes/bracelet_link.STL" />
-        </geometry>
-      </collision>
-    </link>
+        <origin xyz="0.000281 0.011402 -0.029798" rpy="0 0 0" />
+        <mass value="0.5" />
+        <inertia ixx="0.000587" ixy="3E-06" ixz="3E-06" iyy="0.000369" iyz="-0.000118" izz="0.000609" />
+      </inertial>
+      <visual>
+        <origin xyz="0 0 0" rpy="0 0 0" />
+        <geometry>
+          <mesh filename="package://kortex_description/arms/gen3/${dof}dof/meshes/bracelet_with_vision_link.STL" />
+        </geometry>
+        <material name="">
+          <color rgba="0.75294 0.75294 0.75294 1" />
+        </material>
+      </visual>
+      <collision>
+        <origin xyz="0 0 0" rpy="0 0 0" />
+        <geometry>
+          <mesh filename="package://kortex_description/arms/gen3/${dof}dof/meshes/bracelet_with_vision_link.STL" />
+        </geometry>
+      </collision>
+    </link>
+    </xacro:if>
+    <xacro:unless value="${vision}">
+    <link name="${prefix}bracelet_link">
+      <inertial>
+        <origin xyz="-9.3E-05 0.000132 -0.022905" rpy="0 0 0" />
+        <mass value="0.364" />
+        <inertia ixx="0.000214" ixy="0" ixz="1E-06" iyy="0.000223" iyz="-2E-06" izz="0.00024" />
+      </inertial>
+      <visual>
+        <origin xyz="0 0 0" rpy="0 0 0" />
+        <geometry>
+          <mesh filename="package://kortex_description/arms/gen3/${dof}dof/meshes/bracelet_no_vision_link.STL" />
+        </geometry>
+        <material name="">
+          <color rgba="0.75294 0.75294 0.75294 1" />
+        </material>
+      </visual>
+      <collision>
+        <origin xyz="0 0 0" rpy="0 0 0" />
+        <geometry>
+          <mesh filename="package://kortex_description/arms/gen3/${dof}dof/meshes/bracelet_no_vision_link.STL" />
+        </geometry>
+      </collision>
+    </link>
+    </xacro:unless>
     <joint
       name="${prefix}joint_7"
@@ -270,5 +296,5 @@
       <limit
         effort="9"
-        velocity="0.8727" />
+        velocity="1.2218" />
     </joint>
     <link name="${prefix}end_effector_link" />

File: kortex_description/grippers/gen3_lite_2f/urdf/gen3_lite_2f_macro.xacro (robot description, xacro)
@@ -31,24 +31,24 @@
     </link>
     <link name="${prefix}right_finger_prox_link">
-      <inertial>
-        <origin xyz="0.020257 0.0063483 6.991E-05" rpy="0 0 0" />
-        <mass value="0.018385" />
-        <inertia ixx="2.29E-06" ixy="1.43E-06" ixz="0" iyy="4.56E-06" iyz="0" izz="4.77E-06" />
-      </inertial>
-      <visual>
-        <origin xyz="0 0 0" rpy="0 0 0" />
-        <geometry>
-          <mesh filename="package://kortex_description/grippers/gen3_lite_2f/meshes/right_finger_prox_link.STL" />
-        </geometry>
-        <material name="">
-            <color rgba="0.75294 0.75294 0.75294 1" />
-        </material>
-      </visual>
-      <collision>
-        <origin xyz="0 0 0" rpy="0 0 0" />
-        <geometry>
-          <mesh filename="package://kortex_description/grippers/gen3_lite_2f/meshes/right_finger_prox_link.STL" />
-        </geometry>
-      </collision>
+    <inertial>
+      <origin xyz="0.020257 0.0063483 6.991E-05" rpy="0 0 0" />
+      <mass value="0.018385" />
+      <inertia ixx="2.29E-06" ixy="1.43E-06" ixz="0" iyy="4.56E-06" iyz="0" izz="4.77E-06" />
+    </inertial>
+    <visual>
+      <origin xyz="0 0 0" rpy="0 0 0" />
+      <geometry>
+        <mesh filename="package://kortex_description/grippers/gen3_lite_2f/meshes/right_finger_prox_link.STL" />
+      </geometry>
+      <material name="">
+          <color rgba="0.75294 0.75294 0.75294 1" />
+      </material>
+    </visual>
+    <collision>
+      <origin xyz="0 0 0" rpy="0 0 0" />
+      <geometry>
+        <mesh filename="package://kortex_description/grippers/gen3_lite_2f/meshes/right_finger_prox_link.STL" />
+      </geometry>
+    </collision>
     </link>
     <joint name="${prefix}right_finger_bottom_joint" type="revolute">

File: kortex_description/grippers/gen3_lite_2f/urdf/gen3_lite_2f_transmission_macro.xacro (robot description, xacro)
@@ -2,10 +2,10 @@
 <robot xmlns:xacro="http://ros.org/wiki/xacro">
     <xacro:macro name="load_gazebo_gripper_transmissions" params="prefix">
-        <transmission name="${prefix}right_finger_bottom_trans">
+        <transmission name="right_finger_bottom_trans">
             <type>transmission_interface/SimpleTransmission</type>
-            <joint name="${prefix}right_finger_bottom_joint">
+            <joint name="right_finger_bottom_joint">
                 <hardwareInterface>hardware_interface/PositionJointInterface</hardwareInterface>
             </joint>
-            <actuator name="${prefix}right_finger_bottom_motor">
+            <actuator name="right_finger_bottom_motor">
                 <mechanicalReduction>1</mechanicalReduction>
                 <hardwareInterface>hardware_interface/PositionJointInterface</hardwareInterface>
@@ -14,6 +14,6 @@
         <gazebo>
             <plugin filename="libroboticsgroup_gazebo_mimic_joint_plugin.so" name="mimic_gen3_lite_2f_1">
-                <joint>${prefix}right_finger_bottom_joint</joint>
-                <mimicJoint>${prefix}right_finger_tip_joint</mimicJoint>
+                <joint>right_finger_bottom_joint</joint>
+                <mimicJoint>right_finger_tip_joint</mimicJoint>
                 <multiplier>-0.676</multiplier>
                 <offset>0.149</offset>
@@ -22,6 +22,6 @@
             </plugin>
             <plugin filename="libroboticsgroup_gazebo_mimic_joint_plugin.so" name="mimic_gen3_lite_2f_2">
-                <joint>${prefix}right_finger_bottom_joint</joint>
-                <mimicJoint>${prefix}left_finger_bottom_joint</mimicJoint>
+                <joint>right_finger_bottom_joint</joint>
+                <mimicJoint>left_finger_bottom_joint</mimicJoint>
                 <multiplier>-1.0</multiplier>
                 <offset>0.0</offset>
@@ -30,6 +30,6 @@
             </plugin>
             <plugin filename="libroboticsgroup_gazebo_mimic_joint_plugin.so" name="mimic_gen3_lite_2f_3">
-                <joint>${prefix}right_finger_bottom_joint</joint>
-                <mimicJoint>${prefix}left_finger_tip_joint</mimicJoint>
+                <joint>right_finger_bottom_joint</joint>
+                <mimicJoint>left_finger_tip_joint</mimicJoint>
                 <multiplier>-0.676</multiplier>
                 <offset>0.149</offset>
@@ -39,8 +39,8 @@
             <plugin name="gazebo_grasp_fix" filename="libgazebo_grasp_fix.so">
                 <arm>
-                    <arm_name>${prefix}my_gen3_lite_gripper</arm_name>
-                    <palm_link>${prefix}end_effector_link</palm_link> <!-- Gazebo merges links connected by fixed joints, so here we would have put gripper_base_link but it is merged with Bracelet_Link internally -->
-                    <gripper_link> ${prefix}right_finger_dist_link </gripper_link>
-                    <gripper_link> ${prefix}left_finger_dist_link </gripper_link>
+                    <arm_name>my_gen3_lite_gripper</arm_name>
+                    <palm_link>end_effector_link</palm_link> <!-- Gazebo merges links connected by fixed joints, so here we would have put gripper_base_link but it is merged with Bracelet_Link internally -->
+                    <gripper_link> right_finger_dist_link </gripper_link>
+                    <gripper_link> left_finger_dist_link </gripper_link>
                 </arm>
                 <forces_angle_tolerance>100</forces_angle_tolerance>
