Commit message: Add description and moveit configs for release 2.2

File: kortex_description/grippers/robotiq_2f_85/urdf/robotiq_2f_85_macro.xacro (robot description, xacro)
@@ -1,302 +1,7 @@
 <?xml version="1.0"?>
-<robot name="robotiq_85_gripper" xmlns:xacro="http://ros.org/wiki/xacro">
-    <xacro:property name="M_PI" value="3.14159"/>
-    <xacro:macro name="load_gripper" params="parent prefix">
-        <joint name="${prefix}gripper_base_joint" type="fixed">
-            <parent link="${parent}"/>
-            <child link="${prefix}gripper_base_link"/>
-            <origin rpy="1.57 -1.57 0.0" xyz="0.0 0.0 0.0"/>
-        </joint>
-        <link name="${prefix}gripper_base_link">
-            <visual>
-                <geometry>
-                    <mesh filename="package://kortex_description/grippers/robotiq_2f_85/meshes/visual/robotiq_85_base_link.dae"/>
-                </geometry>
-            </visual>
-            <collision>
-                <geometry>
-                    <mesh filename="package://kortex_description/grippers/robotiq_2f_85/meshes/collision/robotiq_85_base_link.stl"/>
-                </geometry>
-            </collision>
-            <inertial>
-                <mass value="0.636951" />
-                <origin xyz="0.0 0.0 0.0" />
-                <inertia ixx = "0.000380" ixy = "0.000000" ixz = "0.000000"
-                         iyx = "0.000000" iyy = "0.001110" iyz = "0.000000"
-                         izx = "0.000000" izy = "0.000000" izz = "0.001171" />
-            </inertial>
-        </link>
-        <gazebo reference="${prefix}gripper_base_link">
-            <implicitSpringDamper>1</implicitSpringDamper>
-            <mu1>100000</mu1>
-            <mu2>100000</mu2>
-            <kp>100000000.0</kp>
-            <kd>1.0</kd>
-        </gazebo>
-        <joint name="${prefix}gripper_finger1_joint" type="revolute">
-            <parent link="${prefix}gripper_base_link"/>
-            <child link="${prefix}gripper_finger1_knuckle_link"/>
-            <axis xyz="0 0 1"/>
-            <origin rpy="${M_PI} 0.0 0.0" xyz="0.05490451627 0.03060114443 0.0"/>
-            <limit lower="0.0" upper="0.804" velocity="2.0" effort="1000"/>
-        </joint>
-        <joint name="${prefix}gripper_finger2_joint" type="revolute">
-            <parent link="${prefix}gripper_base_link"/>
-            <child link="${prefix}gripper_finger2_knuckle_link"/>
-            <axis xyz="0 0 1"/>
-            <origin rpy="0.0 0.0 0.0" xyz="0.05490451627 -0.03060114443 0.0"/>
-            <limit lower="0.0" upper="0.804" velocity="2.0" effort="1000"/>
-            <mimic joint="${prefix}gripper_finger1_joint"/>
-        </joint>
-        <link name="${prefix}gripper_finger1_knuckle_link">
-            <visual>
-                <geometry>
-                    <mesh filename="package://kortex_description/grippers/robotiq_2f_85/meshes/visual/robotiq_85_knuckle_link.dae"/>
-                </geometry>
-            </visual>
-            <collision>
-                <geometry>
-                    <mesh filename="package://kortex_description/grippers/robotiq_2f_85/meshes/collision/robotiq_85_knuckle_link.stl"/>
-                </geometry>
-            </collision>
-            <inertial>
-                <mass value="0.018491" />
-                <origin xyz="0.0 0.0 0.0" />
-                <inertia ixx = "0.000009" ixy = "-0.000001" ixz = "0.000000"
-                         iyx = "-0.000001" iyy = "0.000001" iyz = "0.000000"
-                         izx = "0.000000" izy = "0.000000" izz = "0.000010" />
-            </inertial>
-        </link>
-        <gazebo reference="${prefix}gripper_finger1_knuckle_link">
-            <implicitSpringDamper>1</implicitSpringDamper>
-            <mu1>100000</mu1>
-            <mu2>100000</mu2>
-            <kp>100000000.0</kp>
-            <kd>1.0</kd>
-        </gazebo>
-        <link name="${prefix}gripper_finger2_knuckle_link">
-            <visual>
-                <geometry>
-                    <mesh filename="package://kortex_description/grippers/robotiq_2f_85/meshes/visual/robotiq_85_knuckle_link.dae"/>
-                </geometry>
-            </visual>
-            <collision>
-                <geometry>
-                    <mesh filename="package://kortex_description/grippers/robotiq_2f_85/meshes/collision/robotiq_85_knuckle_link.stl"/>
-                </geometry>
-            </collision>
-            <inertial>
-                <mass value="0.018491" />
-                <origin xyz="0.0 0.0 0.0" />
-                <inertia ixx = "0.000009" ixy = "-0.000001" ixz = "0.000000"
-                         iyx = "-0.000001" iyy = "0.000001" iyz = "0.000000"
-                         izx = "0.000000" izy = "0.000000" izz = "0.000010" />
-            </inertial>
-        </link>
-        <gazebo reference="${prefix}gripper_finger2_knuckle_link">
-            <implicitSpringDamper>1</implicitSpringDamper>
-            <mu1>100000</mu1>
-            <mu2>100000</mu2>
-            <kp>100000000.0</kp>
-            <kd>1.0</kd>
-        </gazebo>
-        <joint name="${prefix}gripper_finger1_finger_joint" type="fixed">
-            <parent link="${prefix}gripper_finger1_knuckle_link"/>
-            <child link="${prefix}gripper_finger1_finger_link"/>
-            <origin xyz="-0.00408552455 -0.03148604435 0.0" rpy="0 0 0" />
-        </joint>
-        <joint name="${prefix}gripper_finger2_finger_joint" type="fixed">
-            <parent link="${prefix}gripper_finger2_knuckle_link"/>
-            <child link="${prefix}gripper_finger2_finger_link"/>
-            <origin xyz="-0.00408552455 -0.03148604435 0.0" rpy="0 0 0" />
-        </joint>
-        <link name="${prefix}gripper_finger1_finger_link">
-            <visual>
-                <geometry>
-                    <mesh filename="package://kortex_description/grippers/robotiq_2f_85/meshes/visual/robotiq_85_finger_link.dae"/>
-                </geometry>
-            </visual>
-            <collision>
-                <geometry>
-                    <mesh filename="package://kortex_description/grippers/robotiq_2f_85/meshes/collision/robotiq_85_finger_link.stl"/>
-                </geometry>
-            </collision>
-            <inertial>
-                <mass value="0.027309" />
-                <origin xyz="0.0 0.0 0.0" />
-                <inertia ixx = "0.000003" ixy = "-0.000002" ixz = "0.000000"
-                         iyx = "-0.000002" iyy = "0.000021" iyz = "0.000000"
-                         izx = "0.000000" izy = "0.000000" izz = "0.000020" />
-            </inertial>
-        </link>
-        <gazebo reference="${prefix}gripper_finger1_finger_link">
-            <implicitSpringDamper>1</implicitSpringDamper>
-            <mu1>100000</mu1>
-            <mu2>100000</mu2>
-            <kp>100000000.0</kp>
-            <kd>1.0</kd>
-        </gazebo>
-        <link name="${prefix}gripper_finger2_finger_link">
-            <visual>
-                <geometry>
-                    <mesh filename="package://kortex_description/grippers/robotiq_2f_85/meshes/visual/robotiq_85_finger_link.dae"/>
-                </geometry>
-            </visual>
-            <collision>
-                <geometry>
-                    <mesh filename="package://kortex_description/grippers/robotiq_2f_85/meshes/collision/robotiq_85_finger_link.stl"/>
-                </geometry>
-            </collision>
-            <inertial>
-                <mass value="0.027309" />
-                <origin xyz="0.0 0.0 0.0" />
-                <inertia ixx = "0.000003" ixy = "-0.000002" ixz = "0.000000"
-                         iyx = "-0.000002" iyy = "0.000021" iyz = "0.000000"
-                         izx = "0.000000" izy = "0.000000" izz = "0.000020" />
-            </inertial>
-        </link>
-        <gazebo reference="${prefix}gripper_finger2_finger_link">
-            <implicitSpringDamper>1</implicitSpringDamper>
-            <mu1>100000</mu1>
-            <mu2>100000</mu2>
-            <kp>100000000.0</kp>
-            <kd>1.0</kd>
-        </gazebo>
-        <joint name="${prefix}gripper_finger1_inner_knuckle_joint" type="continuous">
-            <parent link="${prefix}gripper_base_link"/>
-            <child link="${prefix}gripper_finger1_inner_knuckle_link"/>
-            <axis xyz="0 0 1"/>
-            <origin xyz="0.06142 0.0127 0" rpy="${M_PI} 0.0 0.0" />
-            <limit lower="0.0" upper="0.804" velocity="2.0" effort="0.1"/>
-            <mimic joint="${prefix}gripper_finger1_joint" offset="0"/>
-        </joint>
-        <joint name="${prefix}gripper_finger2_inner_knuckle_joint" type="continuous">
-            <parent link="${prefix}gripper_base_link"/>
-            <child link="${prefix}gripper_finger2_inner_knuckle_link"/>
-            <axis xyz="0 0 1"/>
-            <origin xyz="0.06142 -0.0127 0" rpy="0 0 0"/>
-            <limit lower="0.0" upper="0.804" velocity="2.0" effort="0.1"/>
-            <mimic joint="${prefix}gripper_finger1_joint" offset="0"/>
-        </joint>
-        <link name="${prefix}gripper_finger1_inner_knuckle_link">
-            <visual>
-                <geometry>
-                    <mesh filename="package://kortex_description/grippers/robotiq_2f_85/meshes/visual/robotiq_85_inner_knuckle_link.dae"/>
-                </geometry>
-            </visual>
-            <collision>
-                <geometry>
-                    <mesh filename="package://kortex_description/grippers/robotiq_2f_85/meshes/collision/robotiq_85_inner_knuckle_link.stl"/>
-                </geometry>
-            </collision>
-            <inertial>
-                <mass value="0.029951" />
-                <origin xyz="0.0 0.0 0.0" />
-                <inertia ixx = "0.000039" ixy = "0.000000" ixz = "0.000000"
-                         iyx = "0.000000" iyy = "0.000005" iyz = "0.000000"
-                         izx = "0.000000" izy = "0.000000" izz = "0.000035" />
-            </inertial>
-        </link>
-        <gazebo reference="${prefix}gripper_finger1_inner_knuckle_link">
-            <implicitSpringDamper>1</implicitSpringDamper>
-            <mu1>100000</mu1>
-            <mu2>100000</mu2>
-            <kp>100000000.0</kp>
-            <kd>1.0</kd>
-        </gazebo>
-        <link name="${prefix}gripper_finger2_inner_knuckle_link">
-            <visual>
-                <geometry>
-                    <mesh filename="package://kortex_description/grippers/robotiq_2f_85/meshes/visual/robotiq_85_inner_knuckle_link.dae"/>
-                </geometry>
-            </visual>
-            <collision>
-                <geometry>
-                    <mesh filename="package://kortex_description/grippers/robotiq_2f_85/meshes/collision/robotiq_85_inner_knuckle_link.stl"/>
-                </geometry>
-            </collision>
-            <inertial>
-                <mass value="0.029951" />
-                <origin xyz="0.0 0.0 0.0" />
-                <inertia ixx = "0.000039" ixy = "0.000000" ixz = "0.000000"
-                         iyx = "0.000000" iyy = "0.000005" iyz = "0.000000"
-                         izx = "0.000000" izy = "0.000000" izz = "0.000035" />
-            </inertial>
-        </link>
-        <gazebo reference="${prefix}gripper_finger2_inner_knuckle_link">
-            <implicitSpringDamper>1</implicitSpringDamper>
-            <mu1>100000</mu1>
-            <mu2>100000</mu2>
-            <kp>100000000.0</kp>
-            <kd>1.0</kd>
-        </gazebo>
-        <joint name="${prefix}gripper_finger1_finger_tip_joint" type="continuous">
-            <parent link="${prefix}gripper_finger1_inner_knuckle_link"/>
-            <child link="${prefix}gripper_finger1_finger_tip_link"/>
-            <axis xyz="0 0 1"/>
-            <origin xyz="0.04303959807 -0.03759940821 0.0" rpy="0.0 0.0 0.0"/>
-            <limit lower="0.0" upper="0.804" velocity="2.0" effort="0.1"/>
-            <mimic joint="${prefix}gripper_finger1_joint" multiplier="-1"/>
-        </joint>
-        <joint name="${prefix}gripper_finger2_finger_tip_joint" type="continuous">
-            <parent link="${prefix}gripper_finger2_inner_knuckle_link"/>
-            <child link="${prefix}gripper_finger2_finger_tip_link"/>
-            <axis xyz="0 0 1"/>
-            <origin rpy="0.0 0.0 0.0" xyz="0.04303959807 -0.03759940821  0.0"/>
-            <limit lower="0.0" upper="0.804" velocity="2.0" effort="0.1"/>
-            <mimic joint="${prefix}gripper_finger1_joint" multiplier="-1"/>
-        </joint>
-        <link name="${prefix}gripper_finger1_finger_tip_link">
-            <visual>
-                <geometry>
-                    <mesh filename="package://kortex_description/grippers/robotiq_2f_85/meshes/visual/robotiq_85_finger_tip_link.dae"/>
-                </geometry>
-            </visual>
-            <collision>
-                <geometry>
-                    <mesh filename="package://kortex_description/grippers/robotiq_2f_85/meshes/collision/robotiq_85_finger_tip_link.stl"/>
-                </geometry>
-            </collision>
-            <inertial>
-                <mass value="0.019555" />
-                <origin xyz="0.0 0.0 0.0" />
-                <inertia ixx = "0.000002" ixy = "0.000000" ixz = "0.000000"
-                         iyx = "0.000000" iyy = "0.000005" iyz = "0.000000"
-                         izx = "0.000000" izy = "0.000000" izz = "0.000006" />
-            </inertial>
-        </link>
-        <gazebo reference="${prefix}gripper_finger1_finger_tip_link">
-            <implicitSpringDamper>1</implicitSpringDamper>
-            <mu1>100000</mu1>
-            <mu2>100000</mu2>
-            <kp>100000000.0</kp>
-            <kd>1.0</kd>
-        </gazebo>
-        <link name="${prefix}gripper_finger2_finger_tip_link">
-            <visual>
-                <geometry>
-                    <mesh filename="package://kortex_description/grippers/robotiq_2f_85/meshes/visual/robotiq_85_finger_tip_link.dae"/>
-                </geometry>
-            </visual>
-            <collision>
-                <geometry>
-                    <mesh filename="package://kortex_description/grippers/robotiq_2f_85/meshes/collision/robotiq_85_finger_tip_link.stl"/>
-                </geometry>
-            </collision>
-            <inertial>
-                <mass value="0.019555" />
-                <origin xyz="0.0 0.0 0.0" />
-                <inertia ixx = "0.000002" ixy = "0.000000" ixz = "0.000000"
-                         iyx = "0.000000" iyy = "0.000005" iyz = "0.000000"
-                         izx = "0.000000" izy = "0.000000" izz = "0.000006" />
-            </inertial>
-        </link>
-        <gazebo reference="${prefix}gripper_finger2_finger_tip_link">
-            <implicitSpringDamper>1</implicitSpringDamper>
-            <mu1>100000</mu1>
-            <mu2>100000</mu2>
-            <kp>100000000.0</kp>
-            <kd>1.0</kd>
-        </gazebo>
-    </xacro:macro>
+<robot name="robotiq_arg2f_85_model" xmlns:xacro="http://ros.org/wiki/xacro">
+  <xacro:macro name="load_gripper" params="parent prefix">
+    <xacro:include filename="$(find kortex_description)/grippers/robotiq_2f_85/urdf/robotiq_arg2f_85_model_macro.xacro" />
+    <xacro:robotiq_arg2f_85 parent="${parent}" prefix="${prefix}"/>
+  </xacro:macro>
 </robot>

File: kortex_description/grippers/robotiq_2f_85/urdf/robotiq_2f_85_transmission_macro.xacro (robot description, xacro)
@@ -2,10 +2,10 @@
 <robot xmlns:xacro="http://ros.org/wiki/xacro">
   <xacro:macro name="load_gazebo_gripper_transmissions" params="prefix">
-        <transmission name="${prefix}gripper_finger1_trans">
+        <transmission name="finger_joint_trans">
             <type>transmission_interface/SimpleTransmission</type>
-            <joint name="${prefix}gripper_finger1_joint">
+            <joint name="finger_joint">
                 <hardwareInterface>hardware_interface/PositionJointInterface</hardwareInterface>
             </joint>
-            <actuator name="${prefix}gripper_finger1_motor">
+            <actuator name="finger_joint_motor">
                 <mechanicalReduction>1</mechanicalReduction>
                 <hardwareInterface>hardware_interface/PositionJointInterface</hardwareInterface>
@@ -14,49 +14,44 @@
         <gazebo>
             <plugin filename="libroboticsgroup_gazebo_mimic_joint_plugin.so" name="mimic_robotiq_85_1">
-                <joint>${prefix}gripper_finger1_joint</joint>
-                <mimicJoint>${prefix}gripper_finger2_joint</mimicJoint>
+                <joint>finger_joint</joint>
+                <mimicJoint>right_outer_knuckle_joint</mimicJoint>
                 <multiplier>1.0</multiplier>
                 <offset>0.0</offset>
                 <maxEffort>5.0</maxEffort>
-                <hasPID></hasPID>
             </plugin>
             <plugin filename="libroboticsgroup_gazebo_mimic_joint_plugin.so" name="mimic_robotiq_85_2">
-                <joint>${prefix}gripper_finger1_joint</joint>
-                <mimicJoint>${prefix}gripper_finger2_inner_knuckle_joint</mimicJoint>
+                <joint>finger_joint</joint>
+                <mimicJoint>right_inner_knuckle_joint</mimicJoint>
                 <multiplier>1.0</multiplier>
                 <offset>0.0</offset>
                 <maxEffort>5.0</maxEffort>
-                <hasPID></hasPID>
             </plugin>
             <plugin filename="libroboticsgroup_gazebo_mimic_joint_plugin.so" name="mimic_robotiq_85_3">
-                <joint>${prefix}gripper_finger1_joint</joint>
-                <mimicJoint>${prefix}gripper_finger1_inner_knuckle_joint</mimicJoint>
+                <joint>finger_joint</joint>
+                <mimicJoint>left_inner_knuckle_joint</mimicJoint>
                 <multiplier>1.0</multiplier>
                 <offset>0.0</offset>
                 <maxEffort>5.0</maxEffort>
-                <hasPID></hasPID>
             </plugin>
             <plugin filename="libroboticsgroup_gazebo_mimic_joint_plugin.so" name="mimic_robotiq_85_4">
-                <joint>${prefix}gripper_finger1_joint</joint>
-                <mimicJoint>${prefix}gripper_finger1_finger_tip_joint</mimicJoint>
+                <joint>finger_joint</joint>
+                <mimicJoint>left_inner_finger_joint</mimicJoint>
                 <multiplier>-1.0</multiplier>
                 <offset>0.0</offset>
                 <maxEffort>5.0</maxEffort>
-                <hasPID></hasPID>
             </plugin>
             <plugin filename="libroboticsgroup_gazebo_mimic_joint_plugin.so" name="mimic_robotiq_85_5">
-                <joint>${prefix}gripper_finger1_joint</joint>
-                <mimicJoint>${prefix}gripper_finger2_finger_tip_joint</mimicJoint>
+                <joint>finger_joint</joint>
+                <mimicJoint>right_inner_finger_joint</mimicJoint>
                 <multiplier>-1.0</multiplier>
                 <offset>0.0</offset>
                 <maxEffort>5.0</maxEffort>
-                <hasPID></hasPID>
             </plugin>
             <plugin name="gazebo_grasp_fix" filename="libgazebo_grasp_fix.so">
                 <arm>
                     <arm_name>my_robotiq_gripper</arm_name>
-                    <palm_link>${prefix}bracelet_link</palm_link> <!-- Gazebo merges links connected by fixed joints, so here we would have put gripper_base_link but it is merged with Bracelet_Link internally -->
-                    <gripper_link> ${prefix}gripper_finger1_finger_tip_link </gripper_link>
-                    <gripper_link> ${prefix}gripper_finger2_finger_tip_link </gripper_link>
+                    <palm_link>bracelet_link</palm_link> <!-- Gazebo merges links connected by fixed joints, so here we would have put gripper_base_link but it is merged with Bracelet_Link internally -->
+                    <gripper_link> left_inner_finger </gripper_link>
+                    <gripper_link> right_inner_finger </gripper_link>
                 </arm>
                 <forces_angle_tolerance>100</forces_angle_tolerance>

File: kortex_description/robots/kortex_robot.xacro (robot description, xacro)
@@ -20,5 +20,5 @@
             <link name="world" />
             <joint name="world_to_root" type="fixed">
-                <child link="base_link" />
+                <child link="${prefix}base_link" />
                 <parent link="world" />
                 <origin xyz="0 0 0" rpy="0 0 0" />

Commit message: Added camera frames to gen3-7dof description so the vision module can work correctly

File: kortex_description/arms/gen3/7dof/urdf/gen3_macro.xacro (robot description, xacro)
@@ -310,4 +310,24 @@
         xyz="0 0 0" />
     </joint>
+    <xacro:if value="${vision}">
+      <link name="${prefix}camera_link" />
+      <joint name="${prefix}camera_module" type="fixed">
+        <origin xyz="0 0.05639 -0.00305" rpy="3.14159265358979 3.14159265358979 0" />
+        <parent link="${prefix}end_effector_link" />
+        <child  link="${prefix}camera_link" />
+      </joint>
+      <link name="${prefix}camera_depth_frame" />
+      <joint name="${prefix}depth_module" type="fixed">
+        <origin xyz="0.0275 0.066 -0.00305" rpy="3.14159265358979 3.14159265358979 0" />
+        <parent link="${prefix}end_effector_link" />
+        <child  link="${prefix}camera_depth_frame" />
+      </joint>
+      <link name="${prefix}camera_color_frame" />
+      <joint name="${prefix}color_module" type="fixed">
+        <origin xyz="0 0.05639 -0.00305" rpy="3.14159265358979 3.14159265358979 0" />
+        <parent link="${prefix}end_effector_link" />
+        <child  link="${prefix}camera_color_frame" />
+      </joint>
+    </xacro:if>
   </xacro:macro>
 </robot>
