Commit message: add: simulated depth camera to gen3 moveit gazebo simulation

File: kortex_description/arms/gen3/7dof/urdf/gen3_macro.xacro (robot description, xacro)
@@ -3,5 +3,5 @@
   <!-- Propagate last link name information because it is the gripper's parent link -->
   <xacro:property name="last_arm_link" value="end_effector_link"/>
-  <xacro:macro name="load_arm" params="parent:='' dof vision prefix *origin">
+  <xacro:macro name="load_arm" params="parent:='' dof vision prefix *origin namespace">
       <link name="${prefix}base_link">
         <inertial>
@@ -329,4 +329,18 @@
         <child  link="${prefix}camera_color_frame" />
       </joint>
+      <xacro:if value="${sim}">
+        <link name="${prefix}sim_camera_depth_frame" />
+        <joint name="${prefix}sim_depth_module" type="fixed">
+          <origin xyz="0.0275 0.066 -0.00305" rpy="${pi/2} ${-pi/2} ${-pi/2}" />
+          <parent link="${prefix}end_effector_link" />
+          <child  link="${prefix}sim_camera_depth_frame" />
+        </joint>
+        <link name="${namespace}/${prefix}camera_depth_optical_frame" />
+        <joint name="${prefix}optical_module" type="fixed">
+          <origin xyz="0.0 0.0 0.0" rpy="${-pi/2} 0.0 ${-pi/2}" />
+          <parent link="${prefix}sim_camera_depth_frame" />
+          <child  link="${namespace}/${prefix}camera_depth_optical_frame" />
+        </joint>
+      </xacro:if>
     </xacro:if>
   </xacro:macro>

File: kortex_description/robots/gen3_robotiq_2f_85.xacro (robot description, xacro)
@@ -8,5 +8,6 @@
     <xacro:arg name="sim" default="false" />
     <xacro:arg name="prefix" default="" />
+    <xacro:arg name="namespace" default="" />
     <xacro:include filename="$(find kortex_description)/robots/kortex_robot.xacro" />
-    <xacro:load_robot arm="$(arg arm)" gripper="$(arg gripper)" dof="$(arg dof)" vision="$(arg vision)" sim="$(arg sim)" prefix="$(arg prefix)" />
+    <xacro:load_robot arm="$(arg arm)" gripper="$(arg gripper)" dof="$(arg dof)" vision="$(arg vision)" sim="$(arg sim)" prefix="$(arg prefix)" namespace="$(arg namespace)"/>
 </robot>

File: kortex_description/robots/kortex_robot.xacro (robot description, xacro)
@@ -1,5 +1,5 @@
 <?xml version="1.0"?>
 <robot xmlns:xacro="http://ros.org/wiki/xacro">
-    <xacro:macro name="load_robot" params="arm gripper dof vision sim prefix">
+    <xacro:macro name="load_robot" params="arm gripper dof vision sim prefix namespace">
         <!-- Files to include -->
         <xacro:include filename="$(find kortex_description)/arms/${arm}/${dof}dof/urdf/${arm}_macro.xacro" />
@@ -10,4 +10,5 @@
             <!-- Arm transmission elements-->
             <xacro:include filename="$(find kortex_description)/arms/${arm}/${dof}dof/urdf/${arm}_transmission_macro.xacro" />
+            <xacro:include filename="$(find kortex_description)/robots/gazebo_depth_camera.xacro" />
             <!-- Gripper transmission elements if there is a gripper-->
             <xacro:unless value="${not gripper}">
@@ -26,5 +27,5 @@
         </xacro:if>
         <!-- Load the arm -->
-        <xacro:load_arm parent="" dof="${dof}" vision="${vision}" prefix="${prefix}">
+        <xacro:load_arm parent="" dof="${dof}" vision="${vision}" prefix="${prefix}" namespace="${namespace}">
             <origin xyz="0 0 0" rpy="0 0 0"/>
         </xacro:load_arm>
@@ -47,4 +48,5 @@
         <xacro:if value="${sim}">
             <xacro:load_gazebo_arm_transmissions prefix="${prefix}"/>
+            <xacro:gazebo_depth_camera prefix="${prefix}"/>
             <xacro:unless value="${not gripper}">
                 <xacro:load_gazebo_gripper_transmissions prefix="${prefix}"/>
