Commit message: Fix invalid meshes paths.

File: kortex_description/arms/gen3/7dof/urdf/GEN3_URDF_V12.urdf (robot description, URDF)
Before this commit: robot GEN3_URDF_V12, 9 links, 8 joints
Links:
- link Bracelet_Link: geometry collision mesh filename=package://kortex_description/arms/gen3/7dof/meshes/bracelet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; visual mesh filename=package://kortex_description/arms/gen3/7dof/meshes/bracelet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
- link ForeArm_Link: geometry collision mesh filename=package://kortex_description/arms/gen3/7dof/meshes/forearm_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; visual mesh filename=package://kortex_description/arms/gen3/7dof/meshes/forearm_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
- link HalfArm1_Link: geometry collision mesh filename=package://kortex_description/arms/gen3/7dof/meshes/half_arm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; visual mesh filename=package://kortex_description/arms/gen3/7dof/meshes/half_arm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
- link HalfArm2_Link: geometry collision mesh filename=package://kortex_description/arms/gen3/7dof/meshes/half_arm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; visual mesh filename=package://kortex_description/arms/gen3/7dof/meshes/half_arm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
- link Shoulder_Link: geometry collision mesh filename=package://kortex_description/arms/gen3/7dof/meshes/shoulder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; visual mesh filename=package://kortex_description/arms/gen3/7dof/meshes/shoulder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
- link SphericalWrist1_Link: geometry collision mesh filename=package://kortex_description/arms/gen3/7dof/meshes/spherica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; visual mesh filename=package://kortex_description/arms/gen3/7dof/meshes/spherica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
- link SphericalWrist2_Link: geometry collision mesh filename=package://kortex_description/arms/gen3/7dof/meshes/spherica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; visual mesh filename=package://kortex_description/arms/gen3/7dof/meshes/spherica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
- link base_link: geometry collision mesh filename=package://kortex_description/arms/gen3/7dof/meshes/base_lin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; visual mesh filename=package://kortex_description/arms/gen3/7dof/meshes/base_lin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
