Commit message: edit: launch and xacro files for launching gazebo simulations, add: more arguments for simulation and workstation, namespace argument for simulated workstation camera functionality, add simulated gazebo depth camera to gen3 urdf for working perception in gazebo

File: kortex_description/robots/gen3.xacro (robot description, xacro)
@@ -8,5 +8,7 @@
     <xacro:arg name="sim" default="false" />
     <xacro:arg name="prefix" default="" />
+    <xacro:arg name="namespace" default="" />
+    <xacro:arg name="workstation" default="false" />
     <xacro:include filename="$(find kortex_description)/robots/kortex_robot.xacro" />
-    <xacro:load_robot arm="$(arg arm)" gripper="$(arg gripper)" dof="$(arg dof)" vision="$(arg vision)" sim="$(arg sim)" prefix="$(arg prefix)" />
+    <xacro:load_robot arm="$(arg arm)" gripper="$(arg gripper)" dof="$(arg dof)" vision="$(arg vision)" sim="$(arg sim)" prefix="$(arg prefix)" namespace="$(arg namespace)" workstation="$(arg workstation)"/>
 </robot>

File: kortex_description/robots/gen3_lite_gen3_lite_2f.xacro (robot description, xacro)
@@ -9,5 +9,7 @@
     <xacro:arg name="sim" default="false" />
     <xacro:arg name="prefix" default="" />
+    <xacro:arg name="namespace" default="" />
+    <xacro:arg name="workstation" default="false" />
     <xacro:include filename="$(find kortex_description)/robots/kortex_robot.xacro" />
-    <xacro:load_robot arm="$(arg arm)" gripper="$(arg gripper)" dof="$(arg dof)" vision="false" sim="$(arg sim)"  prefix="$(arg prefix)" />
+    <xacro:load_robot arm="$(arg arm)" gripper="$(arg gripper)" dof="$(arg dof)" vision="false" sim="$(arg sim)"  prefix="$(arg prefix)" namespace="$(arg namespace)" workstation="$(arg workstation)"/>
 </robot>

File: kortex_description/robots/gen3_robotiq_2f_140.xacro (robot description, xacro)
@@ -8,5 +8,7 @@
     <xacro:arg name="sim" default="false" />
     <xacro:arg name="prefix" default="" />
+    <xacro:arg name="namespace" default="" />
+    <xacro:arg name="workstation" default="false" />
     <xacro:include filename="$(find kortex_description)/robots/kortex_robot.xacro" />
-    <xacro:load_robot arm="$(arg arm)" gripper="$(arg gripper)" dof="$(arg dof)" vision="$(arg vision)" sim="$(arg sim)" prefix="$(arg prefix)"/>
+    <xacro:load_robot arm="$(arg arm)" gripper="$(arg gripper)" dof="$(arg dof)" vision="$(arg vision)" sim="$(arg sim)" prefix="$(arg prefix)" namespace="$(arg namespace)" workstation="$(arg workstation)"/>
 </robot>

File: kortex_description/robots/gen3_robotiq_2f_85.xacro (robot description, xacro)
@@ -9,5 +9,6 @@
     <xacro:arg name="prefix" default="" />
     <xacro:arg name="namespace" default="" />
+    <xacro:arg name="workstation" default="false" />
     <xacro:include filename="$(find kortex_description)/robots/kortex_robot.xacro" />
-    <xacro:load_robot arm="$(arg arm)" gripper="$(arg gripper)" dof="$(arg dof)" vision="$(arg vision)" sim="$(arg sim)" prefix="$(arg prefix)" namespace="$(arg namespace)"/>
+    <xacro:load_robot arm="$(arg arm)" gripper="$(arg gripper)" dof="$(arg dof)" vision="$(arg vision)" sim="$(arg sim)" prefix="$(arg prefix)" namespace="$(arg namespace)" workstation="$(arg workstation)"/>
 </robot>

File: kortex_description/robots/kortex_robot.xacro (robot description, xacro)
@@ -1,5 +1,5 @@
 <?xml version="1.0"?>
 <robot xmlns:xacro="http://ros.org/wiki/xacro">
-    <xacro:macro name="load_robot" params="arm gripper dof vision sim prefix namespace">
+    <xacro:macro name="load_robot" params="arm gripper dof vision sim prefix namespace workstation">
         <!-- Files to include -->
         <xacro:include filename="$(find kortex_description)/arms/${arm}/${dof}dof/urdf/${arm}_macro.xacro" />
@@ -15,14 +15,32 @@
                 <xacro:include filename="$(find kortex_description)/grippers/${gripper}/urdf/${gripper}_transmission_macro.xacro" />
             </xacro:unless>
+            <xacro:if value="${workstation}">
+		  <xacro:include filename="$(find uml_hri_nerve_armada_workstation)/workstation_description/workstation_model.urdf.xacro" />
+            </xacro:if>
         </xacro:if>
         <!-- Run the macros -->
         <!-- For gazebo-->
         <xacro:if value="${sim}">
-            <link name="world" />
-            <joint name="world_to_root" type="fixed">
-                <child link="${prefix}base_link" />
-                <parent link="world" />
-                <origin xyz="0 0 0" rpy="0 0 0" />
-            </joint>
+            <xacro:unless value="${workstation}">
+		<link name="world" />
+            	<joint name="world_to_root" type="fixed">
+                    <child link="${prefix}base_link" />
+                    <parent link="world" />
+                    <origin xyz="0 0 0" rpy="0 0 0" />
+                </joint>
+            </xacro:unless>
+            <xacro:if value="${workstation}">
+		<link name="world"/>
+  		<joint name="world_to_table" type="fixed">
+    		    <child link="table_base_link" />
+    		    <parent link="world" />
+    		    <origin xyz="0.0 0.0 0.41" rpy="0.0 0.0 0.0" />
+  		</joint>
+  		<joint name="table_to_root" type="fixed">
+    		    <child link="${prefix}base_link" />
+    		    <parent link="table_mounting_plate_link" />
+    		    <origin xyz="0.0 0.0 0.03625" rpy="0.0 0.0 0.0" />
+  		</joint>
+            </xacro:if>
         </xacro:if>
         <!-- Load the arm -->
@@ -57,4 +75,7 @@
                 </plugin>
             </gazebo>
+            <xacro:if value="${workstation}">
+		<xacro:workstation prefix="${prefix}table_" namespace="${namespace}"/>
+            </xacro:if>
         </xacro:if>
     </xacro:macro>
