Commit message: edit: fix mislabeled argument in spawn_kortex_robot launch file, edit: default robot positioning when spawning with workstation in kortex_robot.xacro

File: kortex_description/robots/kortex_robot.xacro (robot description, xacro)
@@ -40,5 +40,5 @@
     		    <child link="${prefix}base_link" />
     		    <parent link="table_mounting_plate_link" />
-    		    <origin xyz="0.0 0.0 0.03625" rpy="0.0 0.0 0.0" />
+    		    <origin xyz="0.0 0.0 0.03625" rpy="0.0 0.0 ${pi}" />
   		</joint>
             </xacro:if>

Commit message: edit: robot position on workspace; rotate forward

File: kortex_description/robots/kortex_robot.xacro (robot description, xacro)
@@ -40,5 +40,5 @@
     		    <child link="${prefix}base_link" />
     		    <parent link="table_mounting_plate_link" />
-    		    <origin xyz="0.0 0.0 0.03625" rpy="0.0 0.0 ${pi}" />
+    		    <origin xyz="0.0 0.0 0.03625" rpy="0.0 0.0 ${pi/2}" />
   		</joint>
             </xacro:if>

Commit message: added worker standin

File: kortex_description/robots/kortex_robot.xacro (robot description, xacro)
@@ -23,5 +23,10 @@
             <link name="world" />
             <joint name="world_to_root" type="fixed">
-                <child link="base_plate" />
+                <xacro:if value="${base}">
+                    <child link="worker_body_link" />
+                </xacro:if>
+                <xacro:if value="${not base}">
+                    <child link="base_link" />
+                </xacro:if>
                 <parent link="world" />
                 <origin xyz="0 0 0.01" rpy="0 0 0" />

File: kortex_move_it_config/gen3_robotiq_2f_85_move_it_config/config/6dof/gen3_robotiq_2f_85.srdf.xacro (robot description, xacro)
@@ -76,6 +76,4 @@
     <!--END EFFECTOR: Purpose: Represent information about an end effector.-->
     <end_effector name="gripper" parent_link="base_link" group="gripper"/>
-    <!--VIRTUAL JOINT: Purpose: this element defines a virtual joint between a robot link and an external frame of reference (considered fixed with respect to the robot)-->
-    <virtual_joint name="world" type="fixed" parent_frame="world" child_link="base_plate"/>
     <!--PASSIVE JOINT: Purpose: this element is used to mark joints that are not actuated-->
     <passive_joint name="left_inner_finger_joint"/>
@@ -85,15 +83,23 @@
     <passive_joint name="right_inner_finger_joint"/>
     <!--DISABLE COLLISIONS: By default it is assumed that any link of the robot could potentially come into collision with any other link in the robot. This tag disables collision checking between a specified pair of links. -->
-    <disable_collisions link1="base_link" link2="base_plate" reason="Adjacent"/>
     <disable_collisions link1="base_link" link2="bicep_link" reason="Never"/>
-    <disable_collisions link1="base_link" link2="chair" reason="Never"/>
+    <disable_collisions link1="base_link" link2="bio_container_link" reason="Never"/>
+    <disable_collisions link1="base_link" link2="chair_link" reason="Adjacent"/>
     <disable_collisions link1="base_link" link2="forearm_link" reason="Never"/>
+    <disable_collisions link1="base_link" link2="mast_link" reason="Never"/>
     <disable_collisions link1="base_link" link2="shoulder_link" reason="Adjacent"/>
-    <disable_collisions link1="base_plate" link2="bicep_link" reason="Never"/>
-    <disable_collisions link1="base_plate" link2="chair" reason="Adjacent"/>
-    <disable_collisions link1="base_plate" link2="shoulder_link" reason="Never"/>
+    <disable_collisions link1="base_link" link2="spool_link" reason="Never"/>
+    <disable_collisions link1="base_link" link2="worker_body_link" reason="Never"/>
+    <disable_collisions link1="bicep_link" link2="bio_container_link" reason="Never"/>
     <disable_collisions link1="bicep_link" link2="forearm_link" reason="Adjacent"/>
     <disable_collisions link1="bicep_link" link2="shoulder_link" reason="Adjacent"/>
     <disable_collisions link1="bicep_link" link2="spherical_wrist_1_link" reason="Never"/>
+    <disable_collisions link1="bicep_link" link2="spool_link" reason="Never"/>
+    <disable_collisions link1="bicep_link" link2="worker_body_link" reason="Never"/>
+    <disable_collisions link1="bio_container_link" link2="chair_link" reason="Never"/>
+    <disable_collisions link1="bio_container_link" link2="mast_link" reason="Never"/>
+    <disable_collisions link1="bio_container_link" link2="shoulder_link" reason="Never"/>
+    <disable_collisions link1="bio_container_link" link2="spool_link" reason="Never"/>
+    <disable_collisions link1="bio_container_link" link2="worker_body_link" reason="Adjacent"/>
     <disable_collisions link1="bracelet_link" link2="forearm_link" reason="Never"/>
     <disable_collisions link1="bracelet_link" link2="left_inner_finger" reason="Never"/>
@@ -110,5 +116,8 @@
     <disable_collisions link1="bracelet_link" link2="spherical_wrist_1_link" reason="Never"/>
     <disable_collisions link1="bracelet_link" link2="spherical_wrist_2_link" reason="Adjacent"/>
-    <disable_collisions link1="chair" link2="shoulder_link" reason="Never"/>
+    <disable_collisions link1="chair_link" link2="mast_link" reason="Adjacent"/>
+    <disable_collisions link1="chair_link" link2="shoulder_link" reason="Never"/>
+    <disable_collisions link1="chair_link" link2="spool_link" reason="Never"/>
+    <disable_collisions link1="chair_link" link2="worker_body_link" reason="Never"/>
     <disable_collisions link1="forearm_link" link2="left_inner_finger" reason="Never"/>
     <disable_collisions link1="forearm_link" link2="left_inner_finger_pad" reason="Never"/>
@@ -175,4 +184,7 @@
     <disable_collisions link1="left_outer_knuckle" link2="spherical_wrist_1_link" reason="Never"/>
     <disable_collisions link1="left_outer_knuckle" link2="spherical_wrist_2_link" reason="Never"/>
+    <disable_collisions link1="mast_link" link2="shoulder_link" reason="Never"/>
+    <disable_collisions link1="mast_link" link2="spool_link" reason="Adjacent"/>
+    <disable_collisions link1="mast_link" link2="worker_body_link" reason="Adjacent"/>
     <disable_collisions link1="right_inner_finger" link2="right_inner_finger_pad" reason="Adjacent"/>
     <disable_collisions link1="right_inner_finger" link2="right_inner_knuckle" reason="Default"/>
@@ -203,4 +215,7 @@
     <disable_collisions link1="robotiq_arg2f_base_link" link2="spherical_wrist_2_link" reason="Never"/>
     <disable_collisions link1="shoulder_link" link2="spherical_wrist_1_link" reason="Never"/>
+    <disable_collisions link1="shoulder_link" link2="spool_link" reason="Never"/>
+    <disable_collisions link1="shoulder_link" link2="worker_body_link" reason="Never"/>
     <disable_collisions link1="spherical_wrist_1_link" link2="spherical_wrist_2_link" reason="Adjacent"/>
+    <disable_collisions link1="spool_link" link2="worker_body_link" reason="Default"/>
 </robot>

File: kortex_scripts/robot_equipment/urdf/base.xacro (robot description, xacro)
@@ -2,34 +2,15 @@
 <robot xmlns:xacro="http://ros.org/wiki/xacro">
     <xacro:include filename= "$(find kortex_scripts)/robot_equipment/urdf/macros.xacro"/>
+    <xacro:include filename= "$(find kortex_scripts)/robot_equipment/urdf/properties.xacro"/>
+    <xacro:include filename= "$(find kortex_scripts)/robot_equipment/urdf/worker_simple.xacro"/>
     <xacro:macro name="chair">
-        <link name="base_plate">
-            <inertial>
-                <origin xyz="0 0 0" rpy="0 0 0" />
-                <mass value="4" />
-                <xacro:box_inertia mass="4" x="0.1" y="0.1" z="0.01" />
-            </inertial>
-            <visual>
-                <origin xyz="0 0 0" rpy="0 0 0" />
-                <geometry>
-                    <box size="0.1 0.1 0.01"/>
-                </geometry>
-                <material name="grey">
-                    <color rgba="0.75 0.75 0.75 1"/>
-                </material>
-            </visual>
-            <collision>
-                <origin xyz="0 0 0" rpy="0 0 0" />
-                <geometry>
-                    <box size="0.1 0.1 0.01"/>
-                </geometry>
-            </collision>
-        </link>
-        <joint name="base_plate_joint" type="fixed">
-            <origin xyz="0 0 0.005" rpy="0 0 0" />
-            <parent link="base_plate" />
+        <xacro:worker_simple/>
+        <joint name="chair-base_joint" type="fixed">
+            <origin xyz="0.16 0 -0.44" rpy="0 0 0" />
+            <parent link="chair_link" />
             <child link="base_link" />
             <axis xyz="0 0 0" />
         </joint>
-        <link name="chair">
+        <link name="chair_link">
             <inertial>
                 <origin xyz="0 0 0" rpy="0 0 0" />
@@ -53,10 +34,4 @@
             </collision>
         </link>
-        <joint name="chair_joint" type="fixed">
-            <origin xyz="-0.15 0 0.445" rpy="0 0 0" />
-            <parent link="base_plate" />
-            <child link="chair" />
-            <axis xyz="0 0 0" />
-        </joint>
     </xacro:macro>
 </robot>

Commit message: added mag gripper sim functionality

File: kortex_description/robots/kortex_robot.xacro (robot description, xacro)
@@ -4,4 +4,6 @@
         <!-- Files to include -->
         <xacro:include filename="$(find kortex_description)/arms/${arm}/${dof}dof/urdf/${arm}_macro.xacro" />
+        <xacro:include filename= "$(find kortex_scripts)/robot_equipment/urdf/macros.xacro"/>
+        <xacro:include filename= "$(find kortex_scripts)/robot_equipment/urdf/properties.xacro"/>
         <xacro:unless value="${not gripper}">
             <xacro:include filename="$(find kortex_description)/grippers/${gripper}/urdf/${gripper}_macro.xacro" />
@@ -44,4 +46,5 @@
         <!-- If no gripper, define tool frame here -->
         <xacro:if value="${not gripper}">
+            <xacro:include filename="$(find kortex_scripts)/robot_equipment/urdf/mag_gripper_end_effector.xacro" />
             <link name="${prefix}tool_frame"/>
             <joint name="${prefix}tool_frame_joint" type="fixed">
@@ -51,4 +54,5 @@
                 <axis xyz="0 0 0" />
             </joint>
+            <xacro:mag_gripper_end_effector/>
         </xacro:if>
         <!-- Load the Gazebo transmissions and gazebo_ros_control plugin -->

File: kortex_scripts/robot_equipment/urdf/base.xacro (robot description, xacro)
@@ -1,6 +1,4 @@
 <?xml version="1.0"?>
 <robot xmlns:xacro="http://ros.org/wiki/xacro">
-    <xacro:include filename= "$(find kortex_scripts)/robot_equipment/urdf/macros.xacro"/>
-    <xacro:include filename= "$(find kortex_scripts)/robot_equipment/urdf/properties.xacro"/>
     <xacro:include filename= "$(find ant_worker_description)/urdf/worker.urdf.xacro"/>
     <xacro:include filename= "$(find kortex_scripts)/robot_equipment/urdf/worker_mods.xacro"/>

File: kortex_scripts/robot_equipment/urdf/properties.xacro (robot description, xacro)
@@ -8,3 +8,6 @@
     <xacro:property name="bio_container_height" value="0.05"/>
     <xacro:property name="bio_container_mass" value="0.1"/>
+    <xacro:property name="mag_gripper_end_effector_mass" value="0.170"/>
+    <xacro:property name="mag_gripper_end_effector_length" value="0.0865"/>
+    <xacro:property name="mag_gripper_end_effector_radius" value="0.040"/>
 </robot>

Commit message: Added extra world option
This pull request addresses an integration problem where the created "world" link causes conflicts when simulating robotic arm placed on top of Clearpath Husky UGV on Gazebo. By introducing a new "world" parameter in the load_robot macro, with a default value of True, developers can have the flexibility to set it as False in their customized URDF files, controlling where and how to put "world" link in their own urdf files.

File: kortex_description/robots/kortex_robot.xacro (robot description, xacro)
@@ -1,5 +1,5 @@
 <?xml version="1.0"?>
 <robot xmlns:xacro="http://ros.org/wiki/xacro">
-    <xacro:macro name="load_robot" params="arm gripper dof vision sim prefix">
+    <xacro:macro name="load_robot" params="world:=True arm gripper dof vision sim prefix">
         <!-- Files to include -->
         <xacro:include filename="$(find kortex_description)/arms/${arm}/${dof}dof/urdf/${arm}_macro.xacro" />
@@ -17,5 +17,5 @@
         <!-- Run the macros -->
         <!-- For gazebo-->
-        <xacro:if value="${sim}">
+        <xacro:if value="${sim and world}">
             <link name="world" />
             <joint name="world_to_root" type="fixed">

Commit message: Updated robot xacro to facilitate flexible arm mounting on either the world link or a mobile robot base

File: kortex_description/robots/kortex_robot.xacro (robot description, xacro)
@@ -1,5 +1,5 @@
 <?xml version="1.0"?>
 <robot xmlns:xacro="http://ros.org/wiki/xacro">
-    <xacro:macro name="load_robot" params="arm gripper dof vision sim prefix">
+    <xacro:macro name="load_robot" params="arm gripper dof vision sim prefix parent_link:='world' joint_origin_xyz:='0 0 0' joint_origin_rpy:='0 0 0'">
         <!-- Files to include -->
         <xacro:include filename="$(find kortex_description)/arms/${arm}/${dof}dof/urdf/${arm}_macro.xacro" />
@@ -15,14 +15,15 @@
             </xacro:unless>
         </xacro:if>
-        <!-- Run the macros -->
-        <!-- For gazebo-->
-        <xacro:if value="${sim}">
+        <!-- Run the macros and mount the robot -->
+        <!-- For gazebo when parent_link is world -->
+        <xacro:if value="${(sim and parent_link == 'world')}">
             <link name="world" />
-            <joint name="world_to_root" type="fixed">
-                <child link="${prefix}base_link" />
-                <parent link="world" />
-                <origin xyz="0 0 0" rpy="0 0 0" />
-            </joint>
         </xacro:if>
+        <!-- Mount robot with the world or base robot -->
+        <joint name="${prefix}mount_joint" type="fixed">
+            <child link="${prefix}base_link" />
+            <parent link="${parent_link}" />
+            <origin xyz="${joint_origin_xyz}" rpy="${joint_origin_rpy}"/>
+        </joint>
         <!-- Load the arm -->
         <xacro:load_arm parent="" dof="${dof}" vision="${vision}" prefix="${prefix}">

Commit message: Rename param from joint_origin_* to origin_*

File: kortex_description/robots/kortex_robot.xacro (robot description, xacro)
@@ -1,5 +1,5 @@
 <?xml version="1.0"?>
 <robot xmlns:xacro="http://ros.org/wiki/xacro">
-    <xacro:macro name="load_robot" params="arm gripper dof vision sim prefix parent_link:='world' joint_origin_xyz:='0 0 0' joint_origin_rpy:='0 0 0'">
+    <xacro:macro name="load_robot" params="arm gripper dof vision sim prefix parent_link:='world' origin_xyz:='0 0 0' origin_rpy:='0 0 0'">
         <!-- Files to include -->
         <xacro:include filename="$(find kortex_description)/arms/${arm}/${dof}dof/urdf/${arm}_macro.xacro" />
@@ -24,5 +24,5 @@
             <child link="${prefix}base_link" />
             <parent link="${parent_link}" />
-            <origin xyz="${joint_origin_xyz}" rpy="${joint_origin_rpy}"/>
+            <origin xyz="${origin_xyz}" rpy="${origin_rpy}"/>
         </joint>
         <!-- Load the arm -->
