Commit message: resolved stash merge conflicts

File: kortex_move_it_config/gen3_robotiq_2f_85_move_it_config/config/7dof/gen3_robotiq_2f_85.srdf.xacro (robot description, xacro)
@@ -62,4 +62,31 @@
         <joint name="$(arg prefix)joint_6" value="0" />
         <joint name="$(arg prefix)joint_7" value="0" />
+    </group_state>
+    <group_state name="left_snapshot" group="arm">
+        <joint name="$(arg prefix)joint_1" value="-1.75" />
+        <joint name="$(arg prefix)joint_2" value="1.05" />
+        <joint name="$(arg prefix)joint_3" value="1.05" />
+        <joint name="$(arg prefix)joint_4" value="1.57" />
+        <joint name="$(arg prefix)joint_5" value="0" />
+        <joint name="$(arg prefix)joint_6" value="1.05" />
+        <joint name="$(arg prefix)joint_7" value="2.8" />
+    </group_state>
+    <group_state name="right_snapshot" group="arm">
+        <joint name="$(arg prefix)joint_1" value="1.75" />
+        <joint name="$(arg prefix)joint_2" value="1.05" />
+        <joint name="$(arg prefix)joint_3" value="-1.05" />
+        <joint name="$(arg prefix)joint_4" value="1.57" />
+        <joint name="$(arg prefix)joint_5" value="0" />
+        <joint name="$(arg prefix)joint_6" value="1.05" />
+        <joint name="$(arg prefix)joint_7" value="0.45" />
+    </group_state>
+    <group_state name="top_snapshot" group="arm">
+        <joint name="$(arg prefix)joint_1" value="0.043" />
+        <joint name="$(arg prefix)joint_2" value="-0.1824" />
+        <joint name="$(arg prefix)joint_3" value="-0.0133" />
+        <joint name="$(arg prefix)joint_4" value="2.208" />
+        <joint name="$(arg prefix)joint_5" value="-0.0188" />
+        <joint name="$(arg prefix)joint_6" value="0.7828" />
+        <joint name="$(arg prefix)joint_7" value="-1.524" />
     </group_state>
     <group_state name="opened" group="gripper">
