Commit message: added chair model

File: kortex_description/arms/gen3/6dof/urdf/base.xacro (robot description, xacro)
@@ -2,15 +2,15 @@
 <robot xmlns:xacro="http://ros.org/wiki/xacro">
     <xacro:include filename= "$(find kortex_description)/arms/${arm}/${dof}dof/urdf/macros.xacro"/>
-    <xacro:macro name="base_plate">
+    <xacro:macro name="chair">
         <link name="base_plate">
             <inertial>
                 <origin xyz="0 0 0" rpy="0 0 0" />
                 <mass value="4" />
-                <xacro:box_inertia mass="4" x="0.6" y="0.2" z="0.01" />
+                <xacro:box_inertia mass="4" x="0.1" y="0.1" z="0.01" />
             </inertial>
             <visual>
                 <origin xyz="0 0 0" rpy="0 0 0" />
                 <geometry>
-                    <box size="0.6 0.2 0.01"/>
+                    <box size="0.1 0.1 0.01"/>
                 </geometry>
                 <material name="grey">
@@ -21,5 +21,5 @@
                 <origin xyz="0 0 0" rpy="0 0 0" />
                 <geometry>
-                    <box size="0.6 0.2 0.01"/>
+                    <box size="0.1 0.1 0.01"/>
                 </geometry>
             </collision>
@@ -31,4 +31,32 @@
             <axis xyz="0 0 0" />
         </joint>
+        <link name="chair">
+            <inertial>
+                <origin xyz="0 0 0" rpy="0 0 0" />
+                <mass value="4" />
+                <xacro:box_inertia mass="4" x="0.1" y="0.1" z="0.9" />
+            </inertial>
+            <visual>
+                <origin xyz="-0.075 -.075 -0.45" rpy="1.57 0 1.57" />
+                <geometry>
+                    <mesh filename="package://kortex_description/arms/gen3/${dof}dof/meshes/parametric_chair.STL" />
+                </geometry>
+                <material name="grey">
+                    <color rgba="0.75 0.75 0.75 1"/>
+                </material>
+            </visual>
+            <collision>
+                <origin xyz="0 0 0" rpy="0 0 0" />
+                <geometry>
+                    <box size="0.1 0.1 0.9"/>
+                </geometry>
+            </collision>
+        </link>
+        <joint name="chair_joint" type="fixed">
+            <origin xyz="-0.15 0 0.445" rpy="0 0 0" />
+            <parent link="base_plate" />
+            <child link="chair" />
+            <axis xyz="0 0 0" />
+        </joint>
     </xacro:macro>
 </robot>

File: kortex_description/arms/gen3/6dof/urdf/gen3_macro.xacro (robot description, xacro)
@@ -28,5 +28,5 @@
     </link>
     <xacro:if value="${base}">
-      <xacro:base_plate/>
+      <xacro:chair/>
     </xacro:if>
     <link name="${prefix}shoulder_link">

File: kortex_move_it_config/gen3_robotiq_2f_85_move_it_config/config/6dof/gen3_robotiq_2f_85.srdf.xacro (robot description, xacro)
@@ -85,7 +85,12 @@
     <passive_joint name="right_inner_finger_joint"/>
     <!--DISABLE COLLISIONS: By default it is assumed that any link of the robot could potentially come into collision with any other link in the robot. This tag disables collision checking between a specified pair of links. -->
+    <disable_collisions link1="base_link" link2="base_plate" reason="Adjacent"/>
     <disable_collisions link1="base_link" link2="bicep_link" reason="Never"/>
+    <disable_collisions link1="base_link" link2="chair" reason="Never"/>
     <disable_collisions link1="base_link" link2="forearm_link" reason="Never"/>
     <disable_collisions link1="base_link" link2="shoulder_link" reason="Adjacent"/>
+    <disable_collisions link1="base_plate" link2="bicep_link" reason="Never"/>
+    <disable_collisions link1="base_plate" link2="chair" reason="Adjacent"/>
+    <disable_collisions link1="base_plate" link2="shoulder_link" reason="Never"/>
     <disable_collisions link1="bicep_link" link2="forearm_link" reason="Adjacent"/>
     <disable_collisions link1="bicep_link" link2="shoulder_link" reason="Adjacent"/>
@@ -105,4 +110,5 @@
     <disable_collisions link1="bracelet_link" link2="spherical_wrist_1_link" reason="Never"/>
     <disable_collisions link1="bracelet_link" link2="spherical_wrist_2_link" reason="Adjacent"/>
+    <disable_collisions link1="chair" link2="shoulder_link" reason="Never"/>
     <disable_collisions link1="forearm_link" link2="left_inner_finger" reason="Never"/>
     <disable_collisions link1="forearm_link" link2="left_inner_finger_pad" reason="Never"/>
