Commit message: added base plate for mounting arm

File: kortex_move_it_config/gen3_robotiq_2f_85_move_it_config/config/6dof/gen3_robotiq_2f_85.srdf.xacro (robot description, xacro)
@@ -1,9 +1,8 @@
-<?xml version="1.0" ?>
+<?xml version="1.0" encoding="UTF-8"?>
 <!--This does not replace URDF, and is not an extension of URDF.
     This is a format for representing semantic information about the robot structure.
     A URDF file must exist for this robot as well, where the joints and the links that are referenced are defined
 -->
-<robot name="gen3_robotiq_2f_85" xmlns:xacro="http://www.ros.org/wiki/xacro">
-    <xacro:arg name="prefix" default="" />
+<robot name="gen3_robotiq_2f_85">
     <!--GROUPS: Representation of a set of joints and links. This can be useful for specifying DOF to plan for, defining arms, end effectors, etc-->
     <!--LINKS: When a link is specified, the parent joint of that link (if it exists) is automatically included-->
@@ -12,188 +11,190 @@
     <!--SUBGROUPS: Groups can also be formed by referencing to already defined group names-->
     <group name="arm">
-        <joint name="$(arg prefix)joint_1" />
-        <joint name="$(arg prefix)joint_2" />
-        <joint name="$(arg prefix)joint_3" />
-        <joint name="$(arg prefix)joint_4" />
-        <joint name="$(arg prefix)joint_5" />
-        <joint name="$(arg prefix)joint_6" />
-        <joint name="$(arg prefix)end_effector" />
-        <joint name="$(arg prefix)tool_frame_joint" />
+        <joint name="joint_1"/>
+        <joint name="joint_2"/>
+        <joint name="joint_3"/>
+        <joint name="joint_4"/>
+        <joint name="joint_5"/>
+        <joint name="joint_6"/>
+        <joint name="end_effector"/>
+        <joint name="tool_frame_joint"/>
     </group>
     <group name="gripper">
-        <joint name="$(arg prefix)gripper_base_joint" />
-        <joint name="$(arg prefix)finger_joint" />
-        <joint name="$(arg prefix)left_outer_finger_joint" />
-        <joint name="$(arg prefix)left_inner_finger_joint" />
-        <joint name="$(arg prefix)left_inner_finger_pad_joint" />
-        <joint name="$(arg prefix)left_inner_knuckle_joint" />
-        <joint name="$(arg prefix)right_inner_knuckle_joint" />
-        <joint name="$(arg prefix)right_outer_knuckle_joint" />
-        <joint name="$(arg prefix)right_outer_finger_joint" />
-        <joint name="$(arg prefix)right_inner_finger_joint" />
-        <joint name="$(arg prefix)right_inner_finger_pad_joint" />
+        <joint name="gripper_base_joint"/>
+        <joint name="finger_joint"/>
+        <joint name="left_outer_finger_joint"/>
+        <joint name="left_inner_finger_joint"/>
+        <joint name="left_inner_finger_pad_joint"/>
+        <joint name="left_inner_knuckle_joint"/>
+        <joint name="right_inner_knuckle_joint"/>
+        <joint name="right_outer_knuckle_joint"/>
+        <joint name="right_outer_finger_joint"/>
+        <joint name="right_inner_finger_joint"/>
+        <joint name="right_inner_finger_pad_joint"/>
     </group>
     <!--GROUP STATES: Purpose: Define a named state for a particular group, in terms of joint values. This is useful to define states like 'folded arms'-->
     <group_state name="home" group="arm">
-        <joint name="$(arg prefix)joint_1" value="0" />
-        <joint name="$(arg prefix)joint_2" value="0.26" />
-        <joint name="$(arg prefix)joint_3" value="-2.27" />
-        <joint name="$(arg prefix)joint_4" value="0" />
-        <joint name="$(arg prefix)joint_5" value="0.96" />
-        <joint name="$(arg prefix)joint_6" value="1.57" />
+        <joint name="joint_1" value="0"/>
+        <joint name="joint_2" value="0.26"/>
+        <joint name="joint_3" value="-2.27"/>
+        <joint name="joint_4" value="0"/>
+        <joint name="joint_5" value="0.96"/>
+        <joint name="joint_6" value="1.57"/>
     </group_state>
     <group_state name="retract" group="arm">
-        <joint name="$(arg prefix)joint_1" value="0" />
-        <joint name="$(arg prefix)joint_2" value="-0.35" />
-        <joint name="$(arg prefix)joint_3" value="-2.54" />
-        <joint name="$(arg prefix)joint_4" value="0" />
-        <joint name="$(arg prefix)joint_5" value="-0.87" />
-        <joint name="$(arg prefix)joint_6" value="1.57" />
+        <joint name="joint_1" value="0"/>
+        <joint name="joint_2" value="-0.35"/>
+        <joint name="joint_3" value="-2.54"/>
+        <joint name="joint_4" value="0"/>
+        <joint name="joint_5" value="-0.87"/>
+        <joint name="joint_6" value="1.57"/>
     </group_state>
     <group_state name="vertical" group="arm">
-        <joint name="$(arg prefix)joint_1" value="0" />
-        <joint name="$(arg prefix)joint_2" value="0" />
-        <joint name="$(arg prefix)joint_3" value="0" />
-        <joint name="$(arg prefix)joint_4" value="0" />
-        <joint name="$(arg prefix)joint_5" value="0" />
-        <joint name="$(arg prefix)joint_6" value="0" />
+        <joint name="joint_1" value="0"/>
+        <joint name="joint_2" value="0"/>
+        <joint name="joint_3" value="0"/>
+        <joint name="joint_4" value="0"/>
+        <joint name="joint_5" value="0"/>
+        <joint name="joint_6" value="0"/>
     </group_state>
     <group_state name="opened" group="gripper">
-        <joint name="$(arg prefix)left_inner_finger_joint" value="0" />
-        <joint name="$(arg prefix)right_inner_knuckle_joint" value="0" />
-        <joint name="$(arg prefix)finger_joint" value="0" />
-        <joint name="$(arg prefix)right_inner_finger_joint" value="0" />
-        <joint name="$(arg prefix)left_inner_knuckle_joint" value="0" />
-        <joint name="$(arg prefix)right_outer_knuckle_joint" value="0" />
+        <joint name="finger_joint" value="0"/>
+        <joint name="left_inner_finger_joint" value="0"/>
+        <joint name="left_inner_knuckle_joint" value="0"/>
+        <joint name="right_inner_finger_joint" value="0"/>
+        <joint name="right_inner_knuckle_joint" value="0"/>
+        <joint name="right_outer_knuckle_joint" value="0"/>
     </group_state>
     <group_state name="closed" group="gripper">
-        <joint name="$(arg prefix)left_inner_finger_joint" value="0.8" />
-        <joint name="$(arg prefix)right_inner_knuckle_joint" value="0.8" />
-        <joint name="$(arg prefix)finger_joint" value="0.8" />
-        <joint name="$(arg prefix)right_inner_finger_joint" value="-0.8" />
-        <joint name="$(arg prefix)left_inner_knuckle_joint" value="0.8" />
-        <joint name="$(arg prefix)right_outer_knuckle_joint" value="0.8" />
+        <joint name="finger_joint" value="0.8"/>
+        <joint name="left_inner_finger_joint" value="0.8"/>
+        <joint name="left_inner_knuckle_joint" value="0.8"/>
+        <joint name="right_inner_finger_joint" value="-0.8"/>
+        <joint name="right_inner_knuckle_joint" value="0.8"/>
+        <joint name="right_outer_knuckle_joint" value="0.8"/>
     </group_state>
     <!--END EFFECTOR: Purpose: Represent information about an end effector.-->
-    <end_effector name="gripper" parent_link="$(arg prefix)base_link" group="gripper" />
+    <end_effector name="gripper" parent_link="base_link" group="gripper"/>
+    <!--VIRTUAL JOINT: Purpose: this element defines a virtual joint between a robot link and an external frame of reference (considered fixed with respect to the robot)-->
+    <virtual_joint name="world" type="fixed" parent_frame="world" child_link="base_plate"/>
     <!--PASSIVE JOINT: Purpose: this element is used to mark joints that are not actuated-->
-    <passive_joint name="$(arg prefix)left_inner_finger_joint" />
-    <passive_joint name="$(arg prefix)left_inner_knuckle_joint" />
-    <passive_joint name="$(arg prefix)right_inner_knuckle_joint" />
-    <passive_joint name="$(arg prefix)right_outer_knuckle_joint" />
-    <passive_joint name="$(arg prefix)right_inner_finger_joint" />
+    <passive_joint name="left_inner_finger_joint"/>
+    <passive_joint name="left_inner_knuckle_joint"/>
+    <passive_joint name="right_inner_knuckle_joint"/>
+    <passive_joint name="right_outer_knuckle_joint"/>
+    <passive_joint name="right_inner_finger_joint"/>
     <!--DISABLE COLLISIONS: By default it is assumed that any link of the robot could potentially come into collision with any other link in the robot. This tag disables collision checking between a specified pair of links. -->
-    <disable_collisions link1="$(arg prefix)base_link" link2="$(arg prefix)bicep_link" reason="Never" />
-    <disable_collisions link1="$(arg prefix)base_link" link2="$(arg prefix)forearm_link" reason="Never" />
-    <disable_collisions link1="$(arg prefix)base_link" link2="$(arg prefix)shoulder_link" reason="Adjacent" />
-    <disable_collisions link1="$(arg prefix)bicep_link" link2="$(arg prefix)forearm_link" reason="Adjacent" />
-    <disable_collisions link1="$(arg prefix)bicep_link" link2="$(arg prefix)shoulder_link" reason="Adjacent" />
-    <disable_collisions link1="$(arg prefix)bicep_link" link2="$(arg prefix)spherical_wrist_1_link" reason="Never" />
-    <disable_collisions link1="$(arg prefix)bracelet_link" link2="$(arg prefix)forearm_link" reason="Never" />
-    <disable_collisions link1="$(arg prefix)bracelet_link" link2="$(arg prefix)left_inner_finger" reason="Never" />
-    <disable_collisions link1="$(arg prefix)bracelet_link" link2="$(arg prefix)left_inner_finger_pad" reason="Never" />
-    <disable_collisions link1="$(arg prefix)bracelet_link" link2="$(arg prefix)left_inner_knuckle" reason="Never" />
-    <disable_collisions link1="$(arg prefix)bracelet_link" link2="$(arg prefix)left_outer_finger" reason="Never" />
-    <disable_collisions link1="$(arg prefix)bracelet_link" link2="$(arg prefix)left_outer_knuckle" reason="Never" />
-    <disable_collisions link1="$(arg prefix)bracelet_link" link2="$(arg prefix)right_inner_finger" reason="Never" />
-    <disable_collisions link1="$(arg prefix)bracelet_link" link2="$(arg prefix)right_inner_finger_pad" reason="Never" />
-    <disable_collisions link1="$(arg prefix)bracelet_link" link2="$(arg prefix)right_inner_knuckle" reason="Never" />
-    <disable_collisions link1="$(arg prefix)bracelet_link" link2="$(arg prefix)right_outer_finger" reason="Never" />
-    <disable_collisions link1="$(arg prefix)bracelet_link" link2="$(arg prefix)right_outer_knuckle" reason="Never" />
-    <disable_collisions link1="$(arg prefix)bracelet_link" link2="$(arg prefix)robotiq_arg2f_base_link" reason="Adjacent" />
-    <disable_collisions link1="$(arg prefix)bracelet_link" link2="$(arg prefix)spherical_wrist_1_link" reason="Never" />
-    <disable_collisions link1="$(arg prefix)bracelet_link" link2="$(arg prefix)spherical_wrist_2_link" reason="Adjacent" />
-    <disable_collisions link1="$(arg prefix)forearm_link" link2="$(arg prefix)left_inner_finger" reason="Never" />
-    <disable_collisions link1="$(arg prefix)forearm_link" link2="$(arg prefix)left_inner_finger_pad" reason="Never" />
-    <disable_collisions link1="$(arg prefix)forearm_link" link2="$(arg prefix)left_inner_knuckle" reason="Never" />
-    <disable_collisions link1="$(arg prefix)forearm_link" link2="$(arg prefix)left_outer_finger" reason="Never" />
-    <disable_collisions link1="$(arg prefix)forearm_link" link2="$(arg prefix)left_outer_knuckle" reason="Never" />
-    <disable_collisions link1="$(arg prefix)forearm_link" link2="$(arg prefix)right_inner_finger" reason="Never" />
-    <disable_collisions link1="$(arg prefix)forearm_link" link2="$(arg prefix)right_inner_finger_pad" reason="Never" />
-    <disable_collisions link1="$(arg prefix)forearm_link" link2="$(arg prefix)right_inner_knuckle" reason="Never" />
-    <disable_collisions link1="$(arg prefix)forearm_link" link2="$(arg prefix)right_outer_finger" reason="Never" />
-    <disable_collisions link1="$(arg prefix)forearm_link" link2="$(arg prefix)right_outer_knuckle" reason="Never" />
-    <disable_collisions link1="$(arg prefix)forearm_link" link2="$(arg prefix)robotiq_arg2f_base_link" reason="Never" />
-    <disable_collisions link1="$(arg prefix)forearm_link" link2="$(arg prefix)shoulder_link" reason="Never" />
-    <disable_collisions link1="$(arg prefix)forearm_link" link2="$(arg prefix)spherical_wrist_1_link" reason="Adjacent" />
-    <disable_collisions link1="$(arg prefix)forearm_link" link2="$(arg prefix)spherical_wrist_2_link" reason="Never" />
-    <disable_collisions link1="$(arg prefix)left_inner_finger" link2="$(arg prefix)left_inner_finger_pad" reason="Adjacent" />
-    <disable_collisions link1="$(arg prefix)left_inner_finger" link2="$(arg prefix)left_inner_knuckle" reason="Default" />
-    <disable_collisions link1="$(arg prefix)left_inner_finger" link2="$(arg prefix)left_outer_finger" reason="Adjacent" />
-    <disable_collisions link1="$(arg prefix)left_inner_finger" link2="$(arg prefix)left_outer_knuckle" reason="Never" />
-    <disable_collisions link1="$(arg prefix)left_inner_finger" link2="$(arg prefix)right_inner_finger" reason="Never" />
-    <disable_collisions link1="$(arg prefix)left_inner_finger" link2="$(arg prefix)right_inner_finger_pad" reason="Never" />
-    <disable_collisions link1="$(arg prefix)left_inner_finger" link2="$(arg prefix)right_inner_knuckle" reason="Never" />
-    <disable_collisions link1="$(arg prefix)left_inner_finger" link2="$(arg prefix)right_outer_finger" reason="Never" />
-    <disable_collisions link1="$(arg prefix)left_inner_finger" link2="$(arg prefix)right_outer_knuckle" reason="Never" />
-    <disable_collisions link1="$(arg prefix)left_inner_finger" link2="$(arg prefix)robotiq_arg2f_base_link" reason="Never" />
-    <disable_collisions link1="$(arg prefix)left_inner_finger" link2="$(arg prefix)spherical_wrist_1_link" reason="Never" />
-    <disable_collisions link1="$(arg prefix)left_inner_finger" link2="$(arg prefix)spherical_wrist_2_link" reason="Never" />
-    <disable_collisions link1="$(arg prefix)left_inner_finger_pad" link2="$(arg prefix)left_inner_knuckle" reason="Never" />
-    <disable_collisions link1="$(arg prefix)left_inner_finger_pad" link2="$(arg prefix)left_outer_finger" reason="Never" />
-    <disable_collisions link1="$(arg prefix)left_inner_finger_pad" link2="$(arg prefix)left_outer_knuckle" reason="Never" />
-    <disable_collisions link1="$(arg prefix)left_inner_finger_pad" link2="$(arg prefix)right_inner_finger" reason="Never" />
-    <disable_collisions link1="$(arg prefix)left_inner_finger_pad" link2="$(arg prefix)right_inner_finger_pad" reason="Never" />
-    <disable_collisions link1="$(arg prefix)left_inner_finger_pad" link2="$(arg prefix)right_inner_knuckle" reason="Never" />
-    <disable_collisions link1="$(arg prefix)left_inner_finger_pad" link2="$(arg prefix)right_outer_finger" reason="Never" />
-    <disable_collisions link1="$(arg prefix)left_inner_finger_pad" link2="$(arg prefix)right_outer_knuckle" reason="Never" />
-    <disable_collisions link1="$(arg prefix)left_inner_finger_pad" link2="$(arg prefix)robotiq_arg2f_base_link" reason="Never" />
-    <disable_collisions link1="$(arg prefix)left_inner_finger_pad" link2="$(arg prefix)spherical_wrist_1_link" reason="Never" />
-    <disable_collisions link1="$(arg prefix)left_inner_finger_pad" link2="$(arg prefix)spherical_wrist_2_link" reason="Never" />
-    <disable_collisions link1="$(arg prefix)left_inner_knuckle" link2="$(arg prefix)left_outer_finger" reason="Never" />
-    <disable_collisions link1="$(arg prefix)left_inner_knuckle" link2="$(arg prefix)left_outer_knuckle" reason="Never" />
-    <disable_collisions link1="$(arg prefix)left_inner_knuckle" link2="$(arg prefix)right_inner_finger" reason="Never" />
-    <disable_collisions link1="$(arg prefix)left_inner_knuckle" link2="$(arg prefix)right_inner_finger_pad" reason="Never" />
-    <disable_collisions link1="$(arg prefix)left_inner_knuckle" link2="$(arg prefix)right_inner_knuckle" reason="Never" />
-    <disable_collisions link1="$(arg prefix)left_inner_knuckle" link2="$(arg prefix)right_outer_finger" reason="Never" />
-    <disable_collisions link1="$(arg prefix)left_inner_knuckle" link2="$(arg prefix)right_outer_knuckle" reason="Never" />
-    <disable_collisions link1="$(arg prefix)left_inner_knuckle" link2="$(arg prefix)robotiq_arg2f_base_link" reason="Adjacent" />
-    <disable_collisions link1="$(arg prefix)left_inner_knuckle" link2="$(arg prefix)spherical_wrist_1_link" reason="Never" />
-    <disable_collisions link1="$(arg prefix)left_inner_knuckle" link2="$(arg prefix)spherical_wrist_2_link" reason="Never" />
-    <disable_collisions link1="$(arg prefix)left_outer_finger" link2="$(arg prefix)left_outer_knuckle" reason="Adjacent" />
-    <disable_collisions link1="$(arg prefix)left_outer_finger" link2="$(arg prefix)right_inner_finger" reason="Never" />
-    <disable_collisions link1="$(arg prefix)left_outer_finger" link2="$(arg prefix)right_inner_finger_pad" reason="Never" />
-    <disable_collisions link1="$(arg prefix)left_outer_finger" link2="$(arg prefix)right_inner_knuckle" reason="Never" />
-    <disable_collisions link1="$(arg prefix)left_outer_finger" link2="$(arg prefix)right_outer_finger" reason="Never" />
-    <disable_collisions link1="$(arg prefix)left_outer_finger" link2="$(arg prefix)right_outer_knuckle" reason="Never" />
-    <disable_collisions link1="$(arg prefix)left_outer_finger" link2="$(arg prefix)robotiq_arg2f_base_link" reason="Never" />
-    <disable_collisions link1="$(arg prefix)left_outer_finger" link2="$(arg prefix)spherical_wrist_1_link" reason="Never" />
-    <disable_collisions link1="$(arg prefix)left_outer_finger" link2="$(arg prefix)spherical_wrist_2_link" reason="Never" />
-    <disable_collisions link1="$(arg prefix)left_outer_knuckle" link2="$(arg prefix)right_inner_finger" reason="Never" />
-    <disable_collisions link1="$(arg prefix)left_outer_knuckle" link2="$(arg prefix)right_inner_finger_pad" reason="Never" />
-    <disable_collisions link1="$(arg prefix)left_outer_knuckle" link2="$(arg prefix)right_inner_knuckle" reason="Never" />
-    <disable_collisions link1="$(arg prefix)left_outer_knuckle" link2="$(arg prefix)right_outer_finger" reason="Never" />
-    <disable_collisions link1="$(arg prefix)left_outer_knuckle" link2="$(arg prefix)right_outer_knuckle" reason="Never" />
-    <disable_collisions link1="$(arg prefix)left_outer_knuckle" link2="$(arg prefix)robotiq_arg2f_base_link" reason="Adjacent" />
-    <disable_collisions link1="$(arg prefix)left_outer_knuckle" link2="$(arg prefix)spherical_wrist_1_link" reason="Never" />
-    <disable_collisions link1="$(arg prefix)left_outer_knuckle" link2="$(arg prefix)spherical_wrist_2_link" reason="Never" />
-    <disable_collisions link1="$(arg prefix)right_inner_finger" link2="$(arg prefix)right_inner_finger_pad" reason="Adjacent" />
-    <disable_collisions link1="$(arg prefix)right_inner_finger" link2="$(arg prefix)right_inner_knuckle" reason="Default" />
-    <disable_collisions link1="$(arg prefix)right_inner_finger" link2="$(arg prefix)right_outer_finger" reason="Adjacent" />
-    <disable_collisions link1="$(arg prefix)right_inner_finger" link2="$(arg prefix)right_outer_knuckle" reason="Never" />
-    <disable_collisions link1="$(arg prefix)right_inner_finger" link2="$(arg prefix)robotiq_arg2f_base_link" reason="Never" />
-    <disable_collisions link1="$(arg prefix)right_inner_finger" link2="$(arg prefix)spherical_wrist_1_link" reason="Never" />
-    <disable_collisions link1="$(arg prefix)right_inner_finger" link2="$(arg prefix)spherical_wrist_2_link" reason="Never" />
-    <disable_collisions link1="$(arg prefix)right_inner_finger_pad" link2="$(arg prefix)right_inner_knuckle" reason="Never" />
-    <disable_collisions link1="$(arg prefix)right_inner_finger_pad" link2="$(arg prefix)right_outer_finger" reason="Never" />
-    <disable_collisions link1="$(arg prefix)right_inner_finger_pad" link2="$(arg prefix)right_outer_knuckle" reason="Never" />
-    <disable_collisions link1="$(arg prefix)right_inner_finger_pad" link2="$(arg prefix)robotiq_arg2f_base_link" reason="Never" />
-    <disable_collisions link1="$(arg prefix)right_inner_finger_pad" link2="$(arg prefix)spherical_wrist_1_link" reason="Never" />
-    <disable_collisions link1="$(arg prefix)right_inner_finger_pad" link2="$(arg prefix)spherical_wrist_2_link" reason="Never" />
-    <disable_collisions link1="$(arg prefix)right_inner_knuckle" link2="$(arg prefix)right_outer_finger" reason="Never" />
-    <disable_collisions link1="$(arg prefix)right_inner_knuckle" link2="$(arg prefix)right_outer_knuckle" reason="Never" />
-    <disable_collisions link1="$(arg prefix)right_inner_knuckle" link2="$(arg prefix)robotiq_arg2f_base_link" reason="Adjacent" />
-    <disable_collisions link1="$(arg prefix)right_inner_knuckle" link2="$(arg prefix)spherical_wrist_1_link" reason="Never" />
-    <disable_collisions link1="$(arg prefix)right_inner_knuckle" link2="$(arg prefix)spherical_wrist_2_link" reason="Never" />
-    <disable_collisions link1="$(arg prefix)right_outer_finger" link2="$(arg prefix)right_outer_knuckle" reason="Adjacent" />
-    <disable_collisions link1="$(arg prefix)right_outer_finger" link2="$(arg prefix)robotiq_arg2f_base_link" reason="Never" />
-    <disable_collisions link1="$(arg prefix)right_outer_finger" link2="$(arg prefix)spherical_wrist_1_link" reason="Never" />
-    <disable_collisions link1="$(arg prefix)right_outer_finger" link2="$(arg prefix)spherical_wrist_2_link" reason="Never" />
-    <disable_collisions link1="$(arg prefix)right_outer_knuckle" link2="$(arg prefix)robotiq_arg2f_base_link" reason="Adjacent" />
-    <disable_collisions link1="$(arg prefix)right_outer_knuckle" link2="$(arg prefix)spherical_wrist_1_link" reason="Never" />
-    <disable_collisions link1="$(arg prefix)right_outer_knuckle" link2="$(arg prefix)spherical_wrist_2_link" reason="Never" />
-    <disable_collisions link1="$(arg prefix)robotiq_arg2f_base_link" link2="$(arg prefix)spherical_wrist_1_link" reason="Never" />
-    <disable_collisions link1="$(arg prefix)robotiq_arg2f_base_link" link2="$(arg prefix)spherical_wrist_2_link" reason="Never" />
-    <disable_collisions link1="$(arg prefix)shoulder_link" link2="$(arg prefix)spherical_wrist_1_link" reason="Never" />
-    <disable_collisions link1="$(arg prefix)spherical_wrist_1_link" link2="$(arg prefix)spherical_wrist_2_link" reason="Adjacent" />
+    <disable_collisions link1="base_link" link2="bicep_link" reason="Never"/>
+    <disable_collisions link1="base_link" link2="forearm_link" reason="Never"/>
+    <disable_collisions link1="base_link" link2="shoulder_link" reason="Adjacent"/>
+    <disable_collisions link1="bicep_link" link2="forearm_link" reason="Adjacent"/>
+    <disable_collisions link1="bicep_link" link2="shoulder_link" reason="Adjacent"/>
+    <disable_collisions link1="bicep_link" link2="spherical_wrist_1_link" reason="Never"/>
+    <disable_collisions link1="bracelet_link" link2="forearm_link" reason="Never"/>
+    <disable_collisions link1="bracelet_link" link2="left_inner_finger" reason="Never"/>
+    <disable_collisions link1="bracelet_link" link2="left_inner_finger_pad" reason="Never"/>
+    <disable_collisions link1="bracelet_link" link2="left_inner_knuckle" reason="Never"/>
+    <disable_collisions link1="bracelet_link" link2="left_outer_finger" reason="Never"/>
+    <disable_collisions link1="bracelet_link" link2="left_outer_knuckle" reason="Never"/>
+    <disable_collisions link1="bracelet_link" link2="right_inner_finger" reason="Never"/>
+    <disable_collisions link1="bracelet_link" link2="right_inner_finger_pad" reason="Never"/>
+    <disable_collisions link1="bracelet_link" link2="right_inner_knuckle" reason="Never"/>
+    <disable_collisions link1="bracelet_link" link2="right_outer_finger" reason="Never"/>
+    <disable_collisions link1="bracelet_link" link2="right_outer_knuckle" reason="Never"/>
+    <disable_collisions link1="bracelet_link" link2="robotiq_arg2f_base_link" reason="Adjacent"/>
+    <disable_collisions link1="bracelet_link" link2="spherical_wrist_1_link" reason="Never"/>
+    <disable_collisions link1="bracelet_link" link2="spherical_wrist_2_link" reason="Adjacent"/>
+    <disable_collisions link1="forearm_link" link2="left_inner_finger" reason="Never"/>
+    <disable_collisions link1="forearm_link" link2="left_inner_finger_pad" reason="Never"/>
+    <disable_collisions link1="forearm_link" link2="left_inner_knuckle" reason="Never"/>
+    <disable_collisions link1="forearm_link" link2="left_outer_finger" reason="Never"/>
+    <disable_collisions link1="forearm_link" link2="left_outer_knuckle" reason="Never"/>
+    <disable_collisions link1="forearm_link" link2="right_inner_finger" reason="Never"/>
+    <disable_collisions link1="forearm_link" link2="right_inner_finger_pad" reason="Never"/>
+    <disable_collisions link1="forearm_link" link2="right_inner_knuckle" reason="Never"/>
+    <disable_collisions link1="forearm_link" link2="right_outer_finger" reason="Never"/>
+    <disable_collisions link1="forearm_link" link2="right_outer_knuckle" reason="Never"/>
+    <disable_collisions link1="forearm_link" link2="robotiq_arg2f_base_link" reason="Never"/>
+    <disable_collisions link1="forearm_link" link2="shoulder_link" reason="Never"/>
+    <disable_collisions link1="forearm_link" link2="spherical_wrist_1_link" reason="Adjacent"/>
+    <disable_collisions link1="forearm_link" link2="spherical_wrist_2_link" reason="Never"/>
+    <disable_collisions link1="left_inner_finger" link2="left_inner_finger_pad" reason="Adjacent"/>
+    <disable_collisions link1="left_inner_finger" link2="left_inner_knuckle" reason="Default"/>
+    <disable_collisions link1="left_inner_finger" link2="left_outer_finger" reason="Adjacent"/>
+    <disable_collisions link1="left_inner_finger" link2="left_outer_knuckle" reason="Never"/>
+    <disable_collisions link1="left_inner_finger" link2="right_inner_finger" reason="Never"/>
+    <disable_collisions link1="left_inner_finger" link2="right_inner_finger_pad" reason="Never"/>
+    <disable_collisions link1="left_inner_finger" link2="right_inner_knuckle" reason="Never"/>
+    <disable_collisions link1="left_inner_finger" link2="right_outer_finger" reason="Never"/>
+    <disable_collisions link1="left_inner_finger" link2="right_outer_knuckle" reason="Never"/>
+    <disable_collisions link1="left_inner_finger" link2="robotiq_arg2f_base_link" reason="Never"/>
+    <disable_collisions link1="left_inner_finger" link2="spherical_wrist_1_link" reason="Never"/>
+    <disable_collisions link1="left_inner_finger" link2="spherical_wrist_2_link" reason="Never"/>
+    <disable_collisions link1="left_inner_finger_pad" link2="left_inner_knuckle" reason="Never"/>
+    <disable_collisions link1="left_inner_finger_pad" link2="left_outer_finger" reason="Never"/>
+    <disable_collisions link1="left_inner_finger_pad" link2="left_outer_knuckle" reason="Never"/>
+    <disable_collisions link1="left_inner_finger_pad" link2="right_inner_finger" reason="Never"/>
+    <disable_collisions link1="left_inner_finger_pad" link2="right_inner_finger_pad" reason="Never"/>
+    <disable_collisions link1="left_inner_finger_pad" link2="right_inner_knuckle" reason="Never"/>
+    <disable_collisions link1="left_inner_finger_pad" link2="right_outer_finger" reason="Never"/>
+    <disable_collisions link1="left_inner_finger_pad" link2="right_outer_knuckle" reason="Never"/>
+    <disable_collisions link1="left_inner_finger_pad" link2="robotiq_arg2f_base_link" reason="Never"/>
+    <disable_collisions link1="left_inner_finger_pad" link2="spherical_wrist_1_link" reason="Never"/>
+    <disable_collisions link1="left_inner_finger_pad" link2="spherical_wrist_2_link" reason="Never"/>
+    <disable_collisions link1="left_inner_knuckle" link2="left_outer_finger" reason="Never"/>
+    <disable_collisions link1="left_inner_knuckle" link2="left_outer_knuckle" reason="Never"/>
+    <disable_collisions link1="left_inner_knuckle" link2="right_inner_finger" reason="Never"/>
+    <disable_collisions link1="left_inner_knuckle" link2="right_inner_finger_pad" reason="Never"/>
+    <disable_collisions link1="left_inner_knuckle" link2="right_inner_knuckle" reason="Never"/>
+    <disable_collisions link1="left_inner_knuckle" link2="right_outer_finger" reason="Never"/>
+    <disable_collisions link1="left_inner_knuckle" link2="right_outer_knuckle" reason="Never"/>
+    <disable_collisions link1="left_inner_knuckle" link2="robotiq_arg2f_base_link" reason="Adjacent"/>
+    <disable_collisions link1="left_inner_knuckle" link2="spherical_wrist_1_link" reason="Never"/>
+    <disable_collisions link1="left_inner_knuckle" link2="spherical_wrist_2_link" reason="Never"/>
+    <disable_collisions link1="left_outer_finger" link2="left_outer_knuckle" reason="Adjacent"/>
+    <disable_collisions link1="left_outer_finger" link2="right_inner_finger" reason="Never"/>
+    <disable_collisions link1="left_outer_finger" link2="right_inner_finger_pad" reason="Never"/>
+    <disable_collisions link1="left_outer_finger" link2="right_inner_knuckle" reason="Never"/>
+    <disable_collisions link1="left_outer_finger" link2="right_outer_finger" reason="Never"/>
+    <disable_collisions link1="left_outer_finger" link2="right_outer_knuckle" reason="Never"/>
+    <disable_collisions link1="left_outer_finger" link2="robotiq_arg2f_base_link" reason="Never"/>
+    <disable_collisions link1="left_outer_finger" link2="spherical_wrist_1_link" reason="Never"/>
+    <disable_collisions link1="left_outer_finger" link2="spherical_wrist_2_link" reason="Never"/>
+    <disable_collisions link1="left_outer_knuckle" link2="right_inner_finger" reason="Never"/>
+    <disable_collisions link1="left_outer_knuckle" link2="right_inner_finger_pad" reason="Never"/>
+    <disable_collisions link1="left_outer_knuckle" link2="right_inner_knuckle" reason="Never"/>
+    <disable_collisions link1="left_outer_knuckle" link2="right_outer_finger" reason="Never"/>
+    <disable_collisions link1="left_outer_knuckle" link2="right_outer_knuckle" reason="Never"/>
+    <disable_collisions link1="left_outer_knuckle" link2="robotiq_arg2f_base_link" reason="Adjacent"/>
+    <disable_collisions link1="left_outer_knuckle" link2="spherical_wrist_1_link" reason="Never"/>
+    <disable_collisions link1="left_outer_knuckle" link2="spherical_wrist_2_link" reason="Never"/>
+    <disable_collisions link1="right_inner_finger" link2="right_inner_finger_pad" reason="Adjacent"/>
+    <disable_collisions link1="right_inner_finger" link2="right_inner_knuckle" reason="Default"/>
+    <disable_collisions link1="right_inner_finger" link2="right_outer_finger" reason="Adjacent"/>
+    <disable_collisions link1="right_inner_finger" link2="right_outer_knuckle" reason="Never"/>
+    <disable_collisions link1="right_inner_finger" link2="robotiq_arg2f_base_link" reason="Never"/>
+    <disable_collisions link1="right_inner_finger" link2="spherical_wrist_1_link" reason="Never"/>
+    <disable_collisions link1="right_inner_finger" link2="spherical_wrist_2_link" reason="Never"/>
+    <disable_collisions link1="right_inner_finger_pad" link2="right_inner_knuckle" reason="Never"/>
+    <disable_collisions link1="right_inner_finger_pad" link2="right_outer_finger" reason="Never"/>
+    <disable_collisions link1="right_inner_finger_pad" link2="right_outer_knuckle" reason="Never"/>
+    <disable_collisions link1="right_inner_finger_pad" link2="robotiq_arg2f_base_link" reason="Never"/>
+    <disable_collisions link1="right_inner_finger_pad" link2="spherical_wrist_1_link" reason="Never"/>
+    <disable_collisions link1="right_inner_finger_pad" link2="spherical_wrist_2_link" reason="Never"/>
+    <disable_collisions link1="right_inner_knuckle" link2="right_outer_finger" reason="Never"/>
+    <disable_collisions link1="right_inner_knuckle" link2="right_outer_knuckle" reason="Never"/>
+    <disable_collisions link1="right_inner_knuckle" link2="robotiq_arg2f_base_link" reason="Adjacent"/>
+    <disable_collisions link1="right_inner_knuckle" link2="spherical_wrist_1_link" reason="Never"/>
+    <disable_collisions link1="right_inner_knuckle" link2="spherical_wrist_2_link" reason="Never"/>
+    <disable_collisions link1="right_outer_finger" link2="right_outer_knuckle" reason="Adjacent"/>
+    <disable_collisions link1="right_outer_finger" link2="robotiq_arg2f_base_link" reason="Never"/>
+    <disable_collisions link1="right_outer_finger" link2="spherical_wrist_1_link" reason="Never"/>
+    <disable_collisions link1="right_outer_finger" link2="spherical_wrist_2_link" reason="Never"/>
+    <disable_collisions link1="right_outer_knuckle" link2="robotiq_arg2f_base_link" reason="Adjacent"/>
+    <disable_collisions link1="right_outer_knuckle" link2="spherical_wrist_1_link" reason="Never"/>
+    <disable_collisions link1="right_outer_knuckle" link2="spherical_wrist_2_link" reason="Never"/>
+    <disable_collisions link1="robotiq_arg2f_base_link" link2="spherical_wrist_1_link" reason="Never"/>
+    <disable_collisions link1="robotiq_arg2f_base_link" link2="spherical_wrist_2_link" reason="Never"/>
+    <disable_collisions link1="shoulder_link" link2="spherical_wrist_1_link" reason="Never"/>
+    <disable_collisions link1="spherical_wrist_1_link" link2="spherical_wrist_2_link" reason="Adjacent"/>
 </robot>
