Commit message: tweeked configuration for rviz and octomap

File: kortex_description/arms/gen3/6dof/urdf/gen3_macro.xacro (robot description, xacro)
@@ -252,5 +252,5 @@
       <link name="${prefix}camera_depth_frame" />
       <joint name="${prefix}depth_module" type="fixed">
-        <origin xyz="0.0275 0.066 -0.00305" rpy="3.14159265358979 3.14159265358979 0" />
+        <origin xyz="0 0.066 -0.00305" rpy="3.14159265358979 3.14159265358979 0" />
         <parent link="${prefix}end_effector_link" />
         <child  link="${prefix}camera_depth_frame" />

File: kortex_description/arms/gen3/6dof/urdf/rgbd_camera.xacro (robot description, xacro)
@@ -38,6 +38,6 @@
                     <horizontal_fov>1.047198</horizontal_fov>
                     <image>
-                        <width>640</width>
-                        <height>640</height>
+                        <width>600</width>
+                        <height>300</height>
                         <format>R8G8B8</format>
                     </image>

Commit message: restructured some direcotries and files

File: kortex_description/arms/gen3/6dof/urdf/gen3_macro.xacro (robot description, xacro)
@@ -1,5 +1,5 @@
 <?xml version="1.0"?>
 <robot name="gen3_arm" xmlns:xacro="http://ros.org/wiki/xacro">
-  <xacro:include filename="$(find kortex_description)/arms/gen3/6dof/urdf/rgbd_camera.xacro" />
+  <xacro:include filename="$(find kortex_scripts)/robot_equipment/urdf/rgbd_camera.xacro" />
   <!-- Propagate last link name information because it is the gripper's parent link -->
   <xacro:property name="last_arm_link" value="end_effector_link"/>

File: kortex_description/robots/kortex_robot.xacro (robot description, xacro)
@@ -8,5 +8,5 @@
         </xacro:unless>
         <xacro:if value="${base}">
-            <xacro:include filename= "$(find kortex_description)/arms/${arm}/${dof}dof/urdf/base.xacro"/>
+            <xacro:include filename= "$(find kortex_scripts)/robot_equipment/urdf/base.xacro"/>
         </xacro:if>
         <xacro:if value="${sim}">

File: kortex_scripts/objects/urdf/qr_grasp_block.xacro (robot description, xacro)
@@ -1,5 +1,5 @@
 <?xml version="1.0"?>
 <robot name="qr_$(arg type)_block" xmlns:xacro="http://ros.org/wiki/xacro">
-    <xacro:include filename= "$(find kortex_scripts)/objects/macros.xacro"/>
+    <xacro:include filename= "$(find kortex_scripts)/objects/urdf/macros.xacro"/>
     <xacro:property name="block_lenght" value="0.058"/>
     <xacro:property name="block_width" value="0.058"/>
@@ -24,8 +24,8 @@
             <geometry>
                 <xacro:if value="${type == 'tomato'}">
-                    <mesh filename="/home/alex/mor/kinova_dev_alex/catkin_workspace/src/ros_kortex/kortex_scripts/objects/models/tomato_qr_grasp_block.dae" />
+                    <mesh filename="/home/alex/mor/kinova_dev_alex/catkin_workspace/src/ros_kortex/kortex_scripts/objects/meshes/tomato_qr_grasp_block.dae" />
                 </xacro:if>
                 <xacro:if value="${type == 'pepper'}">
-                    <mesh filename="/home/alex/mor/kinova_dev_alex/catkin_workspace/src/ros_kortex/kortex_scripts/objects/models/pepper_qr_grasp_block.dae" />
+                    <mesh filename="/home/alex/mor/kinova_dev_alex/catkin_workspace/src/ros_kortex/kortex_scripts/objects/meshes/pepper_qr_grasp_block.dae" />
                 </xacro:if>
                 <xacro:if value="${type == 'block'}">

File: kortex_scripts/robot_equipment/urdf/base.xacro (robot description, xacro)
@@ -1,5 +1,5 @@
 <?xml version="1.0"?>
 <robot xmlns:xacro="http://ros.org/wiki/xacro">
-    <xacro:include filename= "$(find kortex_description)/arms/${arm}/${dof}dof/urdf/macros.xacro"/>
+    <xacro:include filename= "$(find kortex_scripts)/robot_equipment/urdf/macros.xacro"/>
     <xacro:macro name="chair">
         <link name="base_plate">
@@ -40,5 +40,5 @@
                 <origin xyz="-0.075 -.075 -0.45" rpy="1.57 0 1.57" />
                 <geometry>
-                    <mesh filename="package://kortex_description/arms/gen3/${dof}dof/meshes/parametric_chair.STL" />
+                    <mesh filename="package://kortex_scripts/robot_equipment/meshes/parametric_chair.STL" />
                 </geometry>
                 <material name="grey">

File: kortex_scripts/robot_equipment/urdf/rgbd_camera.xacro (robot description, xacro)
@@ -2,34 +2,4 @@
 <robot xmlns:xacro="http://ros.org/wiki/xacro">
     <xacro:macro name="depth_cam">
-    <!--
-        <link name="camera_offset_link">
-            <inertial>
-                <origin xyz="0 0 0" rpy="0 0 0" />
-                <mass value="0" />
-                <inertia ixx="0" ixy="0" ixz="0" iyy="0" iyz="0" izz="0" />
-            </inertial>
-            <visual>
-                <origin xyz="0 0 0" rpy="0 0 0" />
-                <geometry>
-                    <box size="0.01 0.01 0.01"/>
-                </geometry>
-                <material name="">
-                    <color rgba="0.75294 0.75294 0.75294 1" />
-                </material>
-            </visual>
-            <collision>
-                <origin xyz="0 0 0" rpy="0 0 0" />
-                <geometry>
-                    <box size="0.01 0.01 0.01"/>
-                </geometry>
-            </collision>
-        </link>
-        <joint name="camera_offset_joint" type="fixed">
-            <origin xyz="0 0 0.5" rpy="0 0 0" />
-            <parent link="camera_link" />
-            <child link="camera_offset_link" />
-            <axis xyz="0 0 0" />
-        </joint>
-        -->
         <gazebo reference="camera_link">
             <sensor name="camera" type="depth">

Commit message: upside down arm

File: kortex_description/arms/gen3/6dof/urdf/gen3_macro.xacro (robot description, xacro)
@@ -27,5 +27,5 @@
       </collision>
     </link>
-    <xacro:if value="${base}">
+    <xacro:if value="${base}"> <!--I added this-->
       <xacro:chair/>
     </xacro:if>

File: kortex_scripts/robot_equipment/urdf/base.xacro (robot description, xacro)
@@ -7,5 +7,5 @@
         <xacro:worker_simple/>
         <joint name="chair-base_joint" type="fixed">
-            <origin xyz="0.16 0 -0.44" rpy="0 0 0" />
+            <origin xyz="0.1 0 0" rpy="0 3.14 0" />
             <parent link="chair_link" />
             <child link="base_link" />
@@ -16,10 +16,11 @@
                 <origin xyz="0 0 0" rpy="0 0 0" />
                 <mass value="4" />
-                <xacro:box_inertia mass="4" x="0.1" y="0.1" z="0.9" />
+                <xacro:box_inertia mass="4" x="0.2" y="0.1" z="0.0125" />
             </inertial>
             <visual>
-                <origin xyz="-0.075 -.075 -0.45" rpy="1.57 0 1.57" />
+                <origin xyz="0 0 0" rpy="0 0 0" />
                 <geometry>
-                    <mesh filename="package://kortex_scripts/robot_equipment/meshes/parametric_chair.STL" />
+                    <!-- <mesh filename="package://kortex_scripts/robot_equipment/meshes/parametric_chair.STL" /> -->
+                    <box size="0.2 0.1 0.0125"/>
                 </geometry>
                 <material name="grey">
@@ -30,5 +31,5 @@
                 <origin xyz="0 0 0" rpy="0 0 0" />
                 <geometry>
-                    <box size="0.1 0.1 0.9"/>
+                    <box size="0.2 0.1 0.0125"/>
                 </geometry>
             </collision>

File: kortex_scripts/robot_equipment/urdf/worker_simple.xacro (robot description, xacro)
@@ -109,5 +109,5 @@
         </joint>
         <joint name="mast_chair_joint" type="fixed">
-            <origin xyz="0 0 0.300" rpy="0 0 0" />
+            <origin xyz="0.1 0 0.75" rpy="0 0 0" />
             <parent link="mast_link" />
             <child link="chair_link" />

Commit message: cleaned up implementaion of worker arm

File: kortex_description/arms/gen3/6dof/urdf/gen3_macro.xacro (robot description, xacro)
@@ -1,5 +1,4 @@
 <?xml version="1.0"?>
 <robot name="gen3_arm" xmlns:xacro="http://ros.org/wiki/xacro">
-  <xacro:include filename="$(find kortex_scripts)/robot_equipment/urdf/rgbd_camera.xacro" />
   <!-- Propagate last link name information because it is the gripper's parent link -->
   <xacro:property name="last_arm_link" value="end_effector_link"/>

File: kortex_description/robots/kortex_robot.xacro (robot description, xacro)
@@ -17,20 +17,20 @@
                 <xacro:include filename="$(find kortex_description)/grippers/${gripper}/urdf/${gripper}_transmission_macro.xacro" />
             </xacro:unless>
+            <xacro:if value="${vision}">
+                <xacro:include filename="$(find kortex_scripts)/robot_equipment/urdf/rgbd_camera.xacro" />
+            </xacro:if>
         </xacro:if>
         <!-- Run the macros -->
         <!-- For gazebo-->
-        <!-- <xacro:if value="${sim}">
-            <link name="world" />
-            <joint name="world_to_root" type="fixed">
-                <xacro:if value="${base}">
-                    <child link="worker_body_link" />
-                </xacro:if>
-                <xacro:if value="${not base}">
+        <xacro:if value="${not base}">
+            <xacro:if value="${sim}">
+                <link name="world" />
+                <joint name="world_to_root" type="fixed">
                     <child link="base_link" />
-                </xacro:if>
-                <parent link="world" />
-                <origin xyz="0 0 0.01" rpy="0 0 0" />
-            </joint>
-        </xacro:if> -->
+                    <parent link="world" />
+                    <origin xyz="0 0 0.01" rpy="0 0 0" />
+                </joint>
+            </xacro:if>
+        </xacro:if>
         <!-- Load the arm -->
         <xacro:load_arm parent="" dof="${dof}" vision="${vision}" base="${base}" prefix="${prefix}">

File: kortex_move_it_config/gen3_robotiq_2f_85_move_it_config/config/6dof/gen3_robotiq_2f_85.srdf.xacro (robot description, xacro)
@@ -77,5 +77,5 @@
     <end_effector name="gripper" parent_link="base_link" group="gripper"/>
     <!--VIRTUAL JOINT: Purpose: this element defines a virtual joint between a robot link and an external frame of reference (considered fixed with respect to the robot)-->
-    <virtual_joint name="elevator_chair_link" type="fixed" parent_frame="worker_base_link" child_link="chair_link"/>
+    <!-- <virtual_joint name="elevator_chair_link" type="fixed" parent_frame="worker_base_link" child_link="chair_link"/> -->
     <!--PASSIVE JOINT: Purpose: this element is used to mark joints that are not actuated-->
     <passive_joint name="left_inner_finger_joint"/>

File: kortex_scripts/robot_equipment/urdf/base.xacro (robot description, xacro)
@@ -3,12 +3,10 @@
     <xacro:include filename= "$(find kortex_scripts)/robot_equipment/urdf/macros.xacro"/>
     <xacro:include filename= "$(find kortex_scripts)/robot_equipment/urdf/properties.xacro"/>
-    <!-- <xacro:include filename= "$(find kortex_scripts)/robot_equipment/urdf/worker_simple.xacro"/> -->
     <xacro:include filename= "$(find ant_worker_description)/urdf/worker.urdf.xacro"/>
     <xacro:macro name="chair">
-        <!-- <xacro:worker_simple/> -->
-        <xacro:pls_work/>
+        <xacro:ant_worker/>
         <joint name="elevator_top_joint" type="fixed">
-            <origin xyz="0.1 0 0" rpy="0 3.14 0" />
-            <parent link="elevator_shaft" />
+            <origin xyz="0.1 0 0" rpy="0 0 3.14" />
+            <parent link="elevator_top" />
             <child link="chair_link" />
             <axis xyz="0 0 0" />

File: kortex_scripts/robot_equipment/urdf/properties.xacro (robot description, xacro)
@@ -1,13 +1,4 @@
 <?xml version="1.0"?>
 <robot xmlns:xacro="http://ros.org/wiki/xacro">
-    <xacro:property name="worker_length" value="0.95"/>
-    <xacro:property name="worker_width" value="0.55"/>
-    <xacro:property name="worker_height" value="0.5"/>
-    <xacro:property name="worker_mass" value="100"/>
-    <xacro:property name="mast_length" value="1.5"/>
-    <xacro:property name="mast_radius" value="0.055"/>
-    <xacro:property name="mast_mass" value="30"/>
-    <xacro:property name="mast_edge_center_distance" value="0.1"/>
-    <xacro:property name="mast_height_offset" value="-0.4"/>
     <xacro:property name="spool_length" value="0.1"/>
     <xacro:property name="spool_radius" value="0.2"/>
