Commit message: dockerized

File: kortex_scripts/objects/urdf/qr_grasp_block.xacro (robot description, xacro)
@@ -24,8 +24,8 @@
             <geometry>
                 <xacro:if value="${type == 'tomato'}">
-                    <mesh filename="/home/alex/mor/kinova_dev_alex/catkin_workspace/src/ros_kortex/kortex_scripts/objects/meshes/tomato_qr_grasp_block.dae" />
+                    <mesh filename="package://kortex_scripts/objects/meshes/tomato_qr_grasp_block.dae" />
                 </xacro:if>
                 <xacro:if value="${type == 'pepper'}">
-                    <mesh filename="/home/alex/mor/kinova_dev_alex/catkin_workspace/src/ros_kortex/kortex_scripts/objects/meshes/pepper_qr_grasp_block.dae" />
+                    <mesh filename="package://kortex_scripts/objects/meshes/pepper_qr_grasp_block.dae" />
                 </xacro:if>
                 <xacro:if value="${type == 'block'}">
