Commit message: merged mobile arm code

File: kortex_move_it_config/gen3_robotiq_2f_85_move_it_config/config/6dof/gen3_robotiq_2f_85.srdf.xacro (robot description, xacro)
@@ -77,5 +77,5 @@
     <end_effector name="gripper" parent_link="base_link" group="gripper"/>
     <!--VIRTUAL JOINT: Purpose: this element defines a virtual joint between a robot link and an external frame of reference (considered fixed with respect to the robot)-->
-    <virtual_joint name="mast_base_link" type="fixed" parent_frame="mast_link" child_link="base_link"/>
+    <virtual_joint name="elevator_chair_link" type="fixed" parent_frame="worker_base_link" child_link="chair_link"/>
     <!--PASSIVE JOINT: Purpose: this element is used to mark joints that are not actuated-->
     <passive_joint name="left_inner_finger_joint"/>
@@ -86,24 +86,39 @@
     <!--DISABLE COLLISIONS: By default it is assumed that any link of the robot could potentially come into collision with any other link in the robot. This tag disables collision checking between a specified pair of links. -->
     <disable_collisions link1="base_link" link2="bicep_link" reason="Never"/>
-    <disable_collisions link1="base_link" link2="bio_container_link" reason="Never"/>
     <disable_collisions link1="base_link" link2="chair_link" reason="Adjacent"/>
-    <disable_collisions link1="base_link" link2="mast_link" reason="Never"/>
+    <disable_collisions link1="base_link" link2="elevator_shaft" reason="Never"/>
+    <disable_collisions link1="base_link" link2="elevator_top" reason="Never"/>
+    <disable_collisions link1="base_link" link2="forearm_link" reason="Never"/>
+    <disable_collisions link1="base_link" link2="leg_0" reason="Never"/>
+    <disable_collisions link1="base_link" link2="leg_0_wheel_in" reason="Never"/>
+    <disable_collisions link1="base_link" link2="leg_0_wheel_out" reason="Never"/>
+    <disable_collisions link1="base_link" link2="leg_1" reason="Never"/>
+    <disable_collisions link1="base_link" link2="leg_1_wheel_in" reason="Never"/>
+    <disable_collisions link1="base_link" link2="leg_1_wheel_out" reason="Never"/>
+    <disable_collisions link1="base_link" link2="leg_2" reason="Never"/>
+    <disable_collisions link1="base_link" link2="leg_2_wheel_in" reason="Never"/>
+    <disable_collisions link1="base_link" link2="leg_2_wheel_out" reason="Never"/>
+    <disable_collisions link1="base_link" link2="leg_3" reason="Never"/>
+    <disable_collisions link1="base_link" link2="leg_3_wheel_in" reason="Never"/>
+    <disable_collisions link1="base_link" link2="leg_3_wheel_out" reason="Never"/>
     <disable_collisions link1="base_link" link2="shoulder_link" reason="Adjacent"/>
-    <disable_collisions link1="base_link" link2="spool_link" reason="Never"/>
     <disable_collisions link1="base_link" link2="worker_body_link" reason="Never"/>
-    <disable_collisions link1="bicep_link" link2="bio_container_link" reason="Never"/>
     <disable_collisions link1="bicep_link" link2="chair_link" reason="Never"/>
     <disable_collisions link1="bicep_link" link2="forearm_link" reason="Adjacent"/>
+    <disable_collisions link1="bicep_link" link2="leg_0" reason="Never"/>
+    <disable_collisions link1="bicep_link" link2="leg_0_wheel_in" reason="Never"/>
+    <disable_collisions link1="bicep_link" link2="leg_0_wheel_out" reason="Never"/>
+    <disable_collisions link1="bicep_link" link2="leg_1" reason="Never"/>
+    <disable_collisions link1="bicep_link" link2="leg_1_wheel_in" reason="Never"/>
+    <disable_collisions link1="bicep_link" link2="leg_1_wheel_out" reason="Never"/>
+    <disable_collisions link1="bicep_link" link2="leg_2" reason="Never"/>
+    <disable_collisions link1="bicep_link" link2="leg_2_wheel_in" reason="Never"/>
+    <disable_collisions link1="bicep_link" link2="leg_2_wheel_out" reason="Never"/>
+    <disable_collisions link1="bicep_link" link2="leg_3" reason="Never"/>
+    <disable_collisions link1="bicep_link" link2="leg_3_wheel_in" reason="Never"/>
+    <disable_collisions link1="bicep_link" link2="leg_3_wheel_out" reason="Never"/>
     <disable_collisions link1="bicep_link" link2="shoulder_link" reason="Adjacent"/>
     <disable_collisions link1="bicep_link" link2="spherical_wrist_1_link" reason="Never"/>
-    <disable_collisions link1="bicep_link" link2="spool_link" reason="Never"/>
     <disable_collisions link1="bicep_link" link2="worker_body_link" reason="Never"/>
-    <disable_collisions link1="bio_container_link" link2="chair_link" reason="Never"/>
-    <disable_collisions link1="bio_container_link" link2="forearm_link" reason="Never"/>
-    <disable_collisions link1="bio_container_link" link2="mast_link" reason="Never"/>
-    <disable_collisions link1="bio_container_link" link2="shoulder_link" reason="Never"/>
-    <disable_collisions link1="bio_container_link" link2="spherical_wrist_1_link" reason="Never"/>
-    <disable_collisions link1="bio_container_link" link2="spool_link" reason="Never"/>
-    <disable_collisions link1="bio_container_link" link2="worker_body_link" reason="Adjacent"/>
     <disable_collisions link1="bracelet_link" link2="forearm_link" reason="Never"/>
     <disable_collisions link1="bracelet_link" link2="left_inner_finger" reason="Never"/>
@@ -112,4 +127,16 @@
     <disable_collisions link1="bracelet_link" link2="left_outer_finger" reason="Never"/>
     <disable_collisions link1="bracelet_link" link2="left_outer_knuckle" reason="Never"/>
+    <disable_collisions link1="bracelet_link" link2="leg_0" reason="Never"/>
+    <disable_collisions link1="bracelet_link" link2="leg_0_wheel_in" reason="Never"/>
+    <disable_collisions link1="bracelet_link" link2="leg_0_wheel_out" reason="Never"/>
+    <disable_collisions link1="bracelet_link" link2="leg_1" reason="Never"/>
+    <disable_collisions link1="bracelet_link" link2="leg_1_wheel_in" reason="Never"/>
+    <disable_collisions link1="bracelet_link" link2="leg_1_wheel_out" reason="Never"/>
+    <disable_collisions link1="bracelet_link" link2="leg_2" reason="Never"/>
+    <disable_collisions link1="bracelet_link" link2="leg_2_wheel_in" reason="Never"/>
+    <disable_collisions link1="bracelet_link" link2="leg_2_wheel_out" reason="Never"/>
+    <disable_collisions link1="bracelet_link" link2="leg_3" reason="Never"/>
+    <disable_collisions link1="bracelet_link" link2="leg_3_wheel_in" reason="Never"/>
+    <disable_collisions link1="bracelet_link" link2="leg_3_wheel_out" reason="Never"/>
     <disable_collisions link1="bracelet_link" link2="right_inner_finger" reason="Never"/>
     <disable_collisions link1="bracelet_link" link2="right_inner_finger_pad" reason="Never"/>
@@ -120,9 +147,49 @@
     <disable_collisions link1="bracelet_link" link2="spherical_wrist_1_link" reason="Never"/>
     <disable_collisions link1="bracelet_link" link2="spherical_wrist_2_link" reason="Adjacent"/>
-    <disable_collisions link1="bracelet_link" link2="worker_body_link" reason="Default"/>
-    <disable_collisions link1="chair_link" link2="mast_link" reason="Adjacent"/>
+    <disable_collisions link1="chair_link" link2="elevator_shaft" reason="Adjacent"/>
+    <disable_collisions link1="chair_link" link2="elevator_top" reason="Never"/>
+    <disable_collisions link1="chair_link" link2="leg_0" reason="Never"/>
+    <disable_collisions link1="chair_link" link2="leg_0_wheel_in" reason="Never"/>
+    <disable_collisions link1="chair_link" link2="leg_0_wheel_out" reason="Never"/>
+    <disable_collisions link1="chair_link" link2="leg_1" reason="Never"/>
+    <disable_collisions link1="chair_link" link2="leg_1_wheel_in" reason="Never"/>
+    <disable_collisions link1="chair_link" link2="leg_1_wheel_out" reason="Never"/>
+    <disable_collisions link1="chair_link" link2="leg_2" reason="Never"/>
+    <disable_collisions link1="chair_link" link2="leg_2_wheel_in" reason="Never"/>
+    <disable_collisions link1="chair_link" link2="leg_2_wheel_out" reason="Never"/>
+    <disable_collisions link1="chair_link" link2="leg_3" reason="Never"/>
+    <disable_collisions link1="chair_link" link2="leg_3_wheel_in" reason="Never"/>
+    <disable_collisions link1="chair_link" link2="leg_3_wheel_out" reason="Never"/>
     <disable_collisions link1="chair_link" link2="shoulder_link" reason="Never"/>
-    <disable_collisions link1="chair_link" link2="spool_link" reason="Never"/>
     <disable_collisions link1="chair_link" link2="worker_body_link" reason="Never"/>
+    <disable_collisions link1="elevator_shaft" link2="elevator_top" reason="Adjacent"/>
+    <disable_collisions link1="elevator_shaft" link2="leg_0" reason="Never"/>
+    <disable_collisions link1="elevator_shaft" link2="leg_0_wheel_in" reason="Never"/>
+    <disable_collisions link1="elevator_shaft" link2="leg_0_wheel_out" reason="Never"/>
+    <disable_collisions link1="elevator_shaft" link2="leg_1" reason="Never"/>
+    <disable_collisions link1="elevator_shaft" link2="leg_1_wheel_in" reason="Never"/>
+    <disable_collisions link1="elevator_shaft" link2="leg_1_wheel_out" reason="Never"/>
+    <disable_collisions link1="elevator_shaft" link2="leg_2" reason="Default"/>
+    <disable_collisions link1="elevator_shaft" link2="leg_2_wheel_in" reason="Never"/>
+    <disable_collisions link1="elevator_shaft" link2="leg_2_wheel_out" reason="Never"/>
+    <disable_collisions link1="elevator_shaft" link2="leg_3" reason="Default"/>
+    <disable_collisions link1="elevator_shaft" link2="leg_3_wheel_in" reason="Never"/>
+    <disable_collisions link1="elevator_shaft" link2="leg_3_wheel_out" reason="Never"/>
+    <disable_collisions link1="elevator_shaft" link2="shoulder_link" reason="Never"/>
+    <disable_collisions link1="elevator_shaft" link2="worker_body_link" reason="Default"/>
+    <disable_collisions link1="elevator_top" link2="leg_0" reason="Never"/>
+    <disable_collisions link1="elevator_top" link2="leg_0_wheel_in" reason="Never"/>
+    <disable_collisions link1="elevator_top" link2="leg_0_wheel_out" reason="Never"/>
+    <disable_collisions link1="elevator_top" link2="leg_1" reason="Never"/>
+    <disable_collisions link1="elevator_top" link2="leg_1_wheel_in" reason="Never"/>
+    <disable_collisions link1="elevator_top" link2="leg_1_wheel_out" reason="Never"/>
+    <disable_collisions link1="elevator_top" link2="leg_2" reason="Never"/>
+    <disable_collisions link1="elevator_top" link2="leg_2_wheel_in" reason="Never"/>
+    <disable_collisions link1="elevator_top" link2="leg_2_wheel_out" reason="Never"/>
+    <disable_collisions link1="elevator_top" link2="leg_3" reason="Never"/>
+    <disable_collisions link1="elevator_top" link2="leg_3_wheel_in" reason="Never"/>
+    <disable_collisions link1="elevator_top" link2="leg_3_wheel_out" reason="Never"/>
+    <disable_collisions link1="elevator_top" link2="shoulder_link" reason="Never"/>
+    <disable_collisions link1="elevator_top" link2="worker_body_link" reason="Adjacent"/>
     <disable_collisions link1="forearm_link" link2="left_inner_finger" reason="Never"/>
     <disable_collisions link1="forearm_link" link2="left_inner_finger_pad" reason="Never"/>
@@ -130,4 +197,16 @@
     <disable_collisions link1="forearm_link" link2="left_outer_finger" reason="Never"/>
     <disable_collisions link1="forearm_link" link2="left_outer_knuckle" reason="Never"/>
+    <disable_collisions link1="forearm_link" link2="leg_0" reason="Never"/>
+    <disable_collisions link1="forearm_link" link2="leg_0_wheel_in" reason="Never"/>
+    <disable_collisions link1="forearm_link" link2="leg_0_wheel_out" reason="Never"/>
+    <disable_collisions link1="forearm_link" link2="leg_1" reason="Never"/>
+    <disable_collisions link1="forearm_link" link2="leg_1_wheel_in" reason="Never"/>
+    <disable_collisions link1="forearm_link" link2="leg_1_wheel_out" reason="Never"/>
+    <disable_collisions link1="forearm_link" link2="leg_2" reason="Never"/>
+    <disable_collisions link1="forearm_link" link2="leg_2_wheel_in" reason="Never"/>
+    <disable_collisions link1="forearm_link" link2="leg_2_wheel_out" reason="Never"/>
+    <disable_collisions link1="forearm_link" link2="leg_3" reason="Never"/>
+    <disable_collisions link1="forearm_link" link2="leg_3_wheel_in" reason="Never"/>
+    <disable_collisions link1="forearm_link" link2="leg_3_wheel_out" reason="Never"/>
     <disable_collisions link1="forearm_link" link2="right_inner_finger" reason="Never"/>
     <disable_collisions link1="forearm_link" link2="right_inner_finger_pad" reason="Never"/>
@@ -139,5 +218,4 @@
     <disable_collisions link1="forearm_link" link2="spherical_wrist_1_link" reason="Adjacent"/>
     <disable_collisions link1="forearm_link" link2="spherical_wrist_2_link" reason="Never"/>
-    <disable_collisions link1="forearm_link" link2="spool_link" reason="Never"/>
     <disable_collisions link1="forearm_link" link2="worker_body_link" reason="Never"/>
     <disable_collisions link1="left_inner_finger" link2="left_inner_finger_pad" reason="Adjacent"/>
@@ -145,4 +223,16 @@
     <disable_collisions link1="left_inner_finger" link2="left_outer_finger" reason="Adjacent"/>
     <disable_collisions link1="left_inner_finger" link2="left_outer_knuckle" reason="Never"/>
+    <disable_collisions link1="left_inner_finger" link2="leg_0" reason="Never"/>
+    <disable_collisions link1="left_inner_finger" link2="leg_0_wheel_in" reason="Never"/>
+    <disable_collisions link1="left_inner_finger" link2="leg_0_wheel_out" reason="Never"/>
+    <disable_collisions link1="left_inner_finger" link2="leg_1" reason="Never"/>
+    <disable_collisions link1="left_inner_finger" link2="leg_1_wheel_in" reason="Never"/>
+    <disable_collisions link1="left_inner_finger" link2="leg_1_wheel_out" reason="Never"/>
+    <disable_collisions link1="left_inner_finger" link2="leg_2" reason="Never"/>
+    <disable_collisions link1="left_inner_finger" link2="leg_2_wheel_in" reason="Never"/>
+    <disable_collisions link1="left_inner_finger" link2="leg_2_wheel_out" reason="Never"/>
+    <disable_collisions link1="left_inner_finger" link2="leg_3" reason="Never"/>
+    <disable_collisions link1="left_inner_finger" link2="leg_3_wheel_in" reason="Never"/>
+    <disable_collisions link1="left_inner_finger" link2="leg_3_wheel_out" reason="Never"/>
     <disable_collisions link1="left_inner_finger" link2="right_inner_finger" reason="Never"/>
     <disable_collisions link1="left_inner_finger" link2="right_inner_finger_pad" reason="Never"/>
@@ -153,8 +243,19 @@
     <disable_collisions link1="left_inner_finger" link2="spherical_wrist_1_link" reason="Never"/>
     <disable_collisions link1="left_inner_finger" link2="spherical_wrist_2_link" reason="Never"/>
-    <disable_collisions link1="left_inner_finger" link2="worker_body_link" reason="Default"/>
     <disable_collisions link1="left_inner_finger_pad" link2="left_inner_knuckle" reason="Never"/>
     <disable_collisions link1="left_inner_finger_pad" link2="left_outer_finger" reason="Never"/>
     <disable_collisions link1="left_inner_finger_pad" link2="left_outer_knuckle" reason="Never"/>
+    <disable_collisions link1="left_inner_finger_pad" link2="leg_0" reason="Never"/>
+    <disable_collisions link1="left_inner_finger_pad" link2="leg_0_wheel_in" reason="Never"/>
+    <disable_collisions link1="left_inner_finger_pad" link2="leg_0_wheel_out" reason="Never"/>
+    <disable_collisions link1="left_inner_finger_pad" link2="leg_1" reason="Never"/>
+    <disable_collisions link1="left_inner_finger_pad" link2="leg_1_wheel_in" reason="Never"/>
+    <disable_collisions link1="left_inner_finger_pad" link2="leg_1_wheel_out" reason="Never"/>
+    <disable_collisions link1="left_inner_finger_pad" link2="leg_2" reason="Never"/>
+    <disable_collisions link1="left_inner_finger_pad" link2="leg_2_wheel_in" reason="Never"/>
+    <disable_collisions link1="left_inner_finger_pad" link2="leg_2_wheel_out" reason="Never"/>
+    <disable_collisions link1="left_inner_finger_pad" link2="leg_3" reason="Never"/>
+    <disable_collisions link1="left_inner_finger_pad" link2="leg_3_wheel_in" reason="Never"/>
+    <disable_collisions link1="left_inner_finger_pad" link2="leg_3_wheel_out" reason="Never"/>
     <disable_collisions link1="left_inner_finger_pad" link2="right_inner_finger" reason="Never"/>
     <disable_collisions link1="left_inner_finger_pad" link2="right_inner_finger_pad" reason="Never"/>
@@ -165,7 +266,18 @@
     <disable_collisions link1="left_inner_finger_pad" link2="spherical_wrist_1_link" reason="Never"/>
     <disable_collisions link1="left_inner_finger_pad" link2="spherical_wrist_2_link" reason="Never"/>
-    <disable_collisions link1="left_inner_finger_pad" link2="worker_body_link" reason="Default"/>
     <disable_collisions link1="left_inner_knuckle" link2="left_outer_finger" reason="Never"/>
     <disable_collisions link1="left_inner_knuckle" link2="left_outer_knuckle" reason="Never"/>
+    <disable_collisions link1="left_inner_knuckle" link2="leg_0" reason="Never"/>
+    <disable_collisions link1="left_inner_knuckle" link2="leg_0_wheel_in" reason="Never"/>
+    <disable_collisions link1="left_inner_knuckle" link2="leg_0_wheel_out" reason="Never"/>
+    <disable_collisions link1="left_inner_knuckle" link2="leg_1" reason="Never"/>
+    <disable_collisions link1="left_inner_knuckle" link2="leg_1_wheel_in" reason="Never"/>
+    <disable_collisions link1="left_inner_knuckle" link2="leg_1_wheel_out" reason="Never"/>
+    <disable_collisions link1="left_inner_knuckle" link2="leg_2" reason="Never"/>
+    <disable_collisions link1="left_inner_knuckle" link2="leg_2_wheel_in" reason="Never"/>
+    <disable_collisions link1="left_inner_knuckle" link2="leg_2_wheel_out" reason="Never"/>
+    <disable_collisions link1="left_inner_knuckle" link2="leg_3" reason="Never"/>
+    <disable_collisions link1="left_inner_knuckle" link2="leg_3_wheel_in" reason="Never"/>
+    <disable_collisions link1="left_inner_knuckle" link2="leg_3_wheel_out" reason="Never"/>
     <disable_collisions link1="left_inner_knuckle" link2="right_inner_finger" reason="Never"/>
     <disable_collisions link1="left_inner_knuckle" link2="right_inner_finger_pad" reason="Never"/>
@@ -176,6 +288,17 @@
     <disable_collisions link1="left_inner_knuckle" link2="spherical_wrist_1_link" reason="Never"/>
     <disable_collisions link1="left_inner_knuckle" link2="spherical_wrist_2_link" reason="Never"/>
-    <disable_collisions link1="left_inner_knuckle" link2="worker_body_link" reason="Default"/>
     <disable_collisions link1="left_outer_finger" link2="left_outer_knuckle" reason="Adjacent"/>
+    <disable_collisions link1="left_outer_finger" link2="leg_0" reason="Never"/>
+    <disable_collisions link1="left_outer_finger" link2="leg_0_wheel_in" reason="Never"/>
+    <disable_collisions link1="left_outer_finger" link2="leg_0_wheel_out" reason="Never"/>
+    <disable_collisions link1="left_outer_finger" link2="leg_1" reason="Never"/>
+    <disable_collisions link1="left_outer_finger" link2="leg_1_wheel_in" reason="Never"/>
+    <disable_collisions link1="left_outer_finger" link2="leg_1_wheel_out" reason="Never"/>
+    <disable_collisions link1="left_outer_finger" link2="leg_2" reason="Never"/>
+    <disable_collisions link1="left_outer_finger" link2="leg_2_wheel_in" reason="Never"/>
+    <disable_collisions link1="left_outer_finger" link2="leg_2_wheel_out" reason="Never"/>
+    <disable_collisions link1="left_outer_finger" link2="leg_3" reason="Never"/>
+    <disable_collisions link1="left_outer_finger" link2="leg_3_wheel_in" reason="Never"/>
+    <disable_collisions link1="left_outer_finger" link2="leg_3_wheel_out" reason="Never"/>
     <disable_collisions link1="left_outer_finger" link2="right_inner_finger" reason="Never"/>
     <disable_collisions link1="left_outer_finger" link2="right_inner_finger_pad" reason="Never"/>
@@ -186,5 +309,16 @@
     <disable_collisions link1="left_outer_finger" link2="spherical_wrist_1_link" reason="Never"/>
     <disable_collisions link1="left_outer_finger" link2="spherical_wrist_2_link" reason="Never"/>
-    <disable_collisions link1="left_outer_finger" link2="worker_body_link" reason="Default"/>
+    <disable_collisions link1="left_outer_knuckle" link2="leg_0" reason="Never"/>
+    <disable_collisions link1="left_outer_knuckle" link2="leg_0_wheel_in" reason="Never"/>
+    <disable_collisions link1="left_outer_knuckle" link2="leg_0_wheel_out" reason="Never"/>
+    <disable_collisions link1="left_outer_knuckle" link2="leg_1" reason="Never"/>
+    <disable_collisions link1="left_outer_knuckle" link2="leg_1_wheel_in" reason="Never"/>
+    <disable_collisions link1="left_outer_knuckle" link2="leg_1_wheel_out" reason="Never"/>
+    <disable_collisions link1="left_outer_knuckle" link2="leg_2" reason="Never"/>
+    <disable_collisions link1="left_outer_knuckle" link2="leg_2_wheel_in" reason="Never"/>
+    <disable_collisions link1="left_outer_knuckle" link2="leg_2_wheel_out" reason="Never"/>
+    <disable_collisions link1="left_outer_knuckle" link2="leg_3" reason="Never"/>
+    <disable_collisions link1="left_outer_knuckle" link2="leg_3_wheel_in" reason="Never"/>
+    <disable_collisions link1="left_outer_knuckle" link2="leg_3_wheel_out" reason="Never"/>
     <disable_collisions link1="left_outer_knuckle" link2="right_inner_finger" reason="Never"/>
     <disable_collisions link1="left_outer_knuckle" link2="right_inner_finger_pad" reason="Never"/>
@@ -195,8 +329,190 @@
     <disable_collisions link1="left_outer_knuckle" link2="spherical_wrist_1_link" reason="Never"/>
     <disable_collisions link1="left_outer_knuckle" link2="spherical_wrist_2_link" reason="Never"/>
-    <disable_collisions link1="left_outer_knuckle" link2="worker_body_link" reason="Default"/>
-    <disable_collisions link1="mast_link" link2="shoulder_link" reason="Never"/>
-    <disable_collisions link1="mast_link" link2="spool_link" reason="Adjacent"/>
-    <disable_collisions link1="mast_link" link2="worker_body_link" reason="Adjacent"/>
+    <disable_collisions link1="leg_0" link2="leg_0_wheel_in" reason="Default"/>
+    <disable_collisions link1="leg_0" link2="leg_0_wheel_out" reason="Adjacent"/>
+    <disable_collisions link1="leg_0" link2="leg_1" reason="Default"/>
+    <disable_collisions link1="leg_0" link2="leg_1_wheel_in" reason="Never"/>
+    <disable_collisions link1="leg_0" link2="leg_1_wheel_out" reason="Never"/>
+    <disable_collisions link1="leg_0" link2="leg_2" reason="Never"/>
+    <disable_collisions link1="leg_0" link2="leg_2_wheel_in" reason="Never"/>
+    <disable_collisions link1="leg_0" link2="leg_2_wheel_out" reason="Never"/>
+    <disable_collisions link1="leg_0" link2="leg_3" reason="Never"/>
+    <disable_collisions link1="leg_0" link2="leg_3_wheel_in" reason="Never"/>
+    <disable_collisions link1="leg_0" link2="leg_3_wheel_out" reason="Never"/>
+    <disable_collisions link1="leg_0" link2="right_inner_finger" reason="Never"/>
+    <disable_collisions link1="leg_0" link2="right_inner_finger_pad" reason="Never"/>
+    <disable_collisions link1="leg_0" link2="right_inner_knuckle" reason="Never"/>
+    <disable_collisions link1="leg_0" link2="right_outer_finger" reason="Never"/>
+    <disable_collisions link1="leg_0" link2="right_outer_knuckle" reason="Never"/>
+    <disable_collisions link1="leg_0" link2="robotiq_arg2f_base_link" reason="Never"/>
+    <disable_collisions link1="leg_0" link2="shoulder_link" reason="Never"/>
+    <disable_collisions link1="leg_0" link2="spherical_wrist_1_link" reason="Never"/>
+    <disable_collisions link1="leg_0" link2="spherical_wrist_2_link" reason="Never"/>
+    <disable_collisions link1="leg_0" link2="worker_body_link" reason="Adjacent"/>
+    <disable_collisions link1="leg_0_wheel_in" link2="leg_0_wheel_out" reason="Adjacent"/>
+    <disable_collisions link1="leg_0_wheel_in" link2="leg_1" reason="Never"/>
+    <disable_collisions link1="leg_0_wheel_in" link2="leg_1_wheel_in" reason="Never"/>
+    <disable_collisions link1="leg_0_wheel_in" link2="leg_1_wheel_out" reason="Never"/>
+    <disable_collisions link1="leg_0_wheel_in" link2="leg_2" reason="Never"/>
+    <disable_collisions link1="leg_0_wheel_in" link2="leg_2_wheel_in" reason="Never"/>
+    <disable_collisions link1="leg_0_wheel_in" link2="leg_2_wheel_out" reason="Never"/>
+    <disable_collisions link1="leg_0_wheel_in" link2="leg_3" reason="Never"/>
+    <disable_collisions link1="leg_0_wheel_in" link2="leg_3_wheel_in" reason="Never"/>
+    <disable_collisions link1="leg_0_wheel_in" link2="leg_3_wheel_out" reason="Never"/>
+    <disable_collisions link1="leg_0_wheel_in" link2="right_inner_finger" reason="Never"/>
+    <disable_collisions link1="leg_0_wheel_in" link2="right_inner_finger_pad" reason="Never"/>
+    <disable_collisions link1="leg_0_wheel_in" link2="right_inner_knuckle" reason="Never"/>
+    <disable_collisions link1="leg_0_wheel_in" link2="right_outer_finger" reason="Never"/>
+    <disable_collisions link1="leg_0_wheel_in" link2="right_outer_knuckle" reason="Never"/>
+    <disable_collisions link1="leg_0_wheel_in" link2="robotiq_arg2f_base_link" reason="Never"/>
+    <disable_collisions link1="leg_0_wheel_in" link2="shoulder_link" reason="Never"/>
+    <disable_collisions link1="leg_0_wheel_in" link2="spherical_wrist_1_link" reason="Never"/>
+    <disable_collisions link1="leg_0_wheel_in" link2="spherical_wrist_2_link" reason="Never"/>
+    <disable_collisions link1="leg_0_wheel_in" link2="worker_body_link" reason="Never"/>
+    <disable_collisions link1="leg_0_wheel_out" link2="leg_1" reason="Never"/>
+    <disable_collisions link1="leg_0_wheel_out" link2="leg_1_wheel_in" reason="Never"/>
+    <disable_collisions link1="leg_0_wheel_out" link2="leg_1_wheel_out" reason="Never"/>
+    <disable_collisions link1="leg_0_wheel_out" link2="leg_2" reason="Never"/>
+    <disable_collisions link1="leg_0_wheel_out" link2="leg_2_wheel_in" reason="Never"/>
+    <disable_collisions link1="leg_0_wheel_out" link2="leg_2_wheel_out" reason="Never"/>
+    <disable_collisions link1="leg_0_wheel_out" link2="leg_3" reason="Never"/>
+    <disable_collisions link1="leg_0_wheel_out" link2="leg_3_wheel_in" reason="Never"/>
+    <disable_collisions link1="leg_0_wheel_out" link2="leg_3_wheel_out" reason="Never"/>
+    <disable_collisions link1="leg_0_wheel_out" link2="right_inner_finger" reason="Never"/>
+    <disable_collisions link1="leg_0_wheel_out" link2="right_inner_finger_pad" reason="Never"/>
+    <disable_collisions link1="leg_0_wheel_out" link2="right_inner_knuckle" reason="Never"/>
+    <disable_collisions link1="leg_0_wheel_out" link2="right_outer_finger" reason="Never"/>
+    <disable_collisions link1="leg_0_wheel_out" link2="right_outer_knuckle" reason="Never"/>
+    <disable_collisions link1="leg_0_wheel_out" link2="robotiq_arg2f_base_link" reason="Never"/>
+    <disable_collisions link1="leg_0_wheel_out" link2="shoulder_link" reason="Never"/>
+    <disable_collisions link1="leg_0_wheel_out" link2="spherical_wrist_1_link" reason="Never"/>
+    <disable_collisions link1="leg_0_wheel_out" link2="spherical_wrist_2_link" reason="Never"/>
+    <disable_collisions link1="leg_0_wheel_out" link2="worker_body_link" reason="Never"/>
+    <disable_collisions link1="leg_1" link2="leg_1_wheel_in" reason="Default"/>
+    <disable_collisions link1="leg_1" link2="leg_1_wheel_out" reason="Adjacent"/>
+    <disable_collisions link1="leg_1" link2="leg_2" reason="Never"/>
+    <disable_collisions link1="leg_1" link2="leg_2_wheel_in" reason="Never"/>
+    <disable_collisions link1="leg_1" link2="leg_2_wheel_out" reason="Never"/>
+    <disable_collisions link1="leg_1" link2="leg_3" reason="Never"/>
+    <disable_collisions link1="leg_1" link2="leg_3_wheel_in" reason="Never"/>
+    <disable_collisions link1="leg_1" link2="leg_3_wheel_out" reason="Never"/>
+    <disable_collisions link1="leg_1" link2="right_inner_finger" reason="Never"/>
+    <disable_collisions link1="leg_1" link2="right_inner_finger_pad" reason="Never"/>
+    <disable_collisions link1="leg_1" link2="right_inner_knuckle" reason="Never"/>
+    <disable_collisions link1="leg_1" link2="right_outer_finger" reason="Never"/>
+    <disable_collisions link1="leg_1" link2="right_outer_knuckle" reason="Never"/>
+    <disable_collisions link1="leg_1" link2="robotiq_arg2f_base_link" reason="Never"/>
+    <disable_collisions link1="leg_1" link2="shoulder_link" reason="Never"/>
+    <disable_collisions link1="leg_1" link2="spherical_wrist_1_link" reason="Never"/>
+    <disable_collisions link1="leg_1" link2="spherical_wrist_2_link" reason="Never"/>
+    <disable_collisions link1="leg_1" link2="worker_body_link" reason="Adjacent"/>
+    <disable_collisions link1="leg_1_wheel_in" link2="leg_1_wheel_out" reason="Adjacent"/>
+    <disable_collisions link1="leg_1_wheel_in" link2="leg_2" reason="Never"/>
+    <disable_collisions link1="leg_1_wheel_in" link2="leg_2_wheel_in" reason="Never"/>
+    <disable_collisions link1="leg_1_wheel_in" link2="leg_2_wheel_out" reason="Never"/>
+    <disable_collisions link1="leg_1_wheel_in" link2="leg_3" reason="Never"/>
+    <disable_collisions link1="leg_1_wheel_in" link2="leg_3_wheel_in" reason="Never"/>
+    <disable_collisions link1="leg_1_wheel_in" link2="leg_3_wheel_out" reason="Never"/>
+    <disable_collisions link1="leg_1_wheel_in" link2="right_inner_finger" reason="Never"/>
+    <disable_collisions link1="leg_1_wheel_in" link2="right_inner_finger_pad" reason="Never"/>
+    <disable_collisions link1="leg_1_wheel_in" link2="right_inner_knuckle" reason="Never"/>
+    <disable_collisions link1="leg_1_wheel_in" link2="right_outer_finger" reason="Never"/>
+    <disable_collisions link1="leg_1_wheel_in" link2="right_outer_knuckle" reason="Never"/>
+    <disable_collisions link1="leg_1_wheel_in" link2="robotiq_arg2f_base_link" reason="Never"/>
+    <disable_collisions link1="leg_1_wheel_in" link2="shoulder_link" reason="Never"/>
+    <disable_collisions link1="leg_1_wheel_in" link2="spherical_wrist_1_link" reason="Never"/>
+    <disable_collisions link1="leg_1_wheel_in" link2="spherical_wrist_2_link" reason="Never"/>
+    <disable_collisions link1="leg_1_wheel_in" link2="worker_body_link" reason="Never"/>
+    <disable_collisions link1="leg_1_wheel_out" link2="leg_2" reason="Never"/>
+    <disable_collisions link1="leg_1_wheel_out" link2="leg_2_wheel_in" reason="Never"/>
+    <disable_collisions link1="leg_1_wheel_out" link2="leg_2_wheel_out" reason="Never"/>
+    <disable_collisions link1="leg_1_wheel_out" link2="leg_3" reason="Never"/>
+    <disable_collisions link1="leg_1_wheel_out" link2="leg_3_wheel_in" reason="Never"/>
+    <disable_collisions link1="leg_1_wheel_out" link2="leg_3_wheel_out" reason="Never"/>
+    <disable_collisions link1="leg_1_wheel_out" link2="right_inner_finger" reason="Never"/>
+    <disable_collisions link1="leg_1_wheel_out" link2="right_inner_finger_pad" reason="Never"/>
+    <disable_collisions link1="leg_1_wheel_out" link2="right_inner_knuckle" reason="Never"/>
+    <disable_collisions link1="leg_1_wheel_out" link2="right_outer_finger" reason="Never"/>
+    <disable_collisions link1="leg_1_wheel_out" link2="right_outer_knuckle" reason="Never"/>
+    <disable_collisions link1="leg_1_wheel_out" link2="robotiq_arg2f_base_link" reason="Never"/>
+    <disable_collisions link1="leg_1_wheel_out" link2="shoulder_link" reason="Never"/>
+    <disable_collisions link1="leg_1_wheel_out" link2="spherical_wrist_1_link" reason="Never"/>
+    <disable_collisions link1="leg_1_wheel_out" link2="spherical_wrist_2_link" reason="Never"/>
+    <disable_collisions link1="leg_1_wheel_out" link2="worker_body_link" reason="Never"/>
+    <disable_collisions link1="leg_2" link2="leg_2_wheel_in" reason="Default"/>
+    <disable_collisions link1="leg_2" link2="leg_2_wheel_out" reason="Adjacent"/>
+    <disable_collisions link1="leg_2" link2="leg_3" reason="Default"/>
+    <disable_collisions link1="leg_2" link2="leg_3_wheel_in" reason="Never"/>
+    <disable_collisions link1="leg_2" link2="leg_3_wheel_out" reason="Never"/>
+    <disable_collisions link1="leg_2" link2="right_inner_finger" reason="Never"/>
+    <disable_collisions link1="leg_2" link2="right_inner_finger_pad" reason="Never"/>
+    <disable_collisions link1="leg_2" link2="right_inner_knuckle" reason="Never"/>
+    <disable_collisions link1="leg_2" link2="right_outer_finger" reason="Never"/>
+    <disable_collisions link1="leg_2" link2="right_outer_knuckle" reason="Never"/>
+    <disable_collisions link1="leg_2" link2="robotiq_arg2f_base_link" reason="Never"/>
+    <disable_collisions link1="leg_2" link2="shoulder_link" reason="Never"/>
+    <disable_collisions link1="leg_2" link2="spherical_wrist_1_link" reason="Never"/>
+    <disable_collisions link1="leg_2" link2="spherical_wrist_2_link" reason="Never"/>
+    <disable_collisions link1="leg_2" link2="worker_body_link" reason="Adjacent"/>
+    <disable_collisions link1="leg_2_wheel_in" link2="leg_2_wheel_out" reason="Adjacent"/>
+    <disable_collisions link1="leg_2_wheel_in" link2="leg_3" reason="Never"/>
+    <disable_collisions link1="leg_2_wheel_in" link2="leg_3_wheel_in" reason="Never"/>
+    <disable_collisions link1="leg_2_wheel_in" link2="leg_3_wheel_out" reason="Never"/>
+    <disable_collisions link1="leg_2_wheel_in" link2="right_inner_finger" reason="Never"/>
+    <disable_collisions link1="leg_2_wheel_in" link2="right_inner_finger_pad" reason="Never"/>
+    <disable_collisions link1="leg_2_wheel_in" link2="right_inner_knuckle" reason="Never"/>
+    <disable_collisions link1="leg_2_wheel_in" link2="right_outer_finger" reason="Never"/>
+    <disable_collisions link1="leg_2_wheel_in" link2="right_outer_knuckle" reason="Never"/>
+    <disable_collisions link1="leg_2_wheel_in" link2="robotiq_arg2f_base_link" reason="Never"/>
+    <disable_collisions link1="leg_2_wheel_in" link2="shoulder_link" reason="Never"/>
+    <disable_collisions link1="leg_2_wheel_in" link2="spherical_wrist_1_link" reason="Never"/>
+    <disable_collisions link1="leg_2_wheel_in" link2="spherical_wrist_2_link" reason="Never"/>
+    <disable_collisions link1="leg_2_wheel_in" link2="worker_body_link" reason="Never"/>
+    <disable_collisions link1="leg_2_wheel_out" link2="leg_3" reason="Never"/>
+    <disable_collisions link1="leg_2_wheel_out" link2="leg_3_wheel_in" reason="Never"/>
+    <disable_collisions link1="leg_2_wheel_out" link2="leg_3_wheel_out" reason="Never"/>
+    <disable_collisions link1="leg_2_wheel_out" link2="right_inner_finger" reason="Never"/>
+    <disable_collisions link1="leg_2_wheel_out" link2="right_inner_finger_pad" reason="Never"/>
+    <disable_collisions link1="leg_2_wheel_out" link2="right_inner_knuckle" reason="Never"/>
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