Commit message: sim mag gripper works and can be planned for

File: kortex_scripts/robot_equipment/urdf/mag_gripper_end_effector.xacro (robot description, xacro)
@@ -51,6 +51,6 @@
                 <parent link="mag_gripper_end_effector" />
                 <child link="end_effector" />
-                <origin rpy="0 0 0" xyz="0 0 0.05325" />
-                <limit effort="30" velocity="1.0" lower="0" upper="0" />
+                <origin rpy="0 0 0" xyz="0 0 0.10325" />
+                <limit effort="1000" velocity="1.0" lower="0" upper="0" />
             </joint>
             <gazebo>

Commit message: added joint positions to python parser

File: kortex_scripts/robot_equipment/urdf/mag_gripper_end_effector.xacro (robot description, xacro)
@@ -51,5 +51,5 @@
                 <parent link="mag_gripper_end_effector" />
                 <child link="end_effector" />
-                <origin rpy="0 0 0" xyz="0 0 0.10325" />
+                <origin rpy="0 0 0" xyz="0 0 0.075" />
                 <limit effort="1000" velocity="1.0" lower="0" upper="0" />
             </joint>
